File: Aktive_Balancing/KiCAD/Aktive_Bal/Aktive_Bal.kicad_sch (KiCad schematic)
At the start: 115 parts, among them Q1 NMOS, Q10 NTTFS6H888NL, Q11 NTTFS6H888NL, Q12 NTTFS6H888NL, Q13 NTTFS6H888NL, Q14 NTTFS6H888NL, Q15 NTTFS6H888NL, Q16 NTTFS6H888NL, Q17 NTTFS6H888NL, Q18 NTTFS6H888NL, Q19 NTTFS6H888NL, Q2 NMOS, Q20 NTTFS6H888NL, Q21 NTTFS6H888NL, Q22 NTTFS6H888NL, Q23 NTTFS6H888NL, Q24 NTTFS6H888NL, Q25 NTTFS6H888NL, Q26 NTTFS6H888NL, Q27 NTTFS6H888NL, Q28 NTTFS6H888NL, Q29 NTTFS6H888NL, Q3 NTTFS6H888NL, Q30 NTTFS6H888NL, Q31 NTTFS6H888NL, Q32 NTTFS6H888NL, Q33 NTTFS6H888NL, Q34 NTTFS6H888NL, Q4 NTTFS6H888NL, Q5 NTTFS6H888NL, Q6 NTTFS6H888NL, Q7 NTTFS6H888NL, Q8 NTTFS6H888NL, Q9 NTTFS6H888NL, U1 SCW20C-12, U10 LTV-847S, U11 LTV-847S, U12 LTV-847S, U2 EC1SA16N, U3 LM2596S-ADJ, U4 TL084, U5 ADUM1250ARZ-RL7, U6 PCA9306DC, U7 LM1117IMPX_3_3_NOPB, U8 MCP4725xxx-xCH, U9 LTV-847S

Commit message: kicad
Parts:
- removed Q1: NMOS, symbol Simulation_SPICE:NMOS
- added J1: A-DF_09_A_KG-T4S, A-DF_09_A_KG-T4S:ASSMANN_A-DF_09_A_KG-T4S, symbol Aktive_Bal_Lib:A-DF_09_A_KG-T4S
- added U13: RFP12N10L, TO-220AB_ONS, symbol Aktive_Bal_Lib:RFP12N10L
- added U14: PCF8575CDB, DB24, symbol Aktive_Bal_Lib:PCF8575CDB
Connections:
- net Bat+: now also U1.22 (+Vin), U1.23 (+Vin)
- net Bat_GND: now also U13.2 (DRAIN); no longer U1.2 (-Vin), U1.3 (-Vin)
- net at JP3.2 (B), R16.1, U6.4 (SDA1)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: now also U14.23 (SDA)
- net at JP4.2 (B), R15.1, U6.3 (SCL1)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: now also U14.22 (SCL)
- new net: U1.2 (-Vin), U1.3 (-Vin), U13.3 (SOURCE)
Other:
- note removed: "Enable Mosfet?"
- moved on the sheet: C7, C8, U1, U2, U4E, U7

Commit message: kicad klopf klopf
Parts:
- removed J1: A-DF_09_A_KG-T4S, A-DF_09_A_KG-T4S:ASSMANN_A-DF_09_A_KG-T4S, symbol Aktive_Bal_Lib:A-DF_09_A_KG-T4S
- added C12: 0.1µ, symbol Device:C_Small
- added J2: Sockel_BluePill, Aktive_Bal_Footprints:SockelBluepill Dupont leisten, symbol Aktive_Bal_Lib:Sockel_BluePill
- added J3: A-DF_09_A_KG-T4S, A-DF_09_A_KG-T4S:ASSMANN_A-DF_09_A_KG-T4S, symbol Aktive_Bal_Lib:A-DF_09_A_KG-T4S
- added R53: 120, symbol Device:R
- added R54: CMP-R100-1.0, symbol Aktive_Bal_Lib:CMP-R100-1.0
- added U15: SN65HVD233, Package_SO:SOIC-8_3.9x4.9mm_P1.27mm, symbol Interface_CAN_LIN:SN65HVD233
- R21, R22, R23, R24, R25, R26, R27, R28, R29, R30, R31, R32, R33, R34, R35, R36: value 220 -> 680
Connections:
- net +5V: now also U14.24 (VCC)
- net B1: now also U14.4 (P00)
- net B10: now also U14.19 (P16)
- net B11: now also U14.18 (P15)
- net B12: now also U14.17 (P14)
- net B13: now also U14.16 (P13)
- net B14: now also U14.15 (P12)
- net B15: now also U14.14 (P11)
- net B16: now also U14.13 (P10)
- net B2: now also U14.5 (P01)
- net B3: now also U14.6 (P02)
- net B4: now also U14.7 (P03)
- net B5: now also U14.8 (P04)
- net B6: now also U14.9 (P05)
- net B7: now also U14.10 (P06)
- net B8: now also U14.11 (P07)
- net B9: now also U14.20 (P17)
- net GND_float: no longer U9.11
- net GND_float2: now also U14.12 (GND), R54.4; no longer Q11.1 (S), Q11.2 (S), Q11.3 (S), Q12.1 (S), Q12.2 (S), Q12.3 (S), Q13.1 (S), Q13.2 (S), Q13.3 (S), Q14.1 (S), Q14.2 (S), Q14.3 (S), Q19.1 (S), Q19.2 (S), Q19.3 (S), Q20.1 (S), Q20.2 (S), Q20.3 (S), Q21.1 (S), Q21.2 (S), Q21.3 (S), Q22.1 (S), Q22.2 (S), Q22.3 (S), Q23.1 (S), Q23.2 (S), Q23.3 (S), Q24.1 (S), Q24.2 (S), Q24.3 (S), Q25.1 (S), Q25.2 (S), Q25.3 (S), Q26.1 (S), Q26.2 (S), Q26.3 (S), Q4.1 (S), Q4.2 (S), Q4.3 (S), Q5.1 (S), Q5.2 (S), Q5.3 (S), Q7.1 (S), Q7.2 (S), Q7.3 (S), Q8.1 (S), Q8.2 (S), Q8.3 (S)
- net SCLµC: now also J2.14 (B6)
- net SDAµC: now also J2.15 (B7)
- net V_I_Bal: now also R54.2
- net +3.3Vµ: now reaches C5.1, R10.2, R11.2, U5.1 (VDD1)
- net +3.3Vµ: now also C12.1, J2.20 (3.3), U15.3 (VCC)
- net GNDµ: now reaches C5.2, U5.4 (GND1)
- net GNDµ: now also J2.19 (G)
- new net: Q11.1 (S), Q11.2 (S), Q11.3 (S), Q12.1 (S), Q12.2 (S), Q12.3 (S), Q13.1 (S), Q13.2 (S), Q13.3 (S), Q14.1 (S), Q14.2 (S), Q14.3 (S), Q19.1 (S), Q19.2 (S), Q19.3 (S), Q20.1 (S), Q20.2 (S), Q20.3 (S), Q21.1 (S), Q21.2 (S), Q21.3 (S), Q22.1 (S), Q22.2 (S), Q22.3 (S), Q23.1 (S), Q23.2 (S), Q23.3 (S), Q24.1 (S), Q24.2 (S), Q24.3 (S), Q25.1 (S), Q25.2 (S), Q25.3 (S), Q26.1 (S), Q26.2 (S), Q26.3 (S), Q4.1 (S), Q4.2 (S), Q4.3 (S), Q5.1 (S), Q5.2 (S), Q5.3 (S), Q7.1 (S), Q7.2 (S), Q7.3 (S), Q8.1 (S), Q8.2 (S), Q8.3 (S), R54.1
- new net: J2.9 (A12), U15.1 (D)
- new net: J2.8 (A11), U15.4 (R)
- new net: J3.2, R53.1, U15.6 (CANL)
- new net: J3.7, R53.2, U15.7 (CANH)
- new net CAN_GND: C12.2, J3.3, U15.2 (GND), U15.5 (LBK), U15.8 (Rs)
- no-connect marks 0 -> 8
Other:
- note added: "Adrressee?"
- note added: "SN65HVD233QDRQ1"
- note added: "can gnd und gnd µ gleeiches potential?"
- note added: "invertierte Logik!"
- note added: "iso i2c"
- note added: "optional wenn pc adapter schon hat?!"
- note removed: "3.3v µC?"
- note removed: "gnd µc?"

Commit message: kicad weiter weiter
Parts:
- removed C4: C, symbol Device:C
- removed Q2: NMOS, symbol Simulation_SPICE:NMOS
- added C4: 47µ, symbol Device:C_Polarized
- added Q1: BSS316NH6327XTSA1, Package_TO_SOT_SMD:SOT-23, symbol Aktive_Bal_Lib:BSS316NH6327XTSA1
- R8: value 1k -> 800
Connections:
- net Bal: now also C4.1
- net GND_float: now also C4.2
- net GND_float2: now also R54.3
- net enable: now reaches U13.1 (GATE)
- net at C3.1, R9.2, U3.4 (FB): now also Q1.3 (D)
- net at R7.2, R8.2: now also Q1.2 (S)
- net at R6.2: now also Q1.1 (G)
Other:
- note added: "Feedback weg von der Spule"
- note removed: "welcher mosfet?"
- moved on the sheet: L1, R53

Commit message: fehler im Kicad
Parts:
- removed JP3, JP4: Jumper_2_Open, symbol Jumper:Jumper_2_Open
- C10: value C_Small -> 100p
- R10, R11: value 1k -> 4k7
- R12, R13: value 1k -> 2k2
- R15, R16: value 10k -> 4k7
Connections:
- net GND_float2: now also U14.2 (A1), U14.21 (A0), U14.3 (A2)
- net at R12.1, U5.7 (SDA2), U6.5 (SDA2): now also U14.23 (SDA)
- net at R15.1, U6.3 (SCL1), U8.5 (SCL): no longer U14.22 (SCL)
- net at R16.1, U6.4 (SDA1), U8.4 (SDA): no longer U14.23 (SDA)
- net at R13.1, U5.6 (SCL2), U6.6 (SCL2): now also U14.22 (SCL)
- no-connect marks 8 -> 9
Other:
- note added: "Adresse A0 GND -> 0x60"
- note added: "Adresse A2,A1,A0 GND -> 0x20"
- note added: "optional brücken"
- note removed: "Adrressee?"
- note removed: "welches gnd??"
- moved on the sheet: C1, J2, U14

Commit message: kicad bla bla
Parts:
- added C13, C14: 2.2µ, symbol Device:C_Small
- added C15, C16: 1000p, symbol Device:C_Small
- added C17: 4u7, symbol Device:C_Small
- added C18, C19: 22µ, symbol Device:C_Small
- added FL1: Choke_CommonMode_PulseElectronics_PH9455x156NL, Inductor_THT:L_CommonMode_PulseElectronics_PH9455xxx6NL_2, symbol Filter:Choke_CommonMode_PulseElectronics_PH9455x156NL
- added J1: Conn_01x01_Pin, symbol Connector:Conn_01x01_Pin
- added J4: Screw_Terminal_01x02, symbol Connector:Screw_Terminal_01x02
- added JP3, JP4, JP5: Jumper_2_Open, symbol Jumper:Jumper_2_Open
- added R55: 100, symbol Device:R
- added R56: 1Meg, symbol Device:R
- C9: value C_Small -> 10µ
- R14: value 100m -> 10
Connections:
- net CAN_GND is gone; now on net GNDµ: C12.2, J3.3, U15.2 (GND), U15.5 (LBK), U15.8 (Rs)
- net GND_float is gone; now on net GND_float2: C1.2, C4.2, D1.2 (A), U1.16 (-Vout), U10.11, U10.13, U10.15, U10.9, U11.11, U11.13, U11.15, U11.9, U12.11, U12.13, U12.15, U12.9, U2.1 (+V_Input), U3.3 (GND), U3.5 (~{ON}/OFF), U9.13, U9.15, U9.9
- net +12V: now also C15.1, C17.2
- net +5V: now also C7.1, U7.3 (VI), C19.2
- net -5V: now also C18.1; no longer C7.1, U7.3 (VI)
- net Bat_GND: now also U13.3 (SOURCE), J4.2 (Pin_2); no longer U13.2 (DRAIN)
- net C0: now also R56.2
- net GND_float2: now also U9.11, C16.2, C17.1, C18.2, C19.1
- net at R12.1, U14.23 (SDA), U5.7 (SDA2)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: now also JP5.1 (A)
- net at U1.2 (-Vin), U1.3 (-Vin): now also C14.1, C16.1, FL1.4; no longer U13.3 (SOURCE)
- net at R13.1, U14.22 (SCL), U5.6 (SCL2)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: now also JP4.1 (A)
- net at R15.1, U6.3 (SCL1), U8.5 (SCL): now also JP4.2 (B)
- net at J3.7, U15.7 (CANH): now also JP3.2 (B); no longer R53.2
- net at R16.1, U6.4 (SDA1), U8.4 (SDA): now also JP5.2 (B)
- net at R37.1, U9.16: now also R55.1; no longer Q3.4 (G)
- net Bat+: no longer names the net of U1.22 (+Vin), U1.23 (+Vin)
- net Bat+: now also C14.2, C15.2, FL1.3, J1.1 (Pin_1)
- new net: C13.1, FL1.1, U13.2 (DRAIN)
- new net: C13.2, FL1.2, J4.1 (Pin_1)
- new net: Q3.4 (G), R55.2, R56.1
- new net: JP3.1 (A), R53.2
Other:
- note added: "325 µH"
- note added: "RG RGS"
- note added: "Zugangspins"
- note added: "connector"
- note removed: "can gnd und gnd µ gleeiches potential?"
- note removed: "kapazität?"
- note removed: "optional wenn pc adapter schon hat?!"
- moved on the sheet: C7, C8, R10, R11, R53, U1, U13, U2, U4E, U7

Commit message: kicad export
Parts:
- C10: value 100p -> 0.1n
- C12: value 0.1µ -> 100n
- C13, C14: footprint (none) -> Capacitor_SMD:C_0805_2012Metric
- C15, C16: value 1000p -> 1n
- C17: value 4u7 -> 4.7µ; footprint (none) -> Capacitor_SMD:C_0805_2012Metric
- C18, C19: value 22µ -> 1µ; footprint (none) -> Capacitor_SMD:C_0805_2012Metric
- C5, C6: value 100n -> 0.1µ
- C7, C8: value 10µ -> 10µ tantal; footprint (none) -> Capacitor_SMD:C_0805_2012Metric
- L1: value 48µ -> 47µ
- R1, R53: footprint (none) -> Resistor_SMD:R_0805_2012Metric
- R10, R11, R15, R16: value 4k7 -> 4.7k
- R12, R13: value 2k2 -> 2.2k
- R21, R22, R23, R24, R25, R26, R27, R28, R29, R30, R31, R32, R33, R34, R35, R36: value 680 -> 390
- U4: footprint (none) -> Package_SO:SOIC-14_3.9x8.7mm_P1.27mm
Other:
- note removed: "Tantal"
Changed lines of the file:
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@@
 		)
 	)
-	(text "Tantal\n"
-		(exclude_from_sim no)
-		(at 214.122 26.924 0)
-		(effects
-			(font
-				(size 1.27 1.27)
-			)
-		)
-	)
 	(text "Keramik"
 		(exclude_from_sim no)
@@
 		)
 	)
-	(text "Tantal\n"
-		(exclude_from_sim no)
-		(at 188.468 27.432 0)
-		(effects
-			(font
-				(size 1.27 1.27)
-			)
-		)
-	)
 	(text "invertierte Logik!\n"
 		(exclude_from_sim no)
@@
 	)
 	(junction
-		(at 50.8 29.21)
-		(diameter 0)
-		(color 0 0 0 0)
-	)
-	(junction
 		(at 309.88 160.02)
 		(diameter 0)
@@
 	)
 	(junction
+		(at 50.8 29.21)
+		(diameter 0)
+		(color 0 0 0 0)
+	)
+	(junction
 		(at 215.9 205.74)
 		(diameter 0)
@@
 	(wire
 		(pts
+			(xy 50.8 29.21) (xy 59.69 29.21)
+		)
+		(stroke
+			(width 0)
+			(type default)
+		)
+	)
+	(wire
+		(pts
 			(xy 39.37 50.8) (xy 39.37 54.61)
 		)
@@
 	(wire
 		(pts
-			(xy 50.8 29.21) (xy 50.8 40.64)
-		)
-		(stroke
-			(width 0)
-			(type default)
-		)
-	)
-	(wire
-		(pts
 			(xy 167.64 26.67) (xy 167.64 29.21)
 		)
@@
 	(wire
 		(pts
+			(xy 50.8 29.21) (xy 50.8 40.64)
+		)
+		(stroke
+			(width 0)
+			(type default)
+		)
+	)
+	(wire
+		(pts
 			(xy 238.76 187.96) (xy 254 187.96)
 		)
@@
 	(wire
 		(pts
-			(xy 50.8 29.21) (xy 59.69 29.21)
-		)
-		(stroke
-			(width 0)
-			(type default)
-		)
-	)
-	(wire
-		(pts
 			(xy 171.45 189.23) (xy 204.47 189.23)
 		)
@@
 			)
 		)
-		(property "Value" "2k2"
+		(property "Value" "2.2k"
 			(at 97.79 62.2299 0)
 			(show_name no)
@@
 			)
 		)
-		(property "Value" "100n"
+		(property "Value" "0.1µ"
 			(at 91.694 67.056 0)
 			(show_name no)
@@
 			)
 		)
-		(property "Value" "680"
+		(property "Value" "390"
 			(at 284.48 95.25 90)
 			(show_name no)
@@
 			)
 		)
-		(property "Value" "100p"
+		(property "Value" "0.1n"
 			(at 123.444 76.708 90)
 			(show_name no)
@@
 			)
 		)
-		(property "Value" "680"
+		(property "Value" "390"
 			(at 284.48 146.05 90)
 			(show_name no)
@@
 			)
 		)
-		(property "Value" "4k7"
+		(property "Value" "4.7k"
 			(at 153.67 74.9299 0)
 			(show_name no)
@@
 			)
 		)
-		(property "Value" "4k7"
+		(property "Value" "4.7k"
 			(at 46.99 59.6899 0)
 			(show_name no)
@@
 			)
 		)
-		(property "Value" "1000p"
+		(property "Value" "1n"
 			(at 114.3 46.228 90)
 			(show_name no)
@@
 			)
 		)
-		(property "Value" "100n"
+		(property "Value" "0.1µ"
 			(at 42.164 71.12 0)
 			(show_name no)
@@
 			)
 		)
-		(property "Value" "680"
+		(property "Value" "390"
 			(at 284.48 135.89 90)
 			(show_name no)
@@
 			)
 		)
-		(property "Value" "680"
+		(property "Value" "390"
 			(at 284.48 105.41 90)
 			(show_name no)
@@
 			)
 		)
-		(property "Footprint" ""
+		(property "Footprint" "Package_SO:SOIC-14_3.9x8.7mm_P1.27mm"
 			(at 110.49 218.44 0)
 			(hide yes)
@@
 			)
 		)
-		(property "Footprint" ""
+		(property "Footprint" "Capacitor_SMD:C_0805_2012Metric"
 			(at 72.39 26.67 0)
 			(hide yes)
@@
 			)
 		)
-		(property "Footprint" ""
+		(property "Footprint" "Package_SO:SOIC-14_3.9x8.7mm_P1.27mm"
 			(at 64.77 177.8 0)
 			(hide yes)
@@
 			)
 		)
-		(property "Value" "680"
+		(property "Value" "390"
 			(at 284.48 85.09 90)
 			(show_name no)
@@
 			)
 		)
-		(property "Footprint" ""
+		(property "Footprint" "Package_SO:SOIC-14_3.9x8.7mm_P1.27mm"
 			(at 91.44 175.26 0)
 			(hide yes)
@@
 			)
 		)
-		(property "Value" "22µ"
+		(property "Value" "1µ"
 			(at 172.72 28.194 0)
 			(show_name no)
@@
 			)
 		)
-		(property "Footprint" ""
+		(property "Footprint" "Capacitor_SMD:C_0805_2012Metric"
 			(at 170.18 26.67 0)
 			(hide yes)
@@
 			)
 		)
-		(property "Value" "680"
+		(property "Value" "390"
 			(at 284.48 45.72 90)
 			(show_name no)
@@
 			)
 		)
-		(property "Value" "680"
+		(property "Value" "390"
 			(at 284.48 125.73 90)
 			(show_name no)
@@
 			)
 		)
-		(property "Value" "680"
+		(property "Value" "390"
 			(at 284.48 196.85 90)
 			(show_name no)
@@
 			)
 		)
-		(property "Value" "1000p"
+		(property "Value" "1n"
 			(at 113.03 12.192 90)
 			(show_name no)
@@
 			)
 		)
-		(property "Value" "22µ"
+		(property "Value" "1µ"
 			(at 171.958 22.606 0)
 			(show_name no)
@@
 			)
 		)
-		(property "Footprint" ""
+		(property "Footprint" "Capacitor_SMD:C_0805_2012Metric"
 			(at 170.18 21.59 0)
 			(hide yes)
@@
 			)
 		)
-		(property "Value" "4k7"
+		(property "Value" "4.7k"
 			(at 33.782 59.69 0)
 			(show_name no)
@@
 			)
 		)
-		(property "Value" "2k2"
+		(property "Value" "2.2k"
 			(at 106.426 61.976 0)
 			(show_name no)
@@
 			)
 		)
-		(property "Value" "4u7"
+		(property "Value" "4.7µ"
 			(at 138.43 25.4062 0)
 			(show_name no)
@@
 			)
 		)
-		(property "Footprint" ""
+		(property "Footprint" "Capacitor_SMD:C_0805_2012Metric"
 			(at 135.89 24.13 0)
 			(hide yes)
@@
 			)
 		)
-		(property "Value" "680"
+		(property "Value" "390"
 			(at 284.48 207.01 90)
 			(show_name no)
@@
 			)
 		)
-		(property "Value" "48µ"
+		(property "Value" "47µ"
 			(at 210.82 203.2 90)
 			(show_name no)
@@
 			)
 		)
-		(property "Value" "680"
+		(property "Value" "390"
 			(at 284.48 156.21 90)
 			(show_name no)
@@
 			)
 		)
-		(property "Value" "680"
+		(property "Value" "390"
 			(at 284.48 176.53 90)
 			(show_name no)
@@
 			)
 		)
-		(property "Footprint" ""
+		(property "Footprint" "Package_SO:SOIC-14_3.9x8.7mm_P1.27mm"
 			(at 57.15 214.63 0)
 			(hide yes)
@@
 			)
 		)
-		(property "Footprint" ""
+		(property "Footprint" "Package_SO:SOIC-14_3.9x8.7mm_P1.27mm"
 			(at 119.38 177.8 0)
 			(hide yes)
@@
 			)
 		)
-		(property "Footprint" ""
+		(property "Footprint" "Resistor_SMD:R_0805_2012Metric"
 			(at 42.672 82.55 90)
 			(hide yes)
@@
 			)
 		)
-		(property "Value" "680"
+		(property "Value" "390"
 			(at 284.48 186.69 90)
 			(show_name no)
@@
 			)
 		)
-		(property "Value" "680"
+		(property "Value" "390"
 			(at 284.48 74.93 90)
 			(show_name no)
@@
 			)
 		)
-		(property "Value" "10µ"
+		(property "Value" "10µ tantal"
 			(at 186.69 25.4062 0)
 			(show_name no)
@@
 			)
 		)
-		(property "Footprint" ""
+		(property "Footprint" "Capacitor_SMD:C_0805_2012Metric"
 			(at 184.15 24.13 0)
 			(hide yes)
@@
 			)
 		)
-		(property "Value" "0.1µ"
+		(property "Value" "100n"
 			(at 55.88 134.6262 0)
 			(show_name no)
@@
 			)
 		)
-		(property "Value" "680"
+		(property "Value" "390"
 			(at 284.48 55.88 90)
 			(show_name no)
@@
 			)
 		)
-		(property "Value" "10µ"
+		(property "Value" "10µ tantal"
 			(at 212.09 25.4062 0)
 			(show_name no)
@@
 			)
 		)
-		(property "Footprint" ""
+		(property "Footprint" "Capacitor_SMD:C_0805_2012Metric"
 			(at 209.55 24.13 0)
 			(hide yes)
@@
 			)
 		)
-		(property "Value" "680"
+		(property "Value" "390"
 			(at 284.48 35.56 90)
 			(show_name no)
@@
 			)
 		)
-		(property "Value" "4k7"
+		(property "Value" "4.7k"
 			(at 162.56 74.9299 0)
 			(show_name no)
@@
 			)
 		)
-		(property "Value" "680"
+		(property "Value" "390"
 			(at 284.48 25.4 90)
 			(show_name no)
@@
 			)
 		)
-		(property "Footprint" ""
+		(property "Footprint" "Capacitor_SMD:C_0805_2012Metric"
 			(at 50.8 26.67 0)
 			(hide yes)
@@
 			)
 		)
-		(property "Footprint" ""
+		(property "Footprint" "Resistor_SMD:R_0805_2012Metric"
 			(at 48.26 176.022 90)
 			(hide yes)

Commit message: kicad
Parts:
- added J5, J6: Conn_01x01_Pin, symbol Connector:Conn_01x01_Pin
- added R57, R58, R59, R60, R61, R62, R63, R64, R65, R66, R67, R68, R69, R70, R71: 100, symbol Device:R
- added R72, R73, R74, R75, R76, R77, R78, R79, R80, R81, R82, R83, R84, R85, R86: 1Meg, symbol Device:R
- FL1: value Choke_CommonMode_PulseElectronics_PH9455x156NL -> Choke_CommonMode_TCK_050; footprint Inductor_THT:L_CommonMode_PulseElectronics_PH9455xxx6NL_2 -> (none)
Connections:
- net +12V: now also J5.1 (Pin_1)
- net Bal: no longer Q30.5 (D), Q30.6 (D), Q30.7 (D), Q30.8 (D)
- net C1: now also R72.2
- net C10: now also R81.2
- net C11: no longer Q30.1 (S), Q30.2 (S), Q30.3 (S)
- net C12: now also R83.2
- net C13: now also R84.2
- net C14: now also R85.2
- net C15: now also R86.2
- net C2: now also R73.2
- net C3: now also R74.2
- net C4: now also R75.2
- net C5: now also R76.2
- net C6: now also R77.2
- net C7: now also R78.2
- net C8: now also R79.2
- net C9: now also R80.2
- net at R46.1, U11.14: now also R65.1; no longer Q28.4 (G)
- net at R38.1, U9.14: now also R57.1; no longer Q6.4 (G)
- net at R40.1, U9.10: now also R59.1; no longer Q10.4 (G)
- net at R52.1, U12.10: now also R71.1; no longer Q34.4 (G)
- net at C14.1, C16.1, FL1.4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: now also J6.1 (Pin_1)
- net at R44.1, U10.10: now also R63.1; no longer Q18.4 (G)
- net at R42.1, U10.14: now also R61.1; no longer Q16.4 (G)
- net at R39.1, U9.12: now also R58.1; no longer Q9.4 (G)
- net at R49.1, U12.16: now also R68.1; no longer Q31.4 (G)
- net at R47.1, U11.12: now also R66.1; no longer Q29.4 (G)
- net at R48.1, U11.10: now also R67.1; no longer Q30.4 (G)
- net at R45.1, U11.16: now also R64.1; no longer Q27.4 (G)
- net at R41.1, U10.16: now also R60.1; no longer Q15.4 (G)
- net at R50.1, U12.14: now also R69.1; no longer Q32.4 (G)
- net at R43.1, U10.12: now also R62.1; no longer Q17.4 (G)
- net at R51.1, U12.12: now also R70.1; no longer Q33.4 (G)
- new net: Q33.4 (G), R70.2, R85.1
- new net: Q32.4 (G), R69.2, R84.1
- new net: Q27.4 (G), R64.2, R79.1
- new net: Q15.4 (G), R60.2, R75.1
- new net: Q6.4 (G), R57.2, R72.1
- new net: Q10.4 (G), R59.2, R74.1
- new net: Q30.4 (G), R67.2, R82.1
- new net: Q18.4 (G), R63.2, R78.1
- new net: Q34.4 (G), R71.2, R86.1
- new net: Q31.4 (G), R68.2, R83.1
- new net: Q16.4 (G), R61.2, R76.1
- new net: Q30.1 (S), Q30.2 (S), Q30.3 (S), R82.2
- new net: Q30.5 (D), Q30.6 (D), Q30.7 (D), Q30.8 (D)
- new net: Q9.4 (G), R58.2, R73.1
- new net: Q29.4 (G), R66.2, R81.1
- new net: Q17.4 (G), R62.2, R77.1
- new net: Q28.4 (G), R65.2, R80.1
Other:
- note removed: "Adresse A0 GND -> 0x60"
- note removed: "Adresse A2,A1,A0 GND -> 0x20"
- note removed: "Keramik"
- note removed: "RG RGS"
- note removed: "Zugangspins"
- note removed: "invertierte Logik!"
- moved on the sheet: C14, J1, Q10, Q15, Q16, Q17, Q18, Q27, Q28, Q29, Q3, Q30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

Commit message: Kicad Footprints
Parts:
- C10, C11, C12, C15, C16, C2, C3, C5, C6, C9: footprint (none) -> Capacitor_SMD:C_0805_2012Metric
- D1: footprint Diode_THT:D_DO-41_SOD81_P10.16mm_Horizontal -> (none)
- FL1: footprint (none) -> Aktive_Bal_Footprints:common mode choke foot
- J3: footprint A-DF_09_A_KG-T4S:ASSMANN_A-DF_09_A_KG-T4S -> Aktive_Bal_Footprints:ASSMANN_A-DF_09_A_KG-T4S
- Q10, Q11, Q12, Q13, Q14, Q15, Q16, Q17, Q18, Q19, Q20, Q21, Q22, Q23, Q24, Q25, Q26, Q27, Q28, Q29, Q3, Q30, Q31, Q32, Q33, Q34, Q4, Q5, Q6, Q7, Q8, Q9: footprint (none) -> Aktive_Bal_Footprints:8-WDFN
- R10, R11, R12, R13, R14, R15, R16, R17, R18, R19, R2, R20, R21, R22, R23, R24, R25, R26, R27, R28, R29, R3, R30, R31, R32, R33, R34, R35, R36, R37, R38, R39, R4, R40, R41, R42, R43, R44, R45, R46, R47, R48, R49, R5, R50, R51, R52, R55, R56, R57, R58, R59, R6, R60, R61, R62, R63, R64, R65, R66, R67, R68, R69, R7, R70, R71, R72, R73, R74, R75, R76, R77, R78, R79, R8, R80, R81, R82, R83, R84, R85, R86, R9: footprint (none) -> Resistor_SMD:R_0805_2012Metric
- R54: footprint (none) -> Aktive_Bal_Footprints:CMP-R100-1.0
- U13: footprint TO-220AB_ONS -> (none)
- U14: footprint DB24 -> Package_SO:SSOP-24_5.3x8.2mm_P0.65mm
