File: Aktive_Balancing/KiCAD/Aktive_Bal/Aktive_Bal.kicad_sch (KiCad schematic)
At the start: 59 parts, among them J16 Conn_01x02_Pin, J17 Conn_01x02_Pin, J18 Conn_01x02_Pin, J19 Conn_01x02_Pin, J2 Sockel_BluePill, J20 Conn_01x02_Pin, J21 Conn_01x02_Pin, J3 A-DF_09_A_KG-T4S, J4 Screw_Terminal_01x02, J9 Conn_01x01_Pin, U1 SCW20C-12, U13 RFP12N10L, U14 PCF8575CDB, U15 SN65HVD233, U2 EC1SA16N, U5 ADUM1250ARZ-RL7, U6 PCA9306DC, U7 LM1117IMPX_3_3_NOPB, U8 MCP4725xxx-xCH

Commit message: kicad
Parts:
- removed C5: 4.7µ, Capacitor_SMD:C_0805_2012Metric, symbol Device:C_Small
- removed C6, C7: 10µ, Capacitor_SMD:C_0805_2012Metric, symbol Device:C_Small
- added C17: 4.7µ, symbol Device:C_Polarized_Small
- added C36, C37: 10µ, symbol Device:C_Polarized_Small
- C11, C13, C25: footprint (none) -> Capacitor_SMD:C_0805_2012Metric
- C21: value 10µ -> 10µ tantal
- U13: footprint Aktive_Bal_Footprints:TO-220AB_ONS -> (none)
Connections:
- net +12V: now also C17.1
- net +5V: now also C37.1
- net -5V: now also C36.2
- net GND_float2: now also C17.2, C36.1, C37.2
- net SCLµC: no longer J2.14 (B6), J21.2 (Pin_2)
- net SDAµC: no longer J2.15 (B7), J21.1 (Pin_1)
- net SDA5: now reaches J19.1 (Pin_1), R3.1, U14.23 (SDA), U5.7 (SDA2), U6.5 (SDA2)
- net SDA5: now also JP4.1 (A); no longer JP5.1 (A)
- net SCL5: now reaches J19.2 (Pin_2), R4.1, U14.22 (SCL), U5.6 (SCL2), U6.6 (SCL2)
- net SCL5: now also JP5.1 (A); no longer JP4.1 (A)
- net SCL3.3: now reaches J20.2 (Pin_2), R6.1, U6.3 (SCL1), U8.5 (SCL)
- net SCL3.3: now also JP5.2 (B); no longer JP4.2 (B)
- net at J2.9 (A12): no longer U15.1 (D)
- net at J2.8 (A11): no longer U15.4 (R)
- net CANL: now reaches J3.2, R9.1, U15.6 (CANL)
- net CANH: now reaches J3.7, JP3.2 (B), U15.7 (CANH)
- net SDA3.3: now reaches J20.1 (Pin_1), R7.1, U6.4 (SDA1), U8.4 (SDA)
- net SDA3.3: now also JP4.2 (B); no longer JP5.2 (B)
- new net D: U15.1 (D)
- new net R: U15.4 (R)
Other:
- note added: "adresse"
- moved on the sheet: C16, C18, C19, C20, C21, C22, C23, C24, C25, C26, J16, J2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

Commit message: kicad
Parts:
- removed C11, C13: 0.1µ, Capacitor_SMD:C_0805_2012Metric, symbol Device:C
- removed C17: 4.7µ, symbol Device:C_Polarized_Small
- removed C8, C9: 0.1µ, Capacitor_SMD:C_0805_2012Metric, symbol Device:C_Small
- added C11, C13: 0.1µ, Capacitor_SMD:C_0805_2012Metric, symbol Device:C_Small
- added C17: 4.7µ, Capacitor_SMD:C_0805_2012Metric, symbol Device:C_Small
- added C38: 47µ, symbol Device:C_Polarized_Small
- added J1: Conn_01x01_Pin, symbol Connector:Conn_01x01_Pin
- added J22: Conn_01x02_Pin, symbol Connector:Conn_01x02_Pin
Connections:
- net +12V: now also J17.2 (Pin_2), C17.1, C38.1
- net +3.3V: now also C13.1
- net +5V: now also C11.1
- net GND_float2: now also C11.2, C13.2, C17.2, C38.2; no longer J17.2 (Pin_2)
- net I_Bal_Soll: now also J1.1 (Pin_1)
- net SCL5: now also J22.2 (Pin_2)
- net SDA5: now also J22.1 (Pin_1)
Other:
- moved on the sheet: C10, C12, J9

Commit message: layout
Parts:
- removed J16: Conn_01x02_Pin, symbol Connector:Conn_01x02_Pin
- C36, C37: footprint (none) -> Capacitor_SMD:CP_Elec_4x5.4
- C38: footprint (none) -> Capacitor_SMD:CP_Elec_6.3x5.7
- J1: footprint (none) -> Connector_PinHeader_2.54mm:PinHeader_1x01_P2.54mm_Vertical
- J17, J18, J19, J20, J21, J22: footprint (none) -> Connector_PinHeader_2.54mm:PinHeader_1x02_P2.54mm_Vertical
- JP6: footprint (none) -> Connector_PinHeader_2.54mm:PinHeader_1x03_P2.54mm_Vertical
- U13: footprint (none) -> Aktive_Bal_Footprints:TO-220AB_ONS
Other:
- moved on the sheet: C2
Changed lines of the file:
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@@
 	)
 	(junction
-		(at 60.96 168.91)
+		(at 115.57 38.1)
 		(diameter 0)
 		(color 0 0 0 0)
 	)
 	(junction
-		(at 104.14 33.02)
+		(at 60.96 168.91)
 		(diameter 0)
 		(color 0 0 0 0)
@@
 	)
 	(junction
-		(at 115.57 38.1)
-		(diameter 0)
-		(color 0 0 0 0)
-	)
-	(junction
 		(at 298.45 123.19)
 		(diameter 0)
@@
 	)
 	(junction
-		(at 114.3 33.02)
-		(diameter 0)
-		(color 0 0 0 0)
-	)
-	(junction
-		(at 104.14 38.1)
+		(at 115.57 33.02)
 		(diameter 0)
 		(color 0 0 0 0)
@@
 	(wire
 		(pts
+			(xy 115.57 33.02) (xy 121.92 33.02)
+		)
+		(stroke
+			(width 0)
+			(type default)
+		)
+	)
+	(wire
+		(pts
 			(xy 49.53 96.52) (xy 73.66 96.52)
 		)
@@
 	(wire
 		(pts
+			(xy 115.57 38.1) (xy 121.92 38.1)
+		)
+		(stroke
+			(width 0)
+			(type default)
+		)
+	)
+	(wire
+		(pts
 			(xy 158.75 30.48) (xy 172.72 30.48)
 		)
@@
 	(wire
 		(pts
-			(xy 104.14 33.02) (xy 114.3 33.02)
-		)
-		(stroke
-			(width 0)
-			(type default)
-		)
-	)
-	(wire
-		(pts
 			(xy 185.42 87.63) (xy 186.69 87.63)
 		)
@@
 	(wire
 		(pts
-			(xy 95.25 33.02) (xy 104.14 33.02)
+			(xy 95.25 33.02) (xy 115.57 33.02)
 		)
 		(stroke
@@
 	(wire
 		(pts
-			(xy 114.3 33.02) (xy 114.3 52.07)
-		)
-		(stroke
-			(width 0)
-			(type default)
-		)
-	)
-	(wire
-		(pts
 			(xy 172.72 100.33) (xy 172.72 107.95)
 		)
@@
 	(wire
 		(pts
-			(xy 114.3 33.02) (xy 121.92 33.02)
-		)
-		(stroke
-			(width 0)
-			(type default)
-		)
-	)
-	(wire
-		(pts
 			(xy 95.25 38.1) (xy 115.57 38.1)
 		)
@@
 	(wire
 		(pts
-			(xy 115.57 52.07) (xy 115.57 38.1)
-		)
-		(stroke
-			(width 0)
-			(type default)
-		)
-	)
-	(wire
-		(pts
 			(xy 195.58 85.09) (xy 201.93 85.09)
 		)
@@
 	(wire
 		(pts
-			(xy 116.84 52.07) (xy 115.57 52.07)
-		)
-		(stroke
-			(width 0)
-			(type default)
-		)
-	)
-	(wire
-		(pts
 			(xy 185.42 85.09) (xy 195.58 85.09)
 		)
@@
 	(wire
 		(pts
-			(xy 115.57 38.1) (xy 121.92 38.1)
-		)
-		(stroke
-			(width 0)
-			(type default)
-		)
-	)
-	(wire
-		(pts
 			(xy 64.77 88.9) (xy 64.77 93.98)
 		)
@@
 			)
 		)
-		(property "Footprint" ""
+		(property "Footprint" "Connector_PinHeader_2.54mm:PinHeader_1x01_P2.54mm_Vertical"
 			(at 311.15 127 0)
 			(hide yes)
@@
 			)
 		)
-		(property "Footprint" ""
+		(property "Footprint" "Connector_PinHeader_2.54mm:PinHeader_1x02_P2.54mm_Vertical"
 			(at 236.22 20.32 0)
 			(hide yes)
@@
 			)
 		)
-		(property "Footprint" ""
+		(property "Footprint" "Capacitor_SMD:CP_Elec_4x5.4"
 			(at 204.47 35.56 0)
 			(hide yes)
@@
 			)
 		)
-		(property "Footprint" ""
+		(property "Footprint" "Connector_PinHeader_2.54mm:PinHeader_1x03_P2.54mm_Vertical"
 			(at 298.45 88.9 0)
 			(hide yes)
@@
 	(symbol
 		(lib_id "Device:C_Small")
-		(at 104.14 35.56 0)
+		(at 115.57 35.56 0)
 		(unit 1)
 		(body_style 1)
@@
 		(fields_autoplaced yes)
 		(property "Reference" "C2"
-			(at 106.68 34.2962 0)
+			(at 118.11 34.2962 0)
 			(show_name no)
 			(do_not_autoplace no)
@@
 		)
 		(property "Value" "2.2µ"
-			(at 106.68 36.8362 0)
+			(at 118.11 36.8362 0)
 			(show_name no)
 			(do_not_autoplace no)
@@
 		)
 		(property "Footprint" "Capacitor_SMD:C_0805_2012Metric"
-			(at 104.14 35.56 0)
+			(at 115.57 35.56 0)
 			(hide yes)
 			(show_name no)
@@
 		)
 		(property "Datasheet" ""
-			(at 104.14 35.56 0)
+			(at 115.57 35.56 0)
 			(hide yes)
 			(show_name no)
@@
 		)
 		(property "Description" "Unpolarized capacitor, small symbol"
-			(at 104.14 35.56 0)
+			(at 115.57 35.56 0)
 			(hide yes)
 			(show_name no)
@@
 			)
 		)
-		(property "Footprint" ""
+		(property "Footprint" "Aktive_Bal_Footprints:TO-220AB_ONS"
 			(at 43.688 26.162 0)
 			(hide yes)
@@
 			)
 		)
-		(property "Footprint" ""
+		(property "Footprint" "Connector_PinHeader_2.54mm:PinHeader_1x02_P2.54mm_Vertical"
 			(at 158.75 78.74 0)
 			(hide yes)
@@
 			)
 		)
-		(property "Footprint" ""
+		(property "Footprint" "Connector_PinHeader_2.54mm:PinHeader_1x02_P2.54mm_Vertical"
 			(at 123.19 102.87 0)
 			(hide yes)
@@
 			)
 		)
-		(property "Footprint" ""
+		(property "Footprint" "Connector_PinHeader_2.54mm:PinHeader_1x02_P2.54mm_Vertical"
 			(at 170.18 48.26 0)
 			(hide yes)
@@
 			)
 		)
-		(property "Footprint" ""
+		(property "Footprint" "Capacitor_SMD:CP_Elec_4x5.4"
 			(at 204.47 30.48 0)
 			(hide yes)
@@
 	)
 	(symbol
-		(lib_id "Connector:Conn_01x02_Pin")
-		(at 114.3 57.15 90)
-		(unit 1)
-		(body_style 1)
-		(exclude_from_sim no)
-		(in_bom yes)
-		(on_board yes)
-		(in_pos_files yes)
-		(dnp no)
-		(fields_autoplaced yes)
-		(property "Reference" "J16"
-			(at 118.11 55.2449 90)
-			(show_name no)
-			(do_not_autoplace no)
-			(effects
-				(font
-					(size 1.27 1.27)
-				)
-				(justify right)
-			)
-		)
-		(property "Value" "Conn_01x02_Pin"
-			(at 118.11 57.7849 90)
-			(show_name no)
-			(do_not_autoplace no)
-			(effects
-				(font
-					(size 1.27 1.27)
-				)
-				(justify right)
-			)
-		)
-		(property "Footprint" ""
-			(at 114.3 57.15 0)
-			(hide yes)
-			(show_name no)
-			(do_not_autoplace no)
-			(effects
-				(font
-					(size 1.27 1.27)
-				)
-			)
-		)
-		(property "Datasheet" ""
-			(at 114.3 57.15 0)
-			(hide yes)
-			(show_name no)
-			(do_not_autoplace no)
-			(effects
-				(font
-					(size 1.27 1.27)
-				)
-			)
-		)
-		(property "Description" "Generic connector, single row, 01x02, script generated"
-			(at 114.3 57.15 0)
-			(hide yes)
-			(show_name no)
-			(do_not_autoplace no)
-			(effects
-				(font
-					(size 1.27 1.27)
-				)
-			)
-		)
-		(pin "1"
-		)
-		(pin "2"
-		)
-		(instances
-			(project "Aktive_Bal"
-				(path "/7c40c112-cd2b-4a48-9744-14a65613b3b5"
-					(reference "J16")
-					(unit 1)
-				)
-			)
-		)
-	)
-	(symbol
 		(lib_id "Jumper:Jumper_2_Open")
 		(at 87.63 134.62 270)
@@
 			)
 		)
-		(property "Footprint" ""
+		(property "Footprint" "Connector_PinHeader_2.54mm:PinHeader_1x02_P2.54mm_Vertical"
 			(at 105.41 177.8 0)
 			(hide yes)
@@
 			)
 		)
-		(property "Footprint" ""
+		(property "Footprint" "Connector_PinHeader_2.54mm:PinHeader_1x02_P2.54mm_Vertical"
 			(at 201.93 78.74 0)
 			(hide yes)
@@
 			)
 		)
-		(property "Footprint" ""
+		(property "Footprint" "Capacitor_SMD:CP_Elec_6.3x5.7"
 			(at 158.75 33.02 0)
 			(hide yes)

Commit message: layout
Parts:
- added R2: 100k, Resistor_SMD:R_0805_2012Metric, symbol Device:R
- C7: renamed from C25; value 10µ -> 0.1µ
- renumbered C23 to C1, C38 to C10, C16 to C11, C17 to C12, C19 to C13, C18 to C14, C36 to C15, C37 to C16, C10 to C17, C11 to C18, C26 to C19, C24 to C2, C13 to C20, C12 to C21, C21 to C23, C20 to C24, C14 to C3, C1 to C4, C15 to C5, C2 to C6, C3 to C8, C4 to C9, J4 to J1, J9 to J10, J1 to J11, J3 to J2, J21 to J3, J19 to J4, J2 to J5, J22 to J6, J17 to J7, J20 to J8, J18 to J9, JP3 to JP1, JP4 to JP2, JP5 to JP3, JP6 to JP4, R25 to R1, R7 to R10, R8 to R11, R1 to R3, R2 to R4, R9 to R5, R3 to R6, R4 to R7, R5 to R8, R6 to R9, U13 to U1, U15 to U2, U5 to U3, U1 to U4, U6 to U5, U2 to U6, U14 to U7, U7 to U8, U8 to U9
Connections:
- net Bat_GND: now also R2.2
- net enable: now also R2.1
Other:
- moved on the sheet: C19, J1
