File: Aktive_Balancing/KiCAD/Aktive_Bal/Aktive_Bal.kicad_sch (KiCad schematic)
At the start: 67 parts, among them J1 Screw_Terminal_01x02, J10 Conn_01x02_Pin, J11 Conn_01x02_Pin, J12 Conn_01x02_Pin, J13 Conn_01x02_Pin, J14 Conn_01x02_Pin, J2 A-DF_09_A_KG-T4S, J3 Conn_01x02_Pin, J4 Conn_01x02_Pin, J5 Conn_01x02_Pin, J6 Conn_01x02_Pin, J7 Sockel_BluePill, J8 Conn_01x02_Pin, J9 Conn_01x02_Pin, U1 RFP12N10L, U2 ADUM1250ARZ-RL7, U3 SN65HVD233, U4 SCW20C-12, U5 EC1SA16N, U6 PCA9306DC, U7 PCF8575CDB, U8 LM1117MP-3.3, U9 MCP4725xxx-xCH

Commit message: Bisschen sortiert und so
Parts:
- removed J8: Conn_01x02_Pin, Connector_PinHeader_2.54mm:PinHeader_1x02_P2.54mm_Vertical, symbol Connector:Conn_01x02_Pin
Changed lines of the file:
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@@
 	)
 	(junction
-		(at 121.92 177.8)
-		(diameter 0)
-		(color 0 0 0 0)
-	)
-	(junction
 		(at 205.74 91.44)
 		(diameter 0)
@@
 	)
 	(junction
+		(at 121.92 177.8)
+		(diameter 0)
+		(color 0 0 0 0)
+	)
+	(junction
 		(at 64.77 38.1)
 		(diameter 0)
@@
 	)
 	(junction
-		(at 168.91 91.44)
-		(diameter 0)
-		(color 0 0 0 0)
-	)
-	(junction
 		(at 213.36 177.8)
 		(diameter 0)
@@
 	)
 	(junction
-		(at 124.46 175.26)
-		(diameter 0)
-		(color 0 0 0 0)
-	)
-	(junction
 		(at 31.75 76.2)
 		(diameter 0)
@@
 	)
 	(junction
-		(at 166.37 93.98)
+		(at 124.46 175.26)
 		(diameter 0)
 		(color 0 0 0 0)
@@
 	(wire
 		(pts
-			(xy 124.46 175.26) (xy 130.81 175.26)
-		)
-		(stroke
-			(width 0)
-			(type default)
-		)
-	)
-	(wire
-		(pts
 			(xy 115.57 33.02) (xy 121.92 33.02)
 		)
@@
 	(wire
 		(pts
-			(xy 114.3 175.26) (xy 124.46 175.26)
-		)
-		(stroke
-			(width 0)
-			(type default)
-		)
-	)
-	(wire
-		(pts
-			(xy 168.91 90.17) (xy 168.91 91.44)
-		)
-		(stroke
-			(width 0)
-			(type default)
-		)
-	)
-	(wire
-		(pts
 			(xy 53.34 90.17) (xy 55.88 90.17)
 		)
@@
 	(wire
 		(pts
-			(xy 121.92 177.8) (xy 130.81 177.8)
-		)
-		(stroke
-			(width 0)
-			(type default)
-		)
-	)
-	(wire
-		(pts
 			(xy 195.58 93.98) (xy 196.85 93.98)
 		)
@@
 	(wire
 		(pts
-			(xy 166.37 90.17) (xy 166.37 93.98)
-		)
-		(stroke
-			(width 0)
-			(type default)
-		)
-	)
-	(wire
-		(pts
 			(xy 256.54 149.86) (xy 259.08 149.86)
 		)
@@
 	(wire
 		(pts
+			(xy 49.53 92.71) (xy 55.88 92.71)
+		)
+		(stroke
+			(width 0)
+			(type default)
+		)
+	)
+	(wire
+		(pts
 			(xy 175.26 96.52) (xy 173.99 96.52)
 		)
@@
 	(wire
 		(pts
+			(xy 123.19 175.26) (xy 123.19 173.99)
+		)
+		(stroke
+			(width 0)
+			(type default)
+		)
+	)
+	(wire
+		(pts
 			(xy 114.3 90.17) (xy 118.11 90.17)
 		)
@@
 	(wire
 		(pts
+			(xy 163.83 91.44) (xy 175.26 91.44)
+		)
+		(stroke
+			(width 0)
+			(type default)
+		)
+	)
+	(wire
+		(pts
 			(xy 260.35 147.32) (xy 256.54 147.32)
 		)
@@
 	(wire
 		(pts
-			(xy 168.91 91.44) (xy 175.26 91.44)
-		)
-		(stroke
-			(width 0)
-			(type default)
-		)
-	)
-	(wire
-		(pts
-			(xy 49.53 92.71) (xy 55.88 92.71)
-		)
-		(stroke
-			(width 0)
-			(type default)
-		)
-	)
-	(wire
-		(pts
 			(xy 256.54 152.4) (xy 245.11 152.4)
 		)
@@
 	(wire
 		(pts
-			(xy 163.83 93.98) (xy 166.37 93.98)
-		)
-		(stroke
-			(width 0)
-			(type default)
-		)
-	)
-	(wire
-		(pts
-			(xy 124.46 175.26) (xy 124.46 179.07)
+			(xy 76.2 33.02) (xy 85.09 33.02)
 		)
 		(stroke
@@
 	(wire
 		(pts
-			(xy 76.2 33.02) (xy 85.09 33.02)
+			(xy 298.45 105.41) (xy 298.45 106.68)
 		)
 		(stroke
@@
 	(wire
 		(pts
-			(xy 298.45 105.41) (xy 298.45 106.68)
+			(xy 283.21 123.19) (xy 267.97 123.19)
 		)
 		(stroke
@@
 	(wire
 		(pts
-			(xy 283.21 123.19) (xy 267.97 123.19)
+			(xy 124.46 175.26) (xy 124.46 179.07)
 		)
 		(stroke
@@
 	(wire
 		(pts
+			(xy 130.81 175.26) (xy 124.46 175.26)
+		)
+		(stroke
+			(width 0)
+			(type default)
+		)
+	)
+	(wire
+		(pts
 			(xy 121.92 38.1) (xy 121.92 43.18)
 		)
@@
 	(wire
 		(pts
+			(xy 121.92 177.8) (xy 130.81 177.8)
+		)
+		(stroke
+			(width 0)
+			(type default)
+		)
+	)
+	(wire
+		(pts
 			(xy 256.54 157.48) (xy 245.11 157.48)
 		)
@@
 	(wire
 		(pts
-			(xy 40.64 33.02) (xy 45.72 33.02)
+			(xy 123.19 173.99) (xy 114.3 173.99)
 		)
 		(stroke
@@
 	(wire
 		(pts
-			(xy 177.8 35.56) (xy 177.8 33.02)
+			(xy 40.64 33.02) (xy 45.72 33.02)
 		)
 		(stroke
@@
 	(wire
 		(pts
-			(xy 208.28 33.02) (xy 217.17 33.02)
+			(xy 177.8 35.56) (xy 177.8 33.02)
 		)
 		(stroke
@@
 	(wire
 		(pts
-			(xy 252.73 38.1) (xy 254 38.1)
+			(xy 208.28 33.02) (xy 217.17 33.02)
 		)
 		(stroke
@@
 	(wire
 		(pts
-			(xy 163.83 91.44) (xy 168.91 91.44)
+			(xy 252.73 38.1) (xy 254 38.1)
 		)
 		(stroke
@@
 	(wire
 		(pts
+			(xy 124.46 175.26) (xy 123.19 175.26)
+		)
+		(stroke
+			(width 0)
+			(type default)
+		)
+	)
+	(wire
+		(pts
 			(xy 195.58 91.44) (xy 205.74 91.44)
 		)
@@
 	(wire
 		(pts
-			(xy 166.37 93.98) (xy 175.26 93.98)
+			(xy 163.83 93.98) (xy 175.26 93.98)
 		)
 		(stroke
@@
 	(global_label "SCLµC"
 		(shape output)
-		(at 114.3 175.26 180)
+		(at 114.3 173.99 180)
 		(fields_autoplaced yes)
 		(effects
@@
 		)
 		(property "Intersheetrefs" "${INTERSHEET_REFS}"
-			(at 105.2067 175.26 0)
+			(at 105.2067 173.99 0)
 			(hide yes)
 			(show_name no)
@@
 		(length 2.54)
 		(shape round)
-		(at 27.3252 95.25 0)
+		(at 27.94 95.25 180)
 		(fields_autoplaced yes)
 		(effects
@@
 				(size 1.27 1.27)
 			)
-			(justify left bottom)
+			(justify right bottom)
 		)
 		(property "Netzklasse" "signal"
-			(at 28.0237 92.71 0)
+			(at 28.6385 97.79 0)
 			(show_name no)
 			(do_not_autoplace no)
@@
 		)
 		(property "Component Class" ""
-			(at -28.5548 1.27 0)
+			(at -27.94 1.27 0)
 			(show_name no)
 			(do_not_autoplace no)
@@
 		(length 2.54)
 		(shape round)
-		(at 26.67 91.44 0)
+		(at 33.02 91.44 0)
 		(fields_autoplaced yes)
 		(effects
@@
 		)
 		(property "Netzklasse" "signal"
-			(at 27.3685 88.9 0)
+			(at 33.7185 88.9 0)
 			(show_name no)
 			(do_not_autoplace no)
@@
 		)
 		(property "Component Class" ""
-			(at -271.78 -3.81 0)
+			(at -265.43 -3.81 0)
 			(show_name no)
 			(do_not_autoplace no)
@@
 					(unit 1)
 				)
-			)
-		)
-	)
-	(symbol
-		(lib_id "Connector:Conn_01x02_Pin")
-		(at 168.91 85.09 270)
-		(unit 1)
-		(body_style 1)
-		(exclude_from_sim no)
-		(in_bom yes)
-		(on_board yes)
-		(in_pos_files yes)
-		(dnp no)
-		(fields_autoplaced yes)
-		(property "Reference" "J8"
-			(at 167.64 80.01 90)
-			(show_name no)
-			(do_not_autoplace no)
-			(effects
-				(font
-					(size 1.27 1.27)
-				)
-			)
-		)
-		(property "Value" "Conn_01x02_Pin"
-			(at 167.64 82.55 90)
-			(show_name no)
-			(do_not_autoplace no)
-			(effects
-				(font
-					(size 1.27 1.27)
-				)
-			)
-		)
-		(property "Footprint" "Connector_PinHeader_2.54mm:PinHeader_1x02_P2.54mm_Vertical"
-			(at 168.91 85.09 0)
-			(hide yes)
-			(show_name no)
-			(do_not_autoplace no)
-			(effects
-				(font
-					(size 1.27 1.27)
-				)
-			)
-		)
-		(property "Datasheet" ""
-			(at 168.91 85.09 0)
-			(hide yes)
-			(show_name no)
-			(do_not_autoplace no)
-			(effects
-				(font
-					(size 1.27 1.27)
-				)
-			)
-		)
-		(property "Description" "Generic connector, single row, 01x02, script generated"
-			(at 168.91 85.09 0)
-			(hide yes)
-			(show_name no)
-			(do_not_autoplace no)
-			(effects
-				(font
-					(size 1.27 1.27)
-				)
-			)
-		)
-		(pin "1"
-		)
-		(pin "2"
-		)
-		(instances
-			(project "Aktive_Bal"
-				(path "/7c40c112-cd2b-4a48-9744-14a65613b3b5"
-					(reference "J8")
-					(unit 1)
-				)
