File: Aktive_Balancing/KiCAD/Aktive_Bal/controller.kicad_sch (KiCad schematic)
At the start: 22 parts, among them Q1 BSS316NH6327XTSA1, U3 LM2596S-ADJ, U4 TL084

Commit message: kicad
Parts:
- added C22, C24: 0.1µ, symbol Device:C
Connections:
- net +5V: now also C24.1; no longer U4.4 (V+)
- net -5V: now also C22.2; no longer U4.11 (V-)
- new net: C22.1, U4.11 (V-)
- new net: C24.2, U4.4 (V+)
Changed lines of the file:
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@@
 	(symbol
 		(lib_id "power:+5V")
-		(at 54.61 77.47 0)
+		(at 54.61 69.85 0)
 		(unit 1)
 		(body_style 1)
@@
 		(dnp no)
 		(property "Reference" "#PWR030"
-			(at 54.61 81.28 0)
+			(at 54.61 73.66 0)
 			(hide yes)
 			(show_name no)
@@
 		)
 		(property "Value" "+5V"
-			(at 56.896 76.454 0)
+			(at 56.896 68.834 0)
 			(show_name no)
 			(do_not_autoplace no)
@@
 		)
 		(property "Footprint" ""
-			(at 54.61 77.47 0)
-			(hide yes)
-			(show_name no)
-			(do_not_autoplace no)
-			(effects
-				(font
-					(size 1.27 1.27)
-				)
-			)
-		)
-		(property "Datasheet" ""
-			(at 54.61 77.47 0)
+			(at 54.61 69.85 0)
+			(hide yes)
+			(show_name no)
+			(do_not_autoplace no)
+			(effects
+				(font
+					(size 1.27 1.27)
+				)
+			)
+		)
+		(property "Datasheet" ""
+			(at 54.61 69.85 0)
 			(hide yes)
 			(show_name no)
@@
 		)
 		(property "Description" "Power symbol creates a global label with name \"+5V\""
-			(at 54.61 77.47 0)
+			(at 54.61 69.85 0)
 			(hide yes)
 			(show_name no)
@@
 	(symbol
 		(lib_id "power:-5V")
-		(at 54.61 92.71 180)
+		(at 54.61 100.33 180)
 		(unit 1)
 		(body_style 1)
@@
 		(dnp no)
 		(property "Reference" "#PWR029"
-			(at 54.61 88.9 0)
+			(at 54.61 96.52 0)
 			(hide yes)
 			(show_name no)
@@
 		)
 		(property "Value" "-5V"
-			(at 57.15 92.964 0)
+			(at 57.15 100.584 0)
 			(show_name no)
 			(do_not_autoplace no)
@@
 		)
 		(property "Footprint" ""
-			(at 54.61 92.71 0)
-			(hide yes)
-			(show_name no)
-			(do_not_autoplace no)
-			(effects
-				(font
-					(size 1.27 1.27)
-				)
-			)
-		)
-		(property "Datasheet" ""
-			(at 54.61 92.71 0)
+			(at 54.61 100.33 0)
+			(hide yes)
+			(show_name no)
+			(do_not_autoplace no)
+			(effects
+				(font
+					(size 1.27 1.27)
+				)
+			)
+		)
+		(property "Datasheet" ""
+			(at 54.61 100.33 0)
 			(hide yes)
 			(show_name no)
@@
 		)
 		(property "Description" "Power symbol creates a global label with name \"-5V\""
-			(at 54.61 92.71 0)
+			(at 54.61 100.33 0)
 			(hide yes)
 			(show_name no)
@@
 	)
 	(symbol
+		(lib_id "Device:C")
+		(at 54.61 73.66 0)
+		(unit 1)
+		(body_style 1)
+		(exclude_from_sim no)
+		(in_bom yes)
+		(on_board yes)
+		(in_pos_files yes)
+		(dnp no)
+		(fields_autoplaced yes)
+		(property "Reference" "C24"
+			(at 58.42 72.3899 0)
+			(show_name no)
+			(do_not_autoplace no)
+			(effects
+				(font
+					(size 1.27 1.27)
+				)
+				(justify left)
+			)
+		)
+		(property "Value" "0.1µ"
+			(at 58.42 74.9299 0)
+			(show_name no)
+			(do_not_autoplace no)
+			(effects
+				(font
+					(size 1.27 1.27)
+				)
+				(justify left)
+			)
+		)
+		(property "Footprint" ""
+			(at 55.5752 77.47 0)
+			(hide yes)
+			(show_name no)
+			(do_not_autoplace no)
+			(effects
+				(font
+					(size 1.27 1.27)
+				)
+			)
+		)
+		(property "Datasheet" ""
+			(at 54.61 73.66 0)
+			(hide yes)
+			(show_name no)
+			(do_not_autoplace no)
+			(effects
+				(font
+					(size 1.27 1.27)
+				)
+			)
+		)
+		(property "Description" "Unpolarized capacitor"
+			(at 54.61 73.66 0)
+			(hide yes)
+			(show_name no)
+			(do_not_autoplace no)
+			(effects
+				(font
+					(size 1.27 1.27)
+				)
+			)
+		)
+		(pin "2"
+		)
+		(pin "1"
+		)
+		(instances
+			(project "Aktive_Bal"
+				(path "/7c40c112-cd2b-4a48-9744-14a65613b3b5/7022d0de-596a-4fda-81a7-762d98787f96"
+					(reference "C24")
+					(unit 1)
+				)
+			)
+		)
+	)
+	(symbol
 		(lib_id "Device:R")
 		(at 96.52 97.79 0)
@@
 					(unit 1)
 				)
+			)
+		)
+	)
+	(symbol
+		(lib_id "Device:C")
+		(at 54.61 96.52 0)
+		(unit 1)
+		(body_style 1)
+		(exclude_from_sim no)
+		(in_bom yes)
+		(on_board yes)
+		(in_pos_files yes)
+		(dnp no)
+		(fields_autoplaced yes)
+		(property "Reference" "C22"
+			(at 58.42 95.2499 0)
+			(show_name no)
+			(do_not_autoplace no)
+			(effects
+				(font
+					(size 1.27 1.27)
+				)
+				(justify left)
+			)
+		)
+		(property "Value" "0.1µ"
+			(at 58.42 97.7899 0)
+			(show_name no)
+			(do_not_autoplace no)
+			(effects
+				(font
+					(size 1.27 1.27)
+				)
+				(justify left)
+			)
+		)
+		(property "Footprint" ""
+			(at 55.5752 100.33 0)
+			(hide yes)
+			(show_name no)
+			(do_not_autoplace no)
+			(effects
+				(font
+					(size 1.27 1.27)
+				)
+			)
+		)
+		(property "Datasheet" ""
+			(at 54.61 96.52 0)
+			(hide yes)
+			(show_name no)
+			(do_not_autoplace no)
+			(effects
+				(font
+					(size 1.27 1.27)
+				)
+			)
+		)
+		(property "Description" "Unpolarized capacitor"
+			(at 54.61 96.52 0)
+			(hide yes)
+			(show_name no)
+			(do_not_autoplace no)
+			(effects
+				(font
+					(size 1.27 1.27)
+				)
+			)
+		)
+		(pin "2"
+		)
+		(pin "1"
+		)
+		(instances
+			(project "Aktive_Bal"
+				(path "/7c40c112-cd2b-4a48-9744-14a65613b3b5/7022d0de-596a-4fda-81a7-762d98787f96"
+					(reference "C22")
+					(unit 1)
+				)

Commit message: kicad
Parts:
- added C31: 0.1µ, symbol Device:C
Connections:
- net +12V: now also C31.2
- net +5V: now also C24.2, U4.4 (V+); no longer C24.1
- net -5V: now also U4.11 (V-)
- net GND_float2: now also C22.1, C24.1, C31.1
Other:
- moved on the sheet: C22, C24

Commit message: kicad bom
Parts:
- renumbered C24 to C27, C22 to C28, C15 to C29, C16 to C30, C17 to C32, C18 to C33, C19 to C34
Changed lines of the file:
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@@
 		(in_pos_files yes)
 		(dnp no)
-		(property "Reference" "C16"
+		(property "Reference" "C30"
 			(at 173.99 49.022 90)
 			(show_name no)
@@
 			(project "Aktive_Bal"
 				(path "/7c40c112-cd2b-4a48-9744-14a65613b3b5/7022d0de-596a-4fda-81a7-762d98787f96"
-					(reference "C16")
+					(reference "C30")
 					(unit 1)
 				)
@@
 		(in_pos_files yes)
 		(dnp no)
-		(property "Reference" "C15"
+		(property "Reference" "C29"
 			(at 91.44 61.722 90)
 			(show_name no)
@@
 			(project "Aktive_Bal"
 				(path "/7c40c112-cd2b-4a48-9744-14a65613b3b5/7022d0de-596a-4fda-81a7-762d98787f96"
-					(reference "C15")
+					(reference "C29")
 					(unit 1)
 				)
@@
 		(dnp no)
 		(fields_autoplaced yes)
-		(property "Reference" "C17"
+		(property "Reference" "C32"
 			(at 167.64 71.8438 0)
 			(show_name no)
@@
 			(project "Aktive_Bal"
 				(path "/7c40c112-cd2b-4a48-9744-14a65613b3b5/7022d0de-596a-4fda-81a7-762d98787f96"
-					(reference "C17")
+					(reference "C32")
 					(unit 1)
 				)
@@
 		(dnp no)
 		(fields_autoplaced yes)
-		(property "Reference" "C18"
+		(property "Reference" "C33"
 			(at 218.44 80.3909 0)
 			(show_name no)
@@
 			(project "Aktive_Bal"
 				(path "/7c40c112-cd2b-4a48-9744-14a65613b3b5/7022d0de-596a-4fda-81a7-762d98787f96"
-					(reference "C18")
+					(reference "C33")
 					(unit 1)
 				)
@@
 		(dnp no)
 		(fields_autoplaced yes)
-		(property "Reference" "C24"
+		(property "Reference" "C27"
 			(at 48.26 67.31 90)
 			(show_name no)
@@
 			(project "Aktive_Bal"
 				(path "/7c40c112-cd2b-4a48-9744-14a65613b3b5/7022d0de-596a-4fda-81a7-762d98787f96"
-					(reference "C24")
+					(reference "C27")
 					(unit 1)
 				)
@@
 		(dnp no)
 		(fields_autoplaced yes)
-		(property "Reference" "C22"
+		(property "Reference" "C28"
 			(at 50.8 87.63 90)
 			(show_name no)
@@
 			(project "Aktive_Bal"
 				(path "/7c40c112-cd2b-4a48-9744-14a65613b3b5/7022d0de-596a-4fda-81a7-762d98787f96"
-					(reference "C22")
+					(reference "C28")
 					(unit 1)
 				)
@@
 		(dnp no)
 		(fields_autoplaced yes)
-		(property "Reference" "C19"
+		(property "Reference" "C34"
 			(at 120.65 74.9362 0)
 			(show_name no)
@@
 			(project "Aktive_Bal"
 				(path "/7c40c112-cd2b-4a48-9744-14a65613b3b5/7022d0de-596a-4fda-81a7-762d98787f96"
-					(reference "C19")
-					(unit 1)
-				)
+					(reference "C34")
+					(unit 1)
+				)

Commit message: kicad
Parts:
- C27, C28, C31: footprint (none) -> Capacitor_SMD:C_0805_2012Metric
- R20: value 120k -> 90k
- R21: value 15k -> 10k
Changed lines of the file:
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@@
 		)
 	)
+	(netclass_flag ""
+		(length 2.54)
+		(shape round)
+		(at 214.63 66.04 90)
+		(fields_autoplaced yes)
+		(effects
+			(font
+				(size 1.27 1.27)
+			)
+			(justify left bottom)
+		)
+		(property "Netzklasse" "power"
+			(at 212.09 65.3415 90)
+			(show_name no)
+			(do_not_autoplace no)
+			(effects
+				(font
+					(size 1.27 1.27)
+				)
+				(justify left)
+			)
+		)
+		(property "Component Class" ""
+			(at -22.86 11.43 0)
+			(show_name no)
+			(do_not_autoplace no)
+			(effects
+				(font
+					(size 1.27 1.27)
+					(italic yes)
+				)
+			)
+		)
+	)
+	(netclass_flag ""
+		(length 2.54)
+		(shape diamond)
+		(at 156.21 97.79 0)
+		(fields_autoplaced yes)
+		(effects
+			(font
+				(size 1.27 1.27)
+			)
+			(justify left bottom)
+		)
+		(property "Netzklasse" "PowerGND"
+			(at 157.4165 95.25 0)
+			(show_name no)
+			(do_not_autoplace no)
+			(effects
+				(font
+					(size 1.27 1.27)
+				)
+				(justify left)
+			)
+		)
+		(property "Component Class" ""
+			(at -72.39 26.67 0)
+			(show_name no)
+			(do_not_autoplace no)
+			(effects
+				(font
+					(size 1.27 1.27)
+					(italic yes)
+				)
+			)
+		)
+	)
+	(netclass_flag ""
+		(length 2.54)
+		(shape round)
+		(at 203.2 73.66 0)
+		(fields_autoplaced yes)
+		(effects
+			(font
+				(size 1.27 1.27)
+			)
+			(justify left bottom)
+		)
+		(property "Netzklasse" "power"
+			(at 203.8985 71.12 0)
+			(show_name no)
+			(do_not_autoplace no)
+			(effects
+				(font
+					(size 1.27 1.27)
+				)
+				(justify left)
+			)
+		)
+		(property "Component Class" ""
+			(at -34.29 19.05 0)
+			(show_name no)
+			(do_not_autoplace no)
+			(effects
+				(font
+					(size 1.27 1.27)
+					(italic yes)
+				)
+			)
+		)
+	)
 	(symbol
 		(lib_id "power:GND")
@@
 			)
 		)
-		(property "Footprint" ""
+		(property "Footprint" "Capacitor_SMD:C_0805_2012Metric"
 			(at 172.4152 68.58 0)
 			(hide yes)
@@
 			)
 		)
-		(property "Footprint" ""
+		(property "Footprint" "Capacitor_SMD:C_0805_2012Metric"
 			(at 52.07 73.9648 0)
 			(hide yes)
@@
 			)
 		)
-		(property "Value" "120k"
+		(property "Value" "90k"
 			(at 99.06 99.0599 0)
 			(show_name no)
@@
 			)
 		)
-		(property "Footprint" ""
+		(property "Footprint" "Capacitor_SMD:C_0805_2012Metric"
 			(at 54.61 94.2848 0)
 			(hide yes)
@@
 			)
 		)
-		(property "Value" "15k"
+		(property "Value" "10k"
 			(at 99.06 109.2199 0)
 			(show_name no)

Commit message: kicad
Parts:
- added J5, J6: Conn_01x01_Pin, symbol Connector:Conn_01x01_Pin
- added L2: 10µ, Inductor_SMD:L_Bourns_SRR1260, symbol Device:L
Connections:
- net +12V: now also L2.1; no longer C31.2, C32.1, U3.1 (VIN)
- net I_Bal: now also J5.1 (Pin_1)
- net V_I_Bal: now also J6.1 (Pin_1)
- new net: C31.2, C32.1, L2.2, U3.1 (VIN)

Commit message: layout
Parts:
- J5, J6: footprint (none) -> Connector_PinHeader_2.54mm:PinHeader_1x01_P2.54mm_Vertical
Changed lines of the file:
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@@
 			)
 		)
-		(property "Footprint" ""
+		(property "Footprint" "Connector_PinHeader_2.54mm:PinHeader_1x01_P2.54mm_Vertical"
 			(at 130.81 81.28 0)
 			(hide yes)
@@
 			)
 		)
-		(property "Footprint" ""
+		(property "Footprint" "Connector_PinHeader_2.54mm:PinHeader_1x01_P2.54mm_Vertical"
 			(at 92.71 76.2 0)
 			(hide yes)

Commit message: layout
Parts:
- L1: renamed from L2; footprint Inductor_SMD:L_Bourns_SRR1260 -> Aktive_Bal_Footprints:NRS6045
- renumbered C27 to C25, C28 to C26, C29 to C27, C34 to C28, C32 to C29, C31 to C30, C30 to C31, C33 to C32, J5 to J18, J6 to J19, L1 to L2, R15 to R100, R19 to R101, R16 to R102, R17 to R103, R18 to R104, R10 to R93, R12 to R94, R11 to R95, R13 to R96, R14 to R97, R20 to R98, R21 to R99, U4 to U14, U3 to U15

Commit message: Schaltung Review + Layout
Schaltung Review + Layout
Parts:
- removed J18, J19: Conn_01x01_Pin, Connector_PinHeader_2.54mm:PinHeader_1x01_P2.54mm_Vertical, symbol Connector:Conn_01x01_Pin
- added J21, J22, J23, J24: Conn_01x02_Pin, Connector_PinHeader_2.54mm:PinHeader_1x02_P2.54mm_Vertical, symbol Connector:Conn_01x02_Pin
- renumbered C25 to C24, C26 to C25, C27 to C26, C28 to C27, C29 to C28, C30 to C29, C31 to C30, C32 to C31
Connections:
- net Bal: now also J24.1 (Pin_1)
- net GND_float2: now also J21.2 (Pin_2), J22.1 (Pin_1), J23.2 (Pin_2), J24.2 (Pin_2)
- net I_Bal: now also J21.1 (Pin_1)
- net V_I_Bal: now also J22.2 (Pin_2)
- net at C30.1, Q1.3 (D), R104.2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: now also J23.1 (Pin_1)
