File: Aktive_Balancing/KiCAD/Aktive_Bal/controller.kicad_sch (KiCad schematic)
At the start: 30 parts, among them J21 Conn_01x02_Pin, J22 Conn_01x02_Pin, J23 Conn_01x02_Pin, J24 Conn_01x02_Pin, Q1 BSS316NH6327XTSA1, U14 TL084, U15 LM2596S-ADJ

Commit message: Regelkreis sortiert
Parts:
- U15: footprint Package_TO_SOT_SMD:TO-263-5_TabPin3 -> Aktive_Bal_Footprints:LM2596_5T
Changed lines of the file:
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@@
 			)
 		)
-		(property "Footprint" "Package_TO_SOT_SMD:TO-263-5_TabPin3"
+		(property "Footprint" "Aktive_Bal_Footprints:LM2596_5T"
 			(at 191.77 77.47 0)
 			(hide yes)

Commit message: alles neu
Changed lines of the file:
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@@
+		(length 2.54)
+		(shape round)
+		(at 54.61 44.45 90)
+		(fields_autoplaced yes)
+		(effects
+			(font
+				(size 1.27 1.27)
+			)
+			(justify left bottom)
+		)
+		(property "Netzklasse" "analog"
+			(at 52.07 43.7515 90)
+			(show_name no)
+			(do_not_autoplace no)
+			(effects
+				(font
+					(size 1.27 1.27)
+				)
+				(justify left)
+			)
+		)
+		(property "Component Class" ""
+			(at -171.45 -11.43 0)
+			(show_name no)
+			(do_not_autoplace no)
+			(effects
+				(font
+					(size 1.27 1.27)
+					(italic yes)
+				)
+			)
+		)
+	)
+	(netclass_flag ""
+		(length 2.54)
+		(shape round)
+		(at 54.61 34.29 90)
+		(fields_autoplaced yes)
+		(effects
+			(font
+				(size 1.27 1.27)
+			)
+			(justify left bottom)
+		)
+		(property "Netzklasse" "power"
+			(at 52.07 33.5915 90)
+			(show_name no)
+			(do_not_autoplace no)
+			(effects
+				(font
+					(size 1.27 1.27)
+				)
+				(justify left)
+			)
+		)
+		(property "Component Class" ""
+			(at -125.73 -30.48 0)
+			(show_name no)
+			(do_not_autoplace no)
+			(effects
+				(font
+					(size 1.27 1.27)
+					(italic yes)
+				)
+			)
+		)
+	)
+	(netclass_flag ""
 		(length 2.54)
 		(shape round)
@@
 		(in_pos_files yes)
 		(dnp no)
-		(fields_autoplaced yes)
 		(property "Reference" "L1"
 			(at 158.75 74.9299 0)
@@
 					(size 1.27 1.27)
 				)
-				(justify right)
-			)
-		)
+				(justify left)
+			)
+		)

Commit message: review
Connections:
- net GNDShunt: now reaches R98.2, R99.1, U14.13 (-)
Other:
- note added: "Differenzspannung messen!!"
Changed lines of the file:
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@@
 	(generator_version "10.0")
 	(paper "A4")
+	(text "Differenzspannung messen!!"
+		(exclude_from_sim no)
+		(at 147.574 96.012 0)
+		(effects
+			(font
+				(size 1.27 1.27)
+			)
+		)
+	)
+	(junction
+		(at 119.38 91.44)
+		(diameter 0)
+		(color 0 0 0 0)
+	)
 	(junction
 		(at 83.82 48.26)
@@
 		(pts
 			(xy 203.2 57.15) (xy 203.2 68.58)
+		)
+		(stroke
+			(width 0)
+			(type default)
+		)
+	)
+	(wire
+		(pts
+			(xy 119.38 91.44) (xy 133.35 91.44)
 		)
 		(stroke
@@
 			(hide yes)
 			(show_name no)
+			(do_not_autoplace no)
+			(effects
+				(font
+					(size 1.27 1.27)
+				)
+				(justify left)
+			)
+		)
+	)
+	(global_label "GNDShunt"
+		(shape input)
+		(at 133.35 91.44 0)
+		(fields_autoplaced yes)
+		(effects
+			(font
+				(size 1.27 1.27)
+			)
+			(justify left)
+		)
+		(property "Intersheetrefs" "${INTERSHEET_REFS}"
+			(at 145.5879 91.44 0)
+			(hide yes)
+			(show_name no)

Commit message: Vorläufige finale Version
Diese Version soll in die Fertigung gehen.
Parts:
- added R200: 10k, Resistor_SMD:R_0805_2012Metric, symbol Device:R
- added R201: 100k, Resistor_SMD:R_0805_2012Metric, symbol Device:R
- R98: value 90k -> 100k
Connections:
- net GND_float2: now also J21.1 (Pin_1), R201.1; no longer J21.2 (Pin_2), R99.2
- net I_Bal: now also J21.2 (Pin_2); no longer J21.1 (Pin_1)
- net at C27.2, R101.1: now also R200.2; no longer U14.12 (+)
- net GNDShunt: no longer names the net of R98.2, R99.1, U14.13 (-)
- new net: R200.1, R201.2, U14.12 (+)
- new net V_Shunt_Low: R99.2
Other:
- moved on the sheet: C27, J21, J22, R101, R98, R99, U14D
