File: Aktive_Balancing/KiCAD/Aktive_Bal/Aktive_Bal.kicad_pcb (KiCad board)
At the start: 2 copper layers, 3.3 x 6.6 mm, 170 parts, among them J1 Conn_01x01_Pin, J2 Sockel_BluePill, J3 A-DF_09_A_KG-T4S, J4 Screw_Terminal_01x02, J5 Conn_01x01_Pin, J6 Conn_01x01_Pin, J7 Conn_01x01_Pin, J8 Conn_01x01_Pin, J9 Conn_01x01_Pin, Q1 BSS316NH6327XTSA1, Q10 NTTFS6H888NL, Q11 NTTFS6H888NL, Q12 NTTFS6H888NL, Q13 NTTFS6H888NL, Q14 NTTFS6H888NL, Q15 NTTFS6H888NL, Q16 NTTFS6H888NL, Q17 NTTFS6H888NL, Q18 NTTFS6H888NL, Q19 NTTFS6H888NL, Q20 NTTFS6H888NL, Q21 NTTFS6H888NL, Q22 NTTFS6H888NL, Q23 NTTFS6H888NL, Q24 NTTFS6H888NL, Q25 NTTFS6H888NL, Q26 NTTFS6H888NL, Q27 NTTFS6H888NL, Q28 NTTFS6H888NL, Q29 NTTFS6H888NL, Q3 NTTFS6H888NL, Q30 NTTFS6H888NL, Q31 NTTFS6H888NL, Q32 NTTFS6H888NL, Q33 NTTFS6H888NL, Q34 NTTFS6H888NL, Q4 NTTFS6H888NL, Q5 NTTFS6H888NL, Q6 NTTFS6H888NL, Q7 NTTFS6H888NL, Q8 NTTFS6H888NL, Q9 NTTFS6H888NL, U1 SCW20C-12, U10 LTV-847S, U11 LTV-847S, U12 LTV-847S, U13 RFP12N10L, U14 PCF8575CDB, U15 SN65HVD233, U2 EC1SA16N, U3 LM2596S-ADJ, U4 TL084, U5 ADUM1250ARZ-RL7, U6 PCA9306DC, U7 LM1117IMPX_3_3_NOPB, U8 MCP4725xxx-xCH, U9 LTV-847S

Commit message: kicad
Parts:
- removed C17: 4.7µ, Capacitor_SMD:C_0805_2012Metric
- removed C5, C6: 0.1µ, Capacitor_SMD:C_0805_2012Metric
- removed C7: 10µ tantal, Capacitor_SMD:C_0805_2012Metric
- removed J1, J5, J6, J7, J8: Conn_01x01_Pin, Connector_PinHeader_2.54mm:PinHeader_1x01_P2.54mm_Vertical
- removed JP1: Jumper_2_Bridged, Jumper:SolderJumper-2_P1.3mm_Bridged_Pad1.0x1.5mm
- removed JP2: Jumper_2_Open, Jumper:SolderJumper-2_P1.3mm_Open_TrianglePad1.0x1.5mm
- removed Q10, Q11, Q12, Q13, Q14, Q15, Q16, Q17, Q18, Q19, Q20, Q21, Q22, Q23, Q24, Q25, Q26, Q27, Q28, Q29, Q3, Q30, Q31, Q32, Q33, Q34, Q4, Q5, Q6, Q7, Q8, Q9: NTTFS6H888NL, Aktive_Bal_Footprints:8-WDFN
- removed U13: RFP12N10L, Aktive_Bal_Footprints:TO-220AB_ONS
- added C20: 0.1µ, Capacitor_SMD:C_0805_2012Metric, F.Cu at (30.0, 105.7)
- added C21: 10µ tantal, Capacitor_SMD:C_0805_2012Metric, F.Cu at (30.0, 108.7)
- added C22: 10µ, Capacitor_SMD:C_0805_2012Metric, F.Cu at (30.0, 111.7)
- added C23: 1n, Capacitor_SMD:C_0805_2012Metric, F.Cu at (34.4, 96.7)
- added C24: 0.1µ, Capacitor_SMD:C_0805_2012Metric, F.Cu at (34.4, 99.7)
- added C25: 10µ, Capacitor_SMD:C_0805_2012Metric, F.Cu at (34.4, 102.7)
- added C26: 0.1µ, Capacitor_SMD:C_0805_2012Metric, F.Cu at (34.4, 105.7)
- added C27: 0.1µ, Capacitor_SMD:C_0805_2012Metric, F.Cu at (66.1, 54.4)
- added C28: 0.1µ, Capacitor_SMD:C_0805_2012Metric, F.Cu at (66.1, 57.4)
- added C29: 1µ, Capacitor_SMD:C_0805_2012Metric, F.Cu at (66.1, 60.4)
- added C30: 10n, Capacitor_SMD:C_0805_2012Metric, F.Cu at (66.1, 63.4)
- added C31: 0.1µ, Capacitor_SMD:C_0805_2012Metric, F.Cu at (66.1, 66.4)
- added C32: 470µ, Capacitor_SMD:C_Elec_8x10.2, F.Cu at (75.0, 84.2)
- added C33: 47µ, Capacitor_SMD:CP_Elec_5x5.3, F.Cu at (90.5, 56.3)
- added C34: 1n, Capacitor_SMD:C_0805_2012Metric, F.Cu at (66.1, 69.4)
- added Q10_H1: NTTFS6H888NL, Aktive_Bal_Footprints:8-WDFN, F.Cu at (36.0, 23.3)
- added Q10_L1: NTTFS6H888NL, Aktive_Bal_Footprints:8-WDFN, F.Cu at (40.7, 23.3)
- added Q11_H1: NTTFS6H888NL, Aktive_Bal_Footprints:8-WDFN, F.Cu at (45.4, 23.3)
- added Q11_L1: NTTFS6H888NL, Aktive_Bal_Footprints:8-WDFN, F.Cu at (50.1, 23.3)
- added Q12_H1: NTTFS6H888NL, Aktive_Bal_Footprints:8-WDFN, F.Cu at (54.8, 23.3)
- added Q12_L1: NTTFS6H888NL, Aktive_Bal_Footprints:8-WDFN, F.Cu at (59.6, 23.3)
- added Q13_H1: NTTFS6H888NL, Aktive_Bal_Footprints:8-WDFN, F.Cu at (64.3, 23.3)
- added Q13_L1: NTTFS6H888NL, Aktive_Bal_Footprints:8-WDFN, F.Cu at (36.0, 28.1)
- added Q14_H1: NTTFS6H888NL, Aktive_Bal_Footprints:8-WDFN, F.Cu at (40.7, 28.1)
- added Q14_L1: NTTFS6H888NL, Aktive_Bal_Footprints:8-WDFN, F.Cu at (45.4, 28.1)
- added Q15_H1: NTTFS6H888NL, Aktive_Bal_Footprints:8-WDFN, F.Cu at (50.1, 28.1)
- added Q15_L1: NTTFS6H888NL, Aktive_Bal_Footprints:8-WDFN, F.Cu at (54.8, 28.1)
- added Q16_H1: NTTFS6H888NL, Aktive_Bal_Footprints:8-WDFN, F.Cu at (59.6, 28.1)
- added Q16_L1: NTTFS6H888NL, Aktive_Bal_Footprints:8-WDFN, F.Cu at (64.3, 28.1)
- added Q1_H1: NTTFS6H888NL, Aktive_Bal_Footprints:8-WDFN, F.Cu at (36.0, 32.9)
- added Q1_L1: NTTFS6H888NL, Aktive_Bal_Footprints:8-WDFN, F.Cu at (40.7, 32.9)
- added Q2_H1: NTTFS6H888NL, Aktive_Bal_Footprints:8-WDFN, F.Cu at (45.4, 32.9)
- added Q2_L1: NTTFS6H888NL, Aktive_Bal_Footprints:8-WDFN, F.Cu at (50.1, 32.9)
- added Q3_H1: NTTFS6H888NL, Aktive_Bal_Footprints:8-WDFN, F.Cu at (54.8, 32.9)
- added Q3_L1: NTTFS6H888NL, Aktive_Bal_Footprints:8-WDFN, F.Cu at (59.6, 32.9)
- added Q4_H1: NTTFS6H888NL, Aktive_Bal_Footprints:8-WDFN, F.Cu at (64.3, 32.9)
- added Q4_L1: NTTFS6H888NL, Aktive_Bal_Footprints:8-WDFN, F.Cu at (36.0, 37.8)
- added Q5_H1: NTTFS6H888NL, Aktive_Bal_Footprints:8-WDFN, F.Cu at (40.7, 37.8)
- added Q5_L1: NTTFS6H888NL, Aktive_Bal_Footprints:8-WDFN, F.Cu at (45.4, 37.8)
- added Q6_H1: NTTFS6H888NL, Aktive_Bal_Footprints:8-WDFN, F.Cu at (50.1, 37.8)
- added Q6_L1: NTTFS6H888NL, Aktive_Bal_Footprints:8-WDFN, F.Cu at (54.8, 37.8)
- added Q7_H1: NTTFS6H888NL, Aktive_Bal_Footprints:8-WDFN, F.Cu at (59.6, 37.8)
- added Q7_L1: NTTFS6H888NL, Aktive_Bal_Footprints:8-WDFN, F.Cu at (64.3, 37.8)
- added Q8_H1: NTTFS6H888NL, Aktive_Bal_Footprints:8-WDFN, F.Cu at (36.0, 42.6)
- added Q8_L1: NTTFS6H888NL, Aktive_Bal_Footprints:8-WDFN, F.Cu at (40.7, 42.6)
- added Q9_H1: NTTFS6H888NL, Aktive_Bal_Footprints:8-WDFN, F.Cu at (45.4, 42.6)
- added Q9_L1: NTTFS6H888NL, Aktive_Bal_Footprints:8-WDFN, F.Cu at (50.1, 42.6)
- added R100: 330, Resistor_SMD:R_0805_2012Metric, F.Cu at (32.6, 40.6)
- added R101: 100k, Resistor_SMD:R_0805_2012Metric, F.Cu at (32.6, 43.5)
- added R102: 330, Resistor_SMD:R_0805_2012Metric, F.Cu at (32.6, 46.5)
- added R103: 100k, Resistor_SMD:R_0805_2012Metric, F.Cu at (32.6, 49.4)
- added R87: 100k, Resistor_SMD:R_0805_2012Metric, F.Cu at (28.2, 31.7)
- added R88: 330, Resistor_SMD:R_0805_2012Metric, F.Cu at (28.2, 34.7)
- added R89: 100k, Resistor_SMD:R_0805_2012Metric, F.Cu at (28.2, 37.6)
- added R90: 330, Resistor_SMD:R_0805_2012Metric, F.Cu at (28.2, 40.6)
- added R91: 100k, Resistor_SMD:R_0805_2012Metric, F.Cu at (28.2, 43.5)
- added R92: 330, Resistor_SMD:R_0805_2012Metric, F.Cu at (28.2, 46.5)
- added R93: 100k, Resistor_SMD:R_0805_2012Metric, F.Cu at (28.2, 49.4)
- added R94: 330, Resistor_SMD:R_0805_2012Metric, F.Cu at (32.6, 22.9)
- added R95: 100k, Resistor_SMD:R_0805_2012Metric, F.Cu at (32.6, 25.8)
- added R96: 330, Resistor_SMD:R_0805_2012Metric, F.Cu at (32.6, 28.8)
- added R97: 100k, Resistor_SMD:R_0805_2012Metric, F.Cu at (32.6, 31.7)
- added R98: 330, Resistor_SMD:R_0805_2012Metric, F.Cu at (32.6, 34.7)
- added R99: 100k, Resistor_SMD:R_0805_2012Metric, F.Cu at (32.6, 37.6)
- C1: value 470µ -> 2.2µ; footprint Capacitor_SMD:C_Elec_8x10.2 -> Capacitor_SMD:C_0805_2012Metric
- C10: value 0.1n -> 10µ tantal
- C11, C15: value 1n -> 0.1µ
- C12: value 100n -> 10µ tantal
- C13, C14: value 2.2µ -> 0.1µ
- C16: value 1n -> 0.1n
- C18, C19: value 1µ -> 0.1µ
- C2: value 1µ -> 2.2µ
- C3: value 10n -> 1n
- C4: value 47µ -> 1n; footprint Capacitor_SMD:CP_Elec_5x5.3 -> Capacitor_SMD:C_0805_2012Metric
- C8: value 10µ tantal -> 0.1µ
- C9: value 10µ -> 0.1µ
- R1, R2: value 20k -> 4.7k
- R10, R11: value 4.7k -> 20k
- R12, R13: value 2.2k -> 20k
- R14: value 10 -> 10k
- R15: value 4.7k -> 1k
- R16: value 4.7k -> 20
- R17: value 200k -> 800
- R18: value 47k -> 2.41k
- R19: value 120k -> 47k
- R20: value 15k -> 90k
- R21: value 390 -> 10k
- R25: value 390 -> 1Meg
- R3, R4: value 20k -> 2.2k
- R37, R38: value 10k -> 390
- R39, R40, R41, R42, R43, R44, R45, R46, R47, R48, R49, R50, R51, R52: value 10k -> 100k
- R5: value 10k -> 200k
- R53: value 120 -> 100k
- R55: value 100 -> 100k
- R56, R72, R74, R76, R78, R80, R82, R84, R86: value 1Meg -> 330
- R57, R58, R59, R60, R61, R62, R63, R64, R65, R66, R67, R68, R69, R70, R71: value 100 -> 330
- R6: value 20 -> 4.7k
- R7: value 1k -> 4.7k
- R73, R75, R77, R79, R81, R83, R85: value 1Meg -> 100k
- R8: value 800 -> 10
- R9: value 2.41k -> 120
- moved J2 256.2 mm to (1.54, 54.9)
- moved C10 232.8 mm to (25.5, 96.7)
- moved C11 232.8 mm to (25.5, 99.7)
- moved C12 232.8 mm to (25.5, 102.7)
- moved C19 229.5 mm to (30.0, 102.7)
- moved C2 223.4 mm to (21.1, 99.7)
- moved C3 193.8 mm to (21.1, 102.7)
- moved J3 180.6 mm to (40.5, 77.7)
- moved C1 179.0 mm to (21.1, 96.7), turned to 0 degrees
- moved C4 174.0 mm to (21.1, 105.7), turned to 0 degrees
- moved R54 156.9 mm to (56.5, 0.81)
- moved U3 142.5 mm to (79.1, 59.1)
- moved L1 133.8 mm to (75.4, 72.3), turned to 0 degrees
- moved R33 132.8 mm to (6.12, 22.9)
- moved R22 132.8 mm to (1.71, 22.9)
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Connections:
- net Net-(JP3-B) renamed CANH
- C1 pad 1: +12V -> Net-(U13-D)
- C1 pad 2: GND_float2 -> Net-(J4-Pin_1)
- C10 pad 1: GND_float2 -> +5V
- C10 pad 2: Net-(U6-EN) -> GND_float2
- C11 pad 2: Net-(U4D-+) -> +5V
- C12 pad 1: +3.3Vµ -> +3.3V
- C12 pad 2: GNDµ -> GND_float2
- C13 pad 1: Net-(U13-DRAIN) -> GND_float2
- C13 pad 2: Net-(J4-Pin_1) -> +3.3V
- C14 pad 1: Net-(J6-Pin_1) -> +3.3Vµ
- C14 pad 2: Net-(J1-Pin_1) -> GNDµ
- C15 pad 1: +12V -> +5V
- C15 pad 2: Net-(J1-Pin_1) -> GND_float2
- C16 pad 1: Net-(J6-Pin_1) -> GND_float2
- C16 pad 2: GND_float2 -> Net-(U6-EN)
- C18 pad 1: -5V -> GND_float2
- C18 pad 2: GND_float2 -> +3.3V
- C19 pad 2: +5V -> Net-(U6-EN)
- C2 pad 1: Net-(U4B--) -> Net-(J16-Pin_1)
- C2 pad 2: Net-(U4C-+) -> Net-(J16-Pin_2)
- C3 pad 1: Net-(Q1-D) -> Net-(J16-Pin_1)
- C3 pad 2: Bal -> GND_float2
- C4 pad 1: Bal -> +12V
- C4 pad 2: GND_float2 -> Net-(J16-Pin_2)
- C8 pad 1: +3.3V -> -5V
- C9 pad 2: Net-(JP2-A) -> +5V
- FL1 pad 1: Net-(U13-DRAIN) -> Net-(U13-D)
- FL1 pad 3: Net-(J1-Pin_1) -> Net-(J16-Pin_2)
- FL1 pad 4: Net-(J6-Pin_1) -> Net-(J16-Pin_1)
- J2 pad 14: SCLµC -> unconnected-(J2-B6-Pad14)
- J2 pad 15: SDAµC -> unconnected-(J2-B7-Pad15)
- J2 pad 8: Net-(J2-A11) -> unconnected-(J2-A11-Pad8)
- J2 pad 9: Net-(J2-A12) -> unconnected-(J2-A12-Pad9)
- J3 pad 2: Net-(U15-CANL) -> CANL
- J3 pad 5: unconnected-(J3-Pad5) -> Net-(J3-SHIELD)
- J3 pad S1: unconnected-(J3-SHIELD-PadS1) -> Net-(J3-SHIELD)
- J3 pad S2: unconnected-(J3-SHIELD__1-PadS2) -> Net-(J3-SHIELD)
- JP4 pad 1: Net-(JP4-A) -> SDA5
- JP4 pad 2: Net-(JP4-B) -> SDA3.3
- JP5 pad 1: Net-(JP5-A) -> SCL5
- JP5 pad 2: Net-(JP5-B) -> SCL3.3
- R1 pad 1: Net-(U4A-+) -> SCLµC
- R1 pad 2: I_Bal -> +3.3Vµ
- R10 pad 1: SDAµC -> Net-(U4A-+)
- R10 pad 2: +3.3Vµ -> I_Bal
- R11 pad 1: SCLµC -> GND_float2
- R11 pad 2: +3.3Vµ -> Net-(U4A-+)
- R12 pad 1: Net-(JP5-A) -> I_Bal_Soll
- R12 pad 2: +5V -> Net-(U4A--)
- R13 pad 1: Net-(JP4-A) -> Net-(U4A--)
- R13 pad 2: +5V -> Net-(R13-Pad2)
- R14 pad 1: +5V -> Net-(R13-Pad2)
- R14 pad 2: Net-(JP2-A) -> Net-(U4B--)
- R15 pad 1: Net-(JP4-B) -> Net-(U4C--)
- R15 pad 2: +3.3V -> Net-(Q1-S)
- R16 pad 1: Net-(JP5-B) -> Net-(R16-Pad1)
- R16 pad 2: +3.3V -> Net-(Q1-G)
- R17 pad 1: Net-(U6-EN) -> GND_float2
- R17 pad 2: +5V -> Net-(Q1-S)
- R18 pad 1: Net-(U4D-+) -> Bal
- R18 pad 2: V_I_Bal -> Net-(Q1-D)
- R19 pad 1: I_Bal -> Net-(U4D-+)
- R19 pad 2: Net-(U4D--) -> V_I_Bal
- R2 pad 1: GND_float2 -> SDAµC
- R2 pad 2: Net-(U4A-+) -> +3.3Vµ
- R20 pad 1: Net-(U4D--) -> I_Bal
- R20 pad 2: GND_float2 -> Net-(U4D--)
- R21 pad 1: B1 -> Net-(U4D--)
- R21 pad 2: Net-(R21-Pad2) -> GND_float2
- R22 pad 1: B2 -> B1
- R23 pad 1: B3 -> B2
- R24 pad 1: B4 -> B3
- R25 pad 1: B5 -> GNDµ
- R25 pad 2: Net-(R25-Pad2) -> Net-(J3-SHIELD)
- R26 pad 1: B6 -> B4
- R27 pad 1: B7 -> B5
- R28 pad 1: B8 -> B6
- R29 pad 1: B9 -> B7
- R3 pad 1: Net-(U4A--) -> SDA5
- R3 pad 2: Net-(R3-Pad2) -> +5V
- R30 pad 1: B10 -> B8
- R31 pad 1: B11 -> B9
- R32 pad 1: B12 -> B10
- R33 pad 1: B13 -> B11
- R34 pad 1: B14 -> B12
- R35 pad 1: B15 -> B13
- R36 pad 1: B16 -> B14
- R37 pad 1: Net-(R37-Pad1) -> B15
- R37 pad 2: +12V -> Net-(R37-Pad2)
- R38 pad 1: Net-(R38-Pad1) -> B16
- R38 pad 2: +12V -> Net-(R38-Pad2)
- R39 pad 1: Net-(R39-Pad1) -> Net-(Q1_H1-G)
- R39 pad 2: +12V -> GND_float2
- R4 pad 1: I_Bal_Soll -> SCL5
- R4 pad 2: Net-(U4A--) -> +5V
- R40 pad 1: Net-(R40-Pad1) -> Net-(Q2_H1-G)
- R40 pad 2: +12V -> GND_float2
- R41 pad 1: Net-(R41-Pad1) -> Net-(Q3_H1-G)
- R41 pad 2: +12V -> GND_float2
- R42 pad 1: Net-(R42-Pad1) -> Net-(Q4_H1-G)
- R42 pad 2: +12V -> GND_float2
- R43 pad 1: Net-(R43-Pad1) -> Net-(Q5_H1-G)
- R43 pad 2: +12V -> GND_float2
- R44 pad 1: Net-(R44-Pad1) -> Net-(Q6_H1-G)
- R44 pad 2: +12V -> GND_float2
- R45 pad 1: Net-(R45-Pad1) -> Net-(Q7_H1-G)
- R45 pad 2: +12V -> GND_float2
- R46 pad 1: Net-(R46-Pad1) -> Net-(Q8_H1-G)
- R46 pad 2: +12V -> GND_float2
- R47 pad 1: Net-(R47-Pad1) -> Net-(Q9_H1-G)
- R47 pad 2: +12V -> GND_float2
- R48 pad 1: Net-(R48-Pad1) -> Net-(Q10_H1-G)
- R48 pad 2: +12V -> GND_float2
- R49 pad 1: Net-(R49-Pad1) -> Net-(Q11_H1-G)
- R49 pad 2: +12V -> GND_float2
- R5 pad 1: Net-(R3-Pad2) -> Net-(U6-EN)
- R5 pad 2: Net-(U4B--) -> +5V
- R50 pad 1: Net-(R50-Pad1) -> Net-(Q12_H1-G)
- R50 pad 2: +12V -> GND_float2
- R51 pad 1: Net-(R51-Pad1) -> Net-(Q13_H1-G)
- R51 pad 2: +12V -> GND_float2
- R52 pad 1: Net-(R52-Pad1) -> Net-(Q14_H1-G)
- R52 pad 2: +12V -> GND_float2
- R53 pad 1: Net-(U15-CANL) -> Net-(Q15_H1-G)
- R53 pad 2: Net-(JP3-A) -> GND_float2
- R55 pad 1: Net-(R37-Pad1) -> Net-(Q16_H1-G)
- R55 pad 2: Net-(Q3-G) -> GND_float2
- R56 pad 1: Net-(Q3-G) -> Net-(R56-Pad1)
- R56 pad 2: C0 -> Net-(Q1_H1-G)
- R57 pad 1: Net-(R38-Pad1) -> Net-(R57-Pad1)
- R57 pad 2: Net-(Q6-G) -> Net-(Q2_H1-G)
- R58 pad 1: Net-(R39-Pad1) -> Net-(R58-Pad1)
- R58 pad 2: Net-(Q9-G) -> Net-(Q3_H1-G)
- R59 pad 1: Net-(R40-Pad1) -> Net-(R59-Pad1)
- R59 pad 2: Net-(Q10-G) -> Net-(Q4_H1-G)
- R6 pad 1: Net-(R6-Pad1) -> SCL3.3
- R6 pad 2: Net-(Q1-G) -> +3.3V
- R60 pad 1: Net-(R41-Pad1) -> Net-(R60-Pad1)
- R60 pad 2: Net-(Q15-G) -> Net-(Q5_H1-G)
- R61 pad 1: Net-(R42-Pad1) -> Net-(R61-Pad1)
- R61 pad 2: Net-(Q16-G) -> Net-(Q6_H1-G)
- R62 pad 1: Net-(R43-Pad1) -> Net-(R62-Pad1)
- R62 pad 2: Net-(Q17-G) -> Net-(Q7_H1-G)
- R63 pad 1: Net-(R44-Pad1) -> Net-(R63-Pad1)
- R63 pad 2: Net-(Q18-G) -> Net-(Q8_H1-G)
- R64 pad 1: Net-(R45-Pad1) -> Net-(R64-Pad1)
- R64 pad 2: Net-(Q27-G) -> Net-(Q9_H1-G)
- R65 pad 1: Net-(R46-Pad1) -> Net-(R65-Pad1)
- R65 pad 2: Net-(Q28-G) -> Net-(Q10_H1-G)
- R66 pad 1: Net-(R47-Pad1) -> Net-(R66-Pad1)
- R66 pad 2: Net-(Q29-G) -> Net-(Q11_H1-G)
- R67 pad 1: Net-(R48-Pad1) -> Net-(R67-Pad1)
- R67 pad 2: Net-(Q30-G) -> Net-(Q12_H1-G)
- R68 pad 1: Net-(R49-Pad1) -> Net-(R68-Pad1)
- R68 pad 2: Net-(Q31-G) -> Net-(Q13_H1-G)
- R69 pad 1: Net-(R50-Pad1) -> Net-(R69-Pad1)
- R69 pad 2: Net-(Q32-G) -> Net-(Q14_H1-G)
- R7 pad 1: Net-(U4C--) -> SDA3.3
- R7 pad 2: Net-(Q1-S) -> +3.3V
- R70 pad 1: Net-(R51-Pad1) -> Net-(R70-Pad1)
- R70 pad 2: Net-(Q33-G) -> Net-(Q15_H1-G)
- R71 pad 1: Net-(R52-Pad1) -> Net-(R71-Pad1)
- R71 pad 2: Net-(Q34-G) -> Net-(Q16_H1-G)
- R72 pad 1: Net-(Q6-G) -> B1
- R72 pad 2: C1 -> Net-(Q1_L1-G)
- R73 pad 1: Net-(Q9-G) -> Net-(Q1_L1-G)
- R73 pad 2: C2 -> GND_float2
- R74 pad 1: Net-(Q10-G) -> B2
- R74 pad 2: C3 -> Net-(Q2_L1-G)
- R75 pad 1: Net-(Q15-G) -> Net-(Q2_L1-G)
- R75 pad 2: C4 -> GND_float2
- R76 pad 1: Net-(Q16-G) -> B3
- R76 pad 2: C5 -> Net-(Q3_L1-G)
- R77 pad 1: Net-(Q17-G) -> Net-(Q3_L1-G)
- R77 pad 2: C6 -> GND_float2
- R78 pad 1: Net-(Q18-G) -> B4
- R78 pad 2: C7 -> Net-(Q4_L1-G)
- R79 pad 1: Net-(Q27-G) -> Net-(Q4_L1-G)
- R79 pad 2: C8 -> GND_float2
- R8 pad 1: GND_float2 -> +5V
- R8 pad 2: Net-(Q1-S) -> Net-(JP6-A)
- R80 pad 1: Net-(Q28-G) -> B5
- R80 pad 2: C9 -> Net-(Q5_L1-G)
- R81 pad 1: Net-(Q29-G) -> Net-(Q5_L1-G)
- R81 pad 2: C10 -> GND_float2
- R82 pad 1: Net-(Q30-G) -> B6
- R82 pad 2: Net-(Q30-S-Pad1) -> Net-(Q6_L1-G)
- R83 pad 1: Net-(Q31-G) -> Net-(Q6_L1-G)
- R83 pad 2: C12 -> GND_float2
- R84 pad 1: Net-(Q32-G) -> B7
- R84 pad 2: C13 -> Net-(Q7_L1-G)
- R85 pad 1: Net-(Q33-G) -> Net-(Q7_L1-G)
- R85 pad 2: C14 -> GND_float2
- R86 pad 1: Net-(Q34-G) -> B8
- R86 pad 2: C15 -> Net-(Q8_L1-G)
- R9 pad 1: Bal -> CANL
- R9 pad 2: Net-(Q1-D) -> Net-(JP3-A)
- U1 pad 2: Net-(J6-Pin_1) -> Net-(J16-Pin_1)
- U1 pad 22: Net-(J1-Pin_1) -> Net-(J16-Pin_2)
- U1 pad 23: Net-(J1-Pin_1) -> Net-(J16-Pin_2)
- U1 pad 3: Net-(J6-Pin_1) -> Net-(J16-Pin_1)
- U10 pad 1: Net-(R25-Pad2) -> Net-(R27-Pad2)
- U10 pad 10: Net-(R44-Pad1) -> +12V
- U10 pad 11: GND_float2 -> Net-(R62-Pad1)
- U10 pad 12: Net-(R43-Pad1) -> +12V
- U10 pad 13: GND_float2 -> Net-(R61-Pad1)
- U10 pad 14: Net-(R42-Pad1) -> +12V
- U10 pad 15: GND_float2 -> Net-(R60-Pad1)
- U10 pad 16: Net-(R41-Pad1) -> +12V
- U10 pad 3: Net-(R26-Pad2) -> Net-(R28-Pad2)
- U10 pad 5: Net-(R27-Pad2) -> Net-(R29-Pad2)
- U10 pad 7: Net-(R28-Pad2) -> Net-(R30-Pad2)
- U10 pad 9: GND_float2 -> Net-(R63-Pad1)
- U11 pad 1: Net-(R29-Pad2) -> Net-(R31-Pad2)
- U11 pad 10: Net-(R48-Pad1) -> +12V
- U11 pad 11: GND_float2 -> Net-(R66-Pad1)
- U11 pad 12: Net-(R47-Pad1) -> +12V
- U11 pad 13: GND_float2 -> Net-(R65-Pad1)
- U11 pad 14: Net-(R46-Pad1) -> +12V
- U11 pad 15: GND_float2 -> Net-(R64-Pad1)
- U11 pad 16: Net-(R45-Pad1) -> +12V
- U11 pad 3: Net-(R30-Pad2) -> Net-(R32-Pad2)
- U11 pad 5: Net-(R31-Pad2) -> Net-(R33-Pad2)
- U11 pad 7: Net-(R32-Pad2) -> Net-(R34-Pad2)
- U11 pad 9: GND_float2 -> Net-(R67-Pad1)
- U12 pad 1: Net-(R33-Pad2) -> Net-(R35-Pad2)
- U12 pad 10: Net-(R52-Pad1) -> +12V
- U12 pad 11: GND_float2 -> Net-(R70-Pad1)
- U12 pad 12: Net-(R51-Pad1) -> +12V
- U12 pad 13: GND_float2 -> Net-(R69-Pad1)
- U12 pad 14: Net-(R50-Pad1) -> +12V
- U12 pad 15: GND_float2 -> Net-(R68-Pad1)
- U12 pad 16: Net-(R49-Pad1) -> +12V
- U12 pad 3: Net-(R34-Pad2) -> Net-(R36-Pad2)
- U12 pad 5: Net-(R35-Pad2) -> Net-(R37-Pad2)
- U12 pad 7: Net-(R36-Pad2) -> Net-(R38-Pad2)
- U12 pad 9: GND_float2 -> Net-(R71-Pad1)
- U14 pad 22: Net-(JP4-A) -> SCL5
- U14 pad 23: Net-(JP5-A) -> SDA5
- U15 pad 1: Net-(J2-A12) -> D
- U15 pad 4: Net-(J2-A11) -> R
- U15 pad 6: Net-(U15-CANL) -> CANL
- U4 pad 1: Net-(R3-Pad2) -> Net-(R13-Pad2)
- U4 pad 8: Net-(R6-Pad1) -> Net-(R16-Pad1)
- U5 pad 6: Net-(JP4-A) -> SCL5
- U5 pad 7: Net-(JP5-A) -> SDA5
- U6 pad 3: Net-(JP4-B) -> SCL3.3
- U6 pad 4: Net-(JP5-B) -> SDA3.3
- U6 pad 5: Net-(JP5-A) -> SDA5
- U6 pad 6: Net-(JP4-A) -> SCL5
- U8 pad 4: Net-(JP5-B) -> SDA3.3
- U8 pad 5: Net-(JP4-B) -> SCL3.3
- U9 pad 1: Net-(R21-Pad2) -> Net-(R22-Pad2)
- U9 pad 10: Net-(R40-Pad1) -> +12V
- U9 pad 11: GND_float2 -> Net-(R58-Pad1)
- U9 pad 12: Net-(R39-Pad1) -> +12V
- U9 pad 13: GND_float2 -> Net-(R57-Pad1)
- U9 pad 14: Net-(R38-Pad1) -> +12V
- U9 pad 15: GND_float2 -> Net-(R56-Pad1)
- U9 pad 16: Net-(R37-Pad1) -> +12V
- U9 pad 3: Net-(R22-Pad2) -> Net-(R23-Pad2)
- U9 pad 5: Net-(R23-Pad2) -> Net-(R24-Pad2)
- U9 pad 7: Net-(R24-Pad2) -> Net-(R26-Pad2)
- U9 pad 9: GND_float2 -> Net-(R59-Pad1)
Routing:
- net GND_float2: track 44.5 -> 0.00 mm
- net Net-(J6-Pin_1): track 41.5 -> 0.00 mm
- net +12V: track 40.4 -> 0.00 mm
- net Net-(J1-Pin_1): track 33.8 -> 0.00 mm
- net Net-(J4-Pin_1): track 23.9 -> 0.00 mm
- net +5V: track 18.7 -> 0.00 mm
- net Net-(D1-K): track 18.4 -> 0.00 mm
- net Net-(U13-DRAIN): track 13.5 -> 0.00 mm
- net Bal: track 8.10 -> 0.00 mm
- net Bat_GND: track 8.03 -> 0.00 mm
- net -5V: track 5.44 -> 0.00 mm
- net +3.3V: track 3.05 -> 0.00 mm
Other:
- copper layers 2 -> 4

Commit message: layout
Parts:
- removed C8, C9: 0.1µ, Capacitor_SMD:C_0805_2012Metric
- added C17: 4.7µ, Capacitor_SMD:C_0805_2012Metric, F.Cu at (123.9, 73.1)
- added C36: 10µ, Capacitor_SMD:CP_Elec_4x5.4, F.Cu at (90.1, 27.9)
- added C37: 10µ, Capacitor_SMD:CP_Elec_4x5.4, F.Cu at (90.1, 33.8)
- added C38: 47µ, Capacitor_SMD:CP_Elec_6.3x5.7, F.Cu at (38.7, 81.4)
- added J1: Conn_01x01_Pin, Connector_PinHeader_2.54mm:PinHeader_1x01_P2.54mm_Vertical, F.Cu at (77.6, 84.4)
- added J10: Screw_Terminal_01x03, TerminalBlock_CUI:TerminalBlock_CUI_TB007-508-03_1x03_P5.08mm_Horizontal, F.Cu at (274.0, 51.3)
- added J11: Screw_Terminal_01x03, TerminalBlock_CUI:TerminalBlock_CUI_TB007-508-03_1x03_P5.08mm_Horizontal, F.Cu at (274.0, 68.0)
- added J12: Screw_Terminal_01x03, TerminalBlock_CUI:TerminalBlock_CUI_TB007-508-03_1x03_P5.08mm_Horizontal, F.Cu at (274.0, 84.5)
- added J13: Screw_Terminal_01x03, TerminalBlock_CUI:TerminalBlock_CUI_TB007-508-03_1x03_P5.08mm_Horizontal, F.Cu at (274.0, 100.8)
- added J17: Conn_01x02_Pin, Connector_PinHeader_2.54mm:PinHeader_1x02_P2.54mm_Vertical, F.Cu at (55.1, 69.6)
- added J18: Conn_01x02_Pin, Connector_PinHeader_2.54mm:PinHeader_1x02_P2.54mm_Vertical, F.Cu at (59.7, 69.6)
- added J19: Conn_01x02_Pin, Connector_PinHeader_2.54mm:PinHeader_1x02_P2.54mm_Vertical, F.Cu at (64.3, 69.6)
- added J20: Conn_01x02_Pin, Connector_PinHeader_2.54mm:PinHeader_1x02_P2.54mm_Vertical, F.Cu at (68.9, 69.6)
- added J21: Conn_01x02_Pin, Connector_PinHeader_2.54mm:PinHeader_1x02_P2.54mm_Vertical, F.Cu at (73.5, 69.6)
- added J22: Conn_01x02_Pin, Connector_PinHeader_2.54mm:PinHeader_1x02_P2.54mm_Vertical, F.Cu at (78.1, 69.6)
- added J5: Conn_01x01_Pin, Connector_PinHeader_2.54mm:PinHeader_1x01_P2.54mm_Vertical, F.Cu at (189.0, 83.0)
- added J6: Conn_01x01_Pin, Connector_PinHeader_2.54mm:PinHeader_1x01_P2.54mm_Vertical, F.Cu at (112.0, 184.2)
- added J7: Screw_Terminal_01x03, TerminalBlock_CUI:TerminalBlock_CUI_TB007-508-03_1x03_P5.08mm_Horizontal, F.Cu at (274.0, 17.8)
- added J8: Screw_Terminal_01x03, TerminalBlock_CUI:TerminalBlock_CUI_TB007-508-03_1x03_P5.08mm_Horizontal, F.Cu at (274.0, 35.0)
- added JP6: Jumper_3_Bridged12, Connector_PinHeader_2.54mm:PinHeader_1x03_P2.54mm_Vertical, F.Cu at (98.9, 39.0)
- added L2: 10µ, Inductor_SMD:L_Bourns_SRR1260, F.Cu at (213.9, 118.4)
- added U13: RFP12N10L, Aktive_Bal_Footprints:TO-220AB_ONS, F.Cu at (90.4, 63.1)
- moved R103 207.9 mm to (240.3, 41.1)
- moved R54 189.2 mm to (105.8, 183.5)
- moved Q16_L1 180.9 mm to (244.5, 43.6)
- moved Q4_H1 180.9 mm to (244.5, 48.5)
- moved Q7_L1 180.9 mm to (244.5, 53.3)
- moved U12 180.7 mm to (127.4, 172.7)
- moved Q13_H1 178.4 mm to (242.7, 24.4)
- moved Q12_H1 173.3 mm to (224.2, 59.9)
- moved Q15_L1 173.3 mm to (224.2, 64.7)
- moved Q3_H1 173.3 mm to (224.2, 69.5)
- moved Q6_L1 173.3 mm to (224.2, 74.4)
- moved Q12_L1 172.9 mm to (231.3, 43.6)
- moved Q16_H1 172.9 mm to (231.3, 48.5)
- moved Q3_L1 172.9 mm to (231.3, 53.3)
- moved Q7_H1 172.9 mm to (231.3, 58.1)
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Connections:
- C11 pad 1: GND_float2 -> +5V
- C11 pad 2: +5V -> GND_float2
- C13 pad 1: GND_float2 -> +3.3V
- C13 pad 2: +3.3V -> GND_float2
- C31 pad 2: +12V -> Net-(U3-VIN)
- C32 pad 1: +12V -> Net-(U3-VIN)
- U3 pad 1: +12V -> Net-(U3-VIN)
Routing:
- net Net-(U3-VIN): track 0.00 -> 24.8 mm
- net Net-(Q1-D): track 0.00 -> 23.5 mm
- net Net-(D1-K): track 0.00 -> 20.1 mm
- net I_Bal: track 0.00 -> 4.38 mm

Commit message: layout
Parts:
- added R2: 100k, Resistor_SMD:R_0805_2012Metric, F.Cu at (102.9, 64.9)
- C7: renamed from C25; value 10µ -> 0.1µ
- L1: renamed from L2; footprint Inductor_SMD:L_Bourns_SRR1260 -> Aktive_Bal_Footprints:NRS6045
- moved J5 122.8 mm to (-48.3, 116.8)
- moved U2 86.5 mm to (-35.6, 102.2)
- moved R91 86.1 mm to (233.3, 127.0)
- moved U6 74.7 mm to (109.2, 25.4)
- moved Q16_H1 72.5 mm to (253.1, 17.4), turned to 90 degrees
- moved Q13_L1 69.0 mm to (252.1, 40.3)
- moved Q1_L1 61.7 mm to (249.3, 105.1)
- moved Q15_H1 59.3 mm to (253.1, 23.4), turned to 90 degrees
- moved J2 58.9 mm to (18.1, 66.5), turned to -90 degrees
- moved JP1 55.5 mm to (52.7, 61.3)
- moved Q14_H1 50.2 mm to (253.1, 28.5), turned to 90 degrees
- moved C16 38.5 mm to (126.6, 21.7), turned to 90 degrees
- moved C15 29.5 mm to (118.9, 21.7), turned to -90 degrees
- moved C25 27.0 mm to (158.1, 106.7)
- moved C26 27.0 mm to (174.3, 106.7)
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- renumbered C23 to C1, C38 to C10, C16 to C11, C17 to C12, C19 to C13, C18 to C14, C36 to C15, C37 to C16, C10 to C17, C11 to C18, C26 to C19, C24 to C2, C13 to C20, C12 to C21, C21 to C23, C20 to C24, C27 to C25, C28 to C26, C29 to C27, C34 to C28, C32 to C29, C14 to C3, C31 to C30, C30 to C31, C33 to C32, C1 to C4, C15 to C5, C2 to C6, C3 to C8, C4 to C9, J4 to J1, J9 to J10, J1 to J11, J7 to J12, J8 to J13, J10 to J14, J11 to J15, J12 to J16, J13 to J17, J5 to J18, J6 to J19, J3 to J2, J21 to J3, J19 to J4, J2 to J5, J22 to J6, J17 to J7, J20 to J8, J18 to J9, JP3 to JP1, JP4 to JP2, JP5 to JP3, JP6 to JP4, L1 to L2, Q7_H1 to Q10_H1, Q7_L1 to Q10_L1, Q6_H1 to Q11_H1, Q6_L1 to Q11_L1, Q5_H1 to Q12_H1, Q5_L1 to Q12_L1, Q4_H1 to Q13_H1, Q4_L1 to Q13_L1, Q3_H1 to Q14_H1, Q3_L1 to Q14_L1, Q2_H1 to Q15_H1, Q2_L1 to Q15_L1, Q1_H1 to Q16_H1, Q1_L1 to Q16_L1, Q16_H1 to Q1_H1, Q16_L1 to Q1_L1, Q15_H1 to Q2_H1, Q15_L1 to Q2_L1, Q14_H1 to Q3_H1, Q14_L1 to Q3_L1, Q13_H1 to Q4_H1, Q13_L1 to Q4_L1, Q12_H1 to Q5_H1, Q12_L1 to Q5_L1, Q11_H1 to Q6_H1, Q11_L1 to Q6_L1, Q10_H1 to Q7_H1, Q10_L1 to Q7_L1, Q9_H1 to Q8_H1, Q9_L1 to Q8_L1, Q8_H1 to Q9_H1, Q8_L1 to Q9_L1, R25 to R1, R7 to R10, R15 to R100, R19 to R101, R16 to R102, R17 to R103, R18 to R104, R8 to R11, R22 to R12, R23 to R13, R24 to R14, R26 to R15, R27 to R16, R28 to R17, R29 to R18, R30 to R19, R31 to R20, R32 to R21, R33 to R22, R34 to R23, R35 to R24, R36 to R25, R37 to R26, R38 to R27, R56 to R28, R57 to R29, R1 to R3, R58 to R30, R59 to R31, R60 to R32, R61 to R33, R62 to R34, R63 to R35, R64 to R36, R65 to R37, R66 to R38, R67 to R39, R2 to R4, R68 to R40, R69 to R41, R70 to R42, R71 to R43, R39 to R44, R41 to R45, R43 to R46, R45 to R47, R47 to R48, R9 to R5, R51 to R50, R53 to R51, R40 to R52, R42 to R53, R44 to R54, R46 to R55, R48 to R56, R50 to R57, R52 to R58, R55 to R59, R3 to R6, R72 to R60, R74 to R61, R76 to R62, R78 to R63, R80 to R64, R82 to R65, R84 to R66, R86 to R67, R88 to R68, R90 to R69, R4 to R7, R92 to R70, R94 to R71, R96 to R72, R98 to R73, R100 to R74, R102 to R75, R73 to R76, R75 to R77, R77 to R78, R5 to R8, R81 to R80, R83 to R81, R85 to R82, R87 to R83, R89 to R84, R91 to R85, R93 to R86, R95 to R87, R97 to R88, R99 to R89, R6 to R9, R101 to R90, R103 to R91, R54 to R92, R10 to R93, R12 to R94, R11 to R95, R13 to R96, R14 to R97, R20 to R98, R21 to R99, U13 to U1, U9 to U10, U10 to U11, U11 to U12, U12 to U13, U4 to U14, U3 to U15, U15 to U2, U5 to U3, U1 to U4, U6 to U5, U2 to U6, U14 to U7, U7 to U8, U8 to U9
Connections:
- R12 pad 1: B1 -> B16
- R13 pad 1: B2 -> B15
- R14 pad 1: B3 -> B14
- R15 pad 1: B4 -> B13
- R16 pad 1: B5 -> B12
- R17 pad 1: B6 -> B11
- R18 pad 1: B7 -> B10
- R19 pad 1: B8 -> B9
- R20 pad 1: B9 -> B8
- R21 pad 1: B10 -> B7
- R22 pad 1: B11 -> B6
- R23 pad 1: B12 -> B5
- R24 pad 1: B13 -> B4
- R25 pad 1: B14 -> B3
- R26 pad 1: B15 -> B2
- R27 pad 1: B16 -> B1
- R60 pad 1: B1 -> B16
- R61 pad 1: B2 -> B15
- R62 pad 1: B3 -> B14
- R63 pad 1: B4 -> B13
- R64 pad 1: B5 -> B12
- R65 pad 1: B6 -> B11
- R66 pad 1: B7 -> B10
- R67 pad 1: B8 -> B9
- R68 pad 1: B9 -> B8
- R69 pad 1: B10 -> B7
- R70 pad 1: B11 -> B6
- R71 pad 1: B12 -> B5
- R72 pad 1: B13 -> B4
- R73 pad 1: B14 -> B3
- R74 pad 1: B15 -> B2
- R75 pad 1: B16 -> B1

Commit message: layour
Parts:
- Q10_H1, Q10_L1, Q11_H1, Q11_L1, Q12_H1, Q12_L1, Q13_H1, Q13_L1, Q14_H1, Q14_L1, Q15_H1, Q15_L1, Q16_H1, Q16_L1, Q1_H1, Q1_L1, Q2_H1, Q2_L1, Q3_H1, Q3_L1, Q4_H1, Q4_L1, Q5_H1, Q5_L1, Q6_H1, Q6_L1, Q7_H1, Q7_L1, Q8_H1, Q8_L1, Q9_H1, Q9_L1: footprint Aktive_Bal_Footprints:8-WDFN -> Aktive_Bal_Footprints:TRANS_NVTFS5116PLTAG
- moved R44 252.4 mm to (258.4, 19.8)
- moved R52 250.7 mm to (258.4, 26.2)
- moved R45 249.0 mm to (258.4, 32.6)
- moved R53 247.3 mm to (258.4, 39.1)
- moved R28 232.0 mm to (253.6, 19.8)
- moved R29 231.5 mm to (253.6, 26.2)
- moved R30 231.4 mm to (253.6, 32.6)
- moved R31 229.8 mm to (253.6, 39.1)
- moved R32 228.2 mm to (253.6, 45.5)
- moved R33 226.7 mm to (253.6, 51.9)
- moved R46 225.9 mm to (258.4, 45.5)
- moved R54 225.6 mm to (258.4, 51.9)
- moved R47 225.3 mm to (258.4, 58.3)
- moved R34 225.2 mm to (253.6, 58.3)
- moved R55 225.0 mm to (258.4, 64.7)
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Other:
- board size 3.3 x 6.6 mm -> 380 x 202.9 mm

Commit message: layout
Komponenten geordnet
Parts:
- removed C13: 0.1µ, Capacitor_SMD:C_0805_2012Metric
- moved R11 237.7 mm to (-97.5, 33.5), turned to -90 degrees
- moved C22 227.7 mm to (-97.0, 38.1)
- moved C24 223.0 mm to (-94.0, 43.2), turned to 90 degrees
- moved C23 219.9 mm to (-90.4, 43.2), turned to 90 degrees
- moved C7 198.9 mm to (-53.1, 163.6), turned to 90 degrees
- moved JP4 191.9 mm to (-93.0, 38.1), turned to 180 degrees
- moved J11 174.0 mm to (-88.9, 34.0)
- moved C28 164.2 mm to (26.4, 174.4), turned to -90 degrees
- moved J10 161.1 mm to (171.2, -42.2)
- moved L1 158.7 mm to (60.5, 162.7)
- moved J9 152.2 mm to (163.6, -41.7), turned to -90 degrees
- moved D1 149.2 mm to (53.4, 169.4)
- moved C10 148.2 mm to (130.6, -46.2), turned to 180 degrees
- moved J18 147.6 mm to (31.5, 157.5)
- moved R97 145.8 mm to (28.4, 166.6), turned to -90 degrees
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Connections:
- net Net-(J1-Pin_1) renamed BAT+
- C14 pad 2: +3.3V -> Net-(U5-VREF1)
- J7 pad 2: +12V -> GND_float2
- R10 pad 2: +3.3V -> Net-(U5-VREF1)
- R9 pad 2: +3.3V -> Net-(U5-VREF1)
- U5 pad 2: +3.3V -> Net-(U5-VREF1)
- U7 pad 13: B16 -> B9
- U7 pad 14: B15 -> B10
- U7 pad 15: B14 -> B11
- U7 pad 16: B13 -> B12
- U7 pad 17: B12 -> B13
- U7 pad 18: B11 -> B14
- U7 pad 19: B10 -> B15
- U7 pad 20: B9 -> B16
Routing:
- net Net-(J2-SHIELD): track 0.00 -> 27.7 mm
- net Net-(U15-VIN): track 24.8 -> 0.00 mm
- net Net-(D1-K): track 20.1 -> 0.00 mm
- net Bat_GND: track 0.00 -> 15.8 mm
- net enable: track 0.00 -> 4.68 mm
- net I_Bal: track 4.38 -> 0.00 mm
- net Net-(Q1-D): track 23.5 -> 20.9 mm
Other:
- board size 380 x 202.9 mm -> 3.3 x 6.6 mm
- board text added: "+12 GNDf"
- board text added: "+3.3"
- board text added: "-5 +5"

Commit message: Schaltung Review + Layout
Schaltung Review + Layout
Parts:
- added C13: 0.1µ, Capacitor_SMD:C_0805_2012Metric, F.Cu at (116.8, 98.7)
- added J20: Screw_Terminal_01x03, TerminalBlock_CUI:TerminalBlock_CUI_TB007-508-03_1x03_P5.08mm_Horizontal, F.Cu at (275.3, 105.3)
- added J21: Conn_01x02_Pin, Connector_PinHeader_2.54mm:PinHeader_1x02_P2.54mm_Vertical, F.Cu at (29.7, 128.0)
- added J22: Conn_01x02_Pin, Connector_PinHeader_2.54mm:PinHeader_1x02_P2.54mm_Vertical, F.Cu at (34.3, 128.0)
- added J23: Conn_01x02_Pin, Connector_PinHeader_2.54mm:PinHeader_1x02_P2.54mm_Vertical, F.Cu at (38.9, 128.0)
- added J24: Conn_01x02_Pin, Connector_PinHeader_2.54mm:PinHeader_1x02_P2.54mm_Vertical, F.Cu at (43.5, 128.0)
- added JP5: Jumper_3_Bridged12, Connector_PinHeader_2.54mm:PinHeader_1x03_P2.54mm_Vertical, F.Cu at (133.3, 155.3)
- added JP6: Jumper_2_Open, Jumper:SolderJumper-2_P1.3mm_Open_TrianglePad1.0x1.5mm, F.Cu at (110.5, 87.5)
- added JP7: Jumper_2_Open, Jumper:SolderJumper-2_P1.3mm_Open_TrianglePad1.0x1.5mm, F.Cu at (110.5, 91.4)
- added JP8: Jumper_3_Bridged12, Connector_PinHeader_2.54mm:PinHeader_1x03_P2.54mm_Vertical, F.Cu at (130.0, 106.5)
- added JP9: Jumper_3_Bridged12, Connector_PinHeader_2.54mm:PinHeader_1x03_P2.54mm_Vertical, F.Cu at (135.4, 94.9)
- C14: value 0.1µ -> 10µ; footprint Capacitor_SMD:C_0805_2012Metric -> Capacitor_SMD:CP_Elec_4x5.4
- C16: value 10µ -> 10µ tantal; footprint Capacitor_SMD:CP_Elec_4x5.4 -> Capacitor_SMD:C_0805_2012Metric
- C17, C23: value 10µ tantal -> 0.1µ
- C20: value 0.1µ -> 10µ tantal
- C21: value 10µ tantal -> 10µ
- C22: value 10µ -> 10µ tantal
- C26: value 0.1µ -> 1µ
- C27: value 1µ -> 1n
- C28: value 1n -> 470µ; footprint Capacitor_SMD:C_0805_2012Metric -> Capacitor_SMD:C_Elec_8x10.2
- C29: value 470µ -> 0.1µ; footprint Capacitor_SMD:C_Elec_8x10.2 -> Capacitor_SMD:C_0805_2012Metric
- C30: value 0.1µ -> 10n
- C31: value 10n -> 47µ; footprint Capacitor_SMD:C_0805_2012Metric -> Capacitor_SMD:CP_Elec_5x5.3
- J10, J11: value Conn_01x01_Pin -> Conn_01x02_Pin; footprint Connector_PinHeader_2.54mm:PinHeader_1x01_P2.54mm_Vertical -> Connector_PinHeader_2.54mm:PinHeader_1x02_P2.54mm_Vertical
- J12, J13, J14: value Screw_Terminal_01x03 -> Conn_01x02_Pin; footprint TerminalBlock_CUI:TerminalBlock_CUI_TB007-508-03_1x03_P5.08mm_Horizontal -> Connector_PinHeader_2.54mm:PinHeader_1x02_P2.54mm_Vertical
- J18, J19: value Conn_01x01_Pin -> Screw_Terminal_01x03; footprint Connector_PinHeader_2.54mm:PinHeader_1x01_P2.54mm_Vertical -> TerminalBlock_CUI:TerminalBlock_CUI_TB007-508-03_1x03_P5.08mm_Horizontal
- J5: value Sockel_BluePill -> Conn_01x02_Pin; footprint Aktive_Bal_Footprints:SockelBluepill Dupont leisten -> Connector_PinHeader_2.54mm:PinHeader_1x02_P2.54mm_Vertical
- J7: value Conn_01x02_Pin -> Sockel_BluePill; footprint Connector_PinHeader_2.54mm:PinHeader_1x02_P2.54mm_Vertical -> Aktive_Bal_Footprints:SockelBluepill Dupont leisten
- JP2, JP3: value Jumper_2_Open -> Jumper_2_Bridged; footprint Jumper:SolderJumper-2_P1.3mm_Open_TrianglePad1.0x1.5mm -> Connector_PinHeader_2.54mm:PinHeader_1x02_P2.54mm_Vertical
- R1: value 1Meg -> 4.7k
- R2: value 100k -> 4.7k
- R3: value 4.7k -> 1Meg
- R4: value 4.7k -> 100k
- U2: value SN65HVD233 -> ADUM1250ARZ-RL7; footprint Package_SO:SOIC-8_3.9x4.9mm_P1.27mm -> Aktive_Bal_Footprints:ADUM1250ARZ-RL7_R_8_ADI-M
- U3: value ADUM1250ARZ-RL7 -> SN65HVD233; footprint Aktive_Bal_Footprints:ADUM1250ARZ-RL7_R_8_ADI-M -> Package_SO:SOIC-8_3.9x4.9mm_P1.27mm
- U5: value PCA9306DC -> EC1SA16N; footprint Package_SO:VSSOP-8_2.3x2mm_P0.5mm -> Aktive_Bal_Footprints:EC1SA16N
- U6: value EC1SA16N -> PCA9306DC; footprint Aktive_Bal_Footprints:EC1SA16N -> Package_SO:VSSOP-8_2.3x2mm_P0.5mm
- moved U1 278.5 mm to (279.4, 151.8), turned to 90 degrees
- moved J1 271.6 mm to (278.8, 134.6), turned to -90 degrees
- moved C4 261.0 mm to (273.7, 145.7), turned to 90 degrees
- moved R4 259.6 mm to (274.3, 150.5)
- moved J18 258.5 mm to (275.3, 71.6), turned to -90 degrees
- moved FL1 250.5 mm to (268.6, 141.0), turned to 90 degrees
- moved C22 244.4 mm to (139.7, 99.1)
- moved U4 241.7 mm to (255.9, 148.6), turned to 180 degrees
- moved C23 237.7 mm to (139.7, 102.9), turned to 0 degrees
- moved R11 235.0 mm to (130.8, 88.9)
- moved U9 229.6 mm to (133.3, 101.0)
- moved C10 223.8 mm to (231.1, 153.7), turned to 0 degrees
- moved J9 212.3 mm to (229.9, 160.0), turned to 90 degrees
- moved C15 200.8 mm to (212.1, 152.5), turned to 90 degrees
- moved C12 200.6 mm to (222.9, 143.5)
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Connections:
- C11 pad 2: Net-(U5-EN) -> Net-(U6-EN)
- C14 pad 2: Net-(U5-VREF1) -> -5V
- C15 pad 1: GND_float2 -> +5V
- C15 pad 2: -5V -> GND_float2
- C18 pad 1: +5V -> GND_float2
- C18 pad 2: GND_float2 -> +5V
- C19 pad 1: GND_float2 -> +3.3V
- C19 pad 2: +5V -> GND_float2
- C2 pad 1: GNDµ -> +3.3Vµ
- C2 pad 2: +3.3Vµ -> GNDµ
- C21 pad 1: +3.3V -> GND_float2
- C21 pad 2: GND_float2 -> Net-(JP9-A)
- C22 pad 2: Net-(JP4-A) -> Net-(JP8-B)
- C23 pad 2: Net-(JP4-C) -> Net-(JP8-B)
- C24 pad 2: Net-(JP4-C) -> +5V
- C25 pad 2: +5V -> -5V
- C26 pad 1: GND_float2 -> Net-(U14B--)
- C26 pad 2: -5V -> Net-(U14C-+)
- C27 pad 1: Net-(U14B--) -> GND_float2
- C27 pad 2: Net-(U14C-+) -> Net-(U14D-+)
- C28 pad 1: GND_float2 -> Net-(U15-VIN)
- C28 pad 2: Net-(U14D-+) -> GND_float2
- C29 pad 1: Net-(U15-VIN) -> GND_float2
- C29 pad 2: GND_float2 -> Net-(U15-VIN)
- C3 pad 1: +3.3Vµ -> GNDµ
- C3 pad 2: GNDµ -> +3.3Vµ
- C30 pad 1: GND_float2 -> Net-(J23-Pin_1)
- C30 pad 2: Net-(U15-VIN) -> Bal
- C31 pad 1: Net-(Q1-D) -> Bal
- C31 pad 2: Bal -> GND_float2
- J10 pad 1: +3.3V -> SDA3.3
- J11 pad 1: I_Bal_Soll -> GND_float2
- J12 pad 1: Cell16 -> +5V
- J12 pad 2: Cell15 -> -5V
- J13 pad 1: Cell13 -> GND_float2
- J13 pad 2: Cell12 -> +3.3V
- J14 pad 1: Cell10 -> GND_float2
- J14 pad 2: Cell9 -> I_Bal_Soll
- J15 pad 1: Cell7 -> Cell16
- J15 pad 2: Cell6 -> Cell15
- J15 pad 3: Cell5 -> Cell14
- J16 pad 1: Cell4 -> Cell13
- J16 pad 2: Cell3 -> Cell12
- J16 pad 3: Cell2 -> Cell11
- J17 pad 1: Cell1 -> Cell10
- J17 pad 2: Cell0 -> Cell9
- J17 pad 3: unconnected-(J17-Pin_3-Pad3) -> Cell8
- J18 pad 1: I_Bal -> Cell7
- J19 pad 1: V_I_Bal -> Cell4
- J3 pad 1: unconnected-(J3-Pin_1-Pad1) -> CANL
- J3 pad 2: unconnected-(J3-Pin_2-Pad2) -> CANH
- J4 pad 1: SDA5 -> SCLµC
- J4 pad 2: SCL5 -> SCLµC
- J5 pad 1: unconnected-(J5-B12-Pad1) -> SDA5
- J5 pad 2: unconnected-(J5-B13-Pad2) -> SCL5
- J6 pad 1: SDA5 -> +3.3Vµ
- J6 pad 2: SCL5 -> GNDµ
- J7 pad 1: +12V -> unconnected-(J7-B12-Pad1)
- J7 pad 2: GND_float2 -> unconnected-(J7-B13-Pad2)
- J8 pad 1: SDA3.3 -> Net-(J8-Pin_1)
- J8 pad 2: SCL3.3 -> Net-(J8-Pin_2)
- J9 pad 1: +5V -> +12V
- J9 pad 2: -5V -> GND_float2
- JP2 pad 2: SDA3.3 -> Net-(J8-Pin_1)
- JP3 pad 2: SCL3.3 -> Net-(J8-Pin_2)
- JP4 pad 1: Net-(JP4-A) -> GND_float2
- JP4 pad 3: +3.3V -> +5V
- Q1 pad 3: Net-(Q1-D) -> Net-(J23-Pin_1)
- R1 pad 1: GNDµ -> SCLµC
- R1 pad 2: Net-(J2-SHIELD) -> +3.3Vµ
- R10 pad 2: Net-(U5-VREF1) -> +3.3V
- R104 pad 2: Net-(Q1-D) -> Net-(J23-Pin_1)
- R11 pad 2: Net-(JP4-A) -> Net-(JP9-A)
- R2 pad 1: enable -> SCLµC
- R2 pad 2: Bat_GND -> +3.3Vµ
- R3 pad 1: SCLµC -> GNDµ
- R3 pad 2: +3.3Vµ -> Net-(J2-SHIELD)
- R4 pad 1: SDAµC -> enable
- R4 pad 2: +3.3Vµ -> Bat_GND
- R8 pad 1: Net-(U5-EN) -> Net-(U6-EN)
- R9 pad 2: Net-(U5-VREF1) -> +3.3V
- U15 pad 4: Net-(Q1-D) -> Net-(J23-Pin_1)
- U2 pad 1: D -> +3.3Vµ
- U2 pad 2: GNDµ -> SCLµC
- U2 pad 3: +3.3Vµ -> SCLµC
- U2 pad 4: R -> GNDµ
- U2 pad 5: GNDµ -> GND_float2
- U2 pad 6: CANL -> SCL5
- U2 pad 7: CANH -> SDA5
- U2 pad 8: GNDµ -> +5V
- U3 pad 1: +3.3Vµ -> TX
- U3 pad 2: SDAµC -> GNDµ
- U3 pad 3: SCLµC -> +3.3Vµ
- U3 pad 4: GNDµ -> RX
- U3 pad 5: GND_float2 -> GNDµ
- U3 pad 6: SCL5 -> CANL
- U3 pad 7: SDA5 -> CANH
- U3 pad 8: +5V -> GNDµ
- U5 pad 2: Net-(U5-VREF1) -> +12V
- U5 pad 4: SDA3.3 -> -5V
- U5 pad 5: SDA5 -> GND_float2
- U5 pad 6: SCL5 -> +5V
- U6 pad 2: +12V -> +3.3V
- U6 pad 4: -5V -> SDA3.3
- U6 pad 5: GND_float2 -> Net-(J8-Pin_1)
- U6 pad 6: +5V -> Net-(J8-Pin_2)
- U7 pad 2: GND_float2 -> Net-(JP4-C)
- U7 pad 3: GND_float2 -> Net-(JP5-C)
- U9 pad 3: Net-(JP4-C) -> Net-(JP8-B)
- U9 pad 6: GND_float2 -> Net-(JP8-C)
Routing:
- net Net-(J2-SHIELD): track 27.7 -> 0.00 mm
- net (no net): track 0.00 -> 21.2 mm
- net Net-(Q1-D): track 20.9 -> 0.00 mm
- net Bat_GND: track 15.8 -> 0.00 mm
- net enable: track 4.68 -> 0.00 mm
Other:
- board size 3.3 x 6.6 mm -> 439.5 x 254.5 mm
- board text added: "CAN-Anbindung mit Sub-D-Stecker, Tranceiver, STM32"
- board text added: "I2C-Kram"
- board text added: "Leistungsmosfets"
- board text added: "Spannungsversorgungen"

Commit message: neuer stand
Parts:
- removed C32: 47µ, Capacitor_SMD:CP_Elec_5x5.3
- added U8: LM1117MP-3.3, Package_TO_SOT_SMD:SOT-223-3_TabPin2, F.Cu at (123.7, 100.8)
- moved C6 235.9 mm to (247.5, 154.1)
- moved C9 228.3 mm to (241.5, 152.0)
- moved C8 212.5 mm to (241.5, 156.0)
- moved C20 154.7 mm to (123.5, 108.5)
- moved JP4 147.4 mm to (178.7, 55.4)
- moved J11 146.4 mm to (179.2, 40.9)
- moved JP5 102.7 mm to (178.2, 62.9)
- moved C25 100.8 mm to (31.5, 189.0)
- moved C18 88.0 mm to (185.2, 54.4)
- moved J4 66.7 mm to (48.5, 47.5)
- moved J21 63.7 mm to (46.2, 189.5)
- moved J22 63.7 mm to (50.8, 189.5)
- moved J23 63.7 mm to (55.4, 189.5)
- moved J24 63.7 mm to (60.0, 189.5)
- moved J13 47.4 mm to (125.0, 113.5)
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Connections:
- Q10_H1 pad 5_6_7_8: (no net) -> Bal
- Q10_L1 pad 5_6_7_8: (no net) -> Cell9
- Q11_H1 pad 5_6_7_8: (no net) -> Bal
- Q11_L1 pad 5_6_7_8: (no net) -> Cell10
- Q12_H1 pad 5_6_7_8: (no net) -> Bal
- Q12_L1 pad 5_6_7_8: (no net) -> Cell11
- Q13_H1 pad 5_6_7_8: (no net) -> Bal
- Q13_L1 pad 5_6_7_8: (no net) -> Cell12
- Q14_H1 pad 5_6_7_8: (no net) -> Bal
- Q14_L1 pad 5_6_7_8: (no net) -> Cell13
- Q15_H1 pad 5_6_7_8: (no net) -> Bal
- Q15_L1 pad 5_6_7_8: (no net) -> Cell14
- Q16_H1 pad 5_6_7_8: (no net) -> Bal
- Q16_L1 pad 5_6_7_8: (no net) -> Cell15
- Q1_H1 pad 5_6_7_8: (no net) -> Bal
- Q1_L1 pad 5_6_7_8: (no net) -> Cell0
- Q2_H1 pad 5_6_7_8: (no net) -> Bal
- Q2_L1 pad 5_6_7_8: (no net) -> Cell1
- Q3_H1 pad 5_6_7_8: (no net) -> Bal
- Q3_L1 pad 5_6_7_8: (no net) -> Cell2
- Q4_H1 pad 5_6_7_8: (no net) -> Bal
- Q4_L1 pad 5_6_7_8: (no net) -> Cell3
- Q5_H1 pad 5_6_7_8: (no net) -> Bal
- Q5_L1 pad 5_6_7_8: (no net) -> Cell4
- Q6_H1 pad 5_6_7_8: (no net) -> Bal
- Q6_L1 pad 5_6_7_8: (no net) -> Cell5
- Q7_H1 pad 5_6_7_8: (no net) -> Bal
- Q7_L1 pad 5_6_7_8: (no net) -> Cell6
- Q8_H1 pad 5_6_7_8: (no net) -> Bal
- Q8_L1 pad 5_6_7_8: (no net) -> Cell7
- Q9_H1 pad 5_6_7_8: (no net) -> Bal
- Q9_L1 pad 5_6_7_8: (no net) -> Cell8
Other:
- board size 439.5 x 254.5 mm -> 6.6 x 3.3 mm
- board text added: "OPV mit Regelkreis"
- board text added: "Port Expander"
- board text removed: "+12 GNDf"
- board text removed: "+3.3"
- board text removed: "-5 +5"
