File: Aktive_Balancing/KiCAD/Aktive_Bal/Aktive_Bal.kicad_pcb (KiCad board)
At the start: 4 copper layers, 6.6 x 3.3 mm, 221 parts, among them J1 Screw_Terminal_01x02, J10 Conn_01x02_Pin, J11 Conn_01x02_Pin, J12 Conn_01x02_Pin, J13 Conn_01x02_Pin, J14 Conn_01x02_Pin, J15 Screw_Terminal_01x03, J16 Screw_Terminal_01x03, J17 Screw_Terminal_01x03, J18 Screw_Terminal_01x03, J19 Screw_Terminal_01x03, J2 A-DF_09_A_KG-T4S, J20 Screw_Terminal_01x03, J21 Conn_01x02_Pin, J22 Conn_01x02_Pin, J23 Conn_01x02_Pin, J24 Conn_01x02_Pin, J3 Conn_01x02_Pin, J4 Conn_01x02_Pin, J5 Conn_01x02_Pin, J6 Conn_01x02_Pin, J7 Sockel_BluePill, J8 Conn_01x02_Pin, J9 Conn_01x02_Pin, Q1 BSS316NH6327XTSA1, Q10_H1 NTTFS6H888NL, Q10_L1 NTTFS6H888NL, Q11_H1 NTTFS6H888NL, Q11_L1 NTTFS6H888NL, Q12_H1 NTTFS6H888NL, Q12_L1 NTTFS6H888NL, Q13_H1 NTTFS6H888NL, Q13_L1 NTTFS6H888NL, Q14_H1 NTTFS6H888NL, Q14_L1 NTTFS6H888NL, Q15_H1 NTTFS6H888NL, Q15_L1 NTTFS6H888NL, Q16_H1 NTTFS6H888NL, Q16_L1 NTTFS6H888NL, Q1_H1 NTTFS6H888NL, Q1_L1 NTTFS6H888NL, Q2_H1 NTTFS6H888NL, Q2_L1 NTTFS6H888NL, Q3_H1 NTTFS6H888NL, Q3_L1 NTTFS6H888NL, Q4_H1 NTTFS6H888NL, Q4_L1 NTTFS6H888NL, Q5_H1 NTTFS6H888NL, Q5_L1 NTTFS6H888NL, Q6_H1 NTTFS6H888NL, Q6_L1 NTTFS6H888NL, Q7_H1 NTTFS6H888NL, Q7_L1 NTTFS6H888NL, Q8_H1 NTTFS6H888NL, Q8_L1 NTTFS6H888NL, Q9_H1 NTTFS6H888NL, Q9_L1 NTTFS6H888NL, U1 RFP12N10L, U10 LTV-847S, U11 LTV-847S, U12 LTV-847S, U13 LTV-847S, U14 TL084, U15 LM2596S-ADJ, U2 ADUM1250ARZ-RL7, U3 SN65HVD233, U4 SCW20C-12, U5 EC1SA16N, U6 PCA9306DC, U7 PCF8575CDB, U8 LM1117IMPX_3_3_NOPB, U8 LM1117MP-3.3, U9 MCP4725xxx-xCH

Commit message: Bisschen sortiert und so
Parts:
- removed J8: Conn_01x02_Pin, Connector_PinHeader_2.54mm:PinHeader_1x02_P2.54mm_Vertical
- removed the U8 at (200.0, 156.8)
- moved J14 136.0 mm to (16.5, 73.8)
- moved C23 122.8 mm to (20.2, 74.2), turned to -90 degrees
- moved C22 118.8 mm to (23.5, 74.2), turned to -90 degrees
- moved JP8 116.6 mm to (16.5, 79.8)
- moved U9 108.5 mm to (28.4, 73.5)
- moved J10 103.4 mm to (16.0, 88.5), turned to 180 degrees
- moved U8 100.8 mm to (217.2, 138.3), turned to 90 degrees
- moved C20 100.0 mm to (215.6, 147.5), turned to 180 degrees
- moved J13 98.2 mm to (214.5, 154.0), turned to 180 degrees
- moved C21 95.3 mm to (40.0, 90.2), turned to 0 degrees
- moved R10 92.2 mm to (28.1, 82.0), turned to 180 degrees
- moved JP9 92.1 mm to (43.7, 86.2), turned to 90 degrees
- moved C19 91.9 mm to (215.6, 144.5), turned to 180 degrees
- moved R9 90.2 mm to (28.1, 78.5), turned to 180 degrees
- moved C13 89.8 mm to (28.0, 85.5), turned to 180 degrees
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Connections:
- J4 pad 1: SCLµC -> SDAµC
- J7 pad 15: SCLµC -> SDAµC
- R2 pad 1: SCLµC -> SDAµC
- U2 pad 2: SCLµC -> SDAµC
