File: Aktive_Balancing/KiCAD/Aktive_Bal/power_mosfet.kicad_sch (KiCad schematic)
At the start: 118 parts, among them J10 Screw_Terminal_01x17, Q10_H1 NTTFS6H888NL, Q10_L1 NTTFS6H888NL, Q11_H1 NTTFS6H888NL, Q11_L1 NTTFS6H888NL, Q12_H1 NTTFS6H888NL, Q12_L1 NTTFS6H888NL, Q13_H1 NTTFS6H888NL, Q13_L1 NTTFS6H888NL, Q14_H1 NTTFS6H888NL, Q14_L1 NTTFS6H888NL, Q15_H1 NTTFS6H888NL, Q15_L1 NTTFS6H888NL, Q16_H1 NTTFS6H888NL, Q16_L1 NTTFS6H888NL, Q1_H1 NTTFS6H888NL, Q1_L1 NTTFS6H888NL, Q2_H1 NTTFS6H888NL, Q2_L1 NTTFS6H888NL, Q3_H1 NTTFS6H888NL, Q3_L1 NTTFS6H888NL, Q4_H1 NTTFS6H888NL, Q4_L1 NTTFS6H888NL, Q5_H1 NTTFS6H888NL, Q5_L1 NTTFS6H888NL, Q6_H1 NTTFS6H888NL, Q6_L1 NTTFS6H888NL, Q7_H1 NTTFS6H888NL, Q7_L1 NTTFS6H888NL, Q8_H1 NTTFS6H888NL, Q8_L1 NTTFS6H888NL, Q9_H1 NTTFS6H888NL, Q9_L1 NTTFS6H888NL, U10 LTV-847S, U11 LTV-847S, U12 LTV-847S, U9 LTV-847S

Commit message: kicad
Connections:
- net B1: now also R22.1; no longer U9.2
- net B10: now also R32.1; no longer U11.4
- net B11: now also R33.1; no longer U11.6
- net B12: now also R34.1; no longer U11.8
- net B13: now also R35.1; no longer U12.2
- net B14: now also R36.1; no longer U12.4
- net B15: now also R37.1; no longer U12.6
- net B16: now also R38.1; no longer U12.8
- net B2: now also R23.1; no longer U9.4
- net B3: now also R24.1; no longer U9.6
- net B4: now also R26.1; no longer U9.8
- net B5: now also R27.1; no longer U10.2
- net B6: now also R28.1; no longer U10.4
- net B7: now also R29.1; no longer U10.6
- net B8: now also R30.1; no longer U10.8
- net B9: now also R31.1; no longer U11.2
- net Cell0: now also J10.17 (Pin_17), Q16_L1.5 (D), Q16_L1.6 (D), Q16_L1.7 (D), Q16_L1.8 (D); no longer J10.1 (Pin_1), Q1_H1.1 (S), Q1_H1.2 (S), Q1_H1.3 (S)
- net Cell1: now also J10.16 (Pin_16), Q15_L1.5 (D), Q15_L1.6 (D), Q15_L1.7 (D), Q15_L1.8 (D), Q16_H1.1 (S), Q16_H1.2 (S), Q16_H1.3 (S); no longer J10.2 (Pin_2), Q1_L1.5 (D), Q1_L1.6 (D), Q1_L1.7 (D), Q1_L1.8 (D), Q2_H1.1 (S), Q2_H1.2 (S), Q2_H1.3 (S)
- net Cell10: now also J10.7 (Pin_7), Q6_L1.5 (D), Q6_L1.6 (D), Q6_L1.7 (D), Q6_L1.8 (D), Q7_H1.1 (S), Q7_H1.2 (S), Q7_H1.3 (S); no longer J10.11 (Pin_11), Q10_L1.5 (D), Q10_L1.6 (D), Q10_L1.7 (D), Q10_L1.8 (D), Q11_H1.1 (S), Q11_H1.2 (S), Q11_H1.3 (S)
- net Cell11: now also J10.6 (Pin_6), Q5_L1.5 (D), Q5_L1.6 (D), Q5_L1.7 (D), Q5_L1.8 (D), Q6_H1.1 (S), Q6_H1.2 (S), Q6_H1.3 (S); no longer J10.12 (Pin_12), Q11_L1.5 (D), Q11_L1.6 (D), Q11_L1.7 (D), Q11_L1.8 (D), Q12_H1.1 (S), Q12_H1.2 (S), Q12_H1.3 (S)
- net Cell12: now also J10.5 (Pin_5), Q4_L1.5 (D), Q4_L1.6 (D), Q4_L1.7 (D), Q4_L1.8 (D), Q5_H1.1 (S), Q5_H1.2 (S), Q5_H1.3 (S); no longer J10.13 (Pin_13), Q12_L1.5 (D), Q12_L1.6 (D), Q12_L1.7 (D), Q12_L1.8 (D), Q13_H1.1 (S), Q13_H1.2 (S), Q13_H1.3 (S)
- net Cell13: now also J10.4 (Pin_4), Q3_L1.5 (D), Q3_L1.6 (D), Q3_L1.7 (D), Q3_L1.8 (D), Q4_H1.1 (S), Q4_H1.2 (S), Q4_H1.3 (S); no longer J10.14 (Pin_14), Q13_L1.5 (D), Q13_L1.6 (D), Q13_L1.7 (D), Q13_L1.8 (D), Q14_H1.1 (S), Q14_H1.2 (S), Q14_H1.3 (S)
- net Cell14: now also J10.3 (Pin_3), Q2_L1.5 (D), Q2_L1.6 (D), Q2_L1.7 (D), Q2_L1.8 (D), Q3_H1.1 (S), Q3_H1.2 (S), Q3_H1.3 (S); no longer J10.15 (Pin_15), Q14_L1.5 (D), Q14_L1.6 (D), Q14_L1.7 (D), Q14_L1.8 (D), Q15_H1.1 (S), Q15_H1.2 (S), Q15_H1.3 (S)
- net Cell15: now also J10.2 (Pin_2), Q1_L1.5 (D), Q1_L1.6 (D), Q1_L1.7 (D), Q1_L1.8 (D), Q2_H1.1 (S), Q2_H1.2 (S), Q2_H1.3 (S); no longer J10.16 (Pin_16), Q15_L1.5 (D), Q15_L1.6 (D), Q15_L1.7 (D), Q15_L1.8 (D), Q16_H1.1 (S), Q16_H1.2 (S), Q16_H1.3 (S)
- net Cell16: now also J10.1 (Pin_1), Q1_H1.1 (S), Q1_H1.2 (S), Q1_H1.3 (S); no longer J10.17 (Pin_17), Q16_L1.5 (D), Q16_L1.6 (D), Q16_L1.7 (D), Q16_L1.8 (D)
- net Cell2: now also J10.15 (Pin_15), Q14_L1.5 (D), Q14_L1.6 (D), Q14_L1.7 (D), Q14_L1.8 (D), Q15_H1.1 (S), Q15_H1.2 (S), Q15_H1.3 (S); no longer J10.3 (Pin_3), Q2_L1.5 (D), Q2_L1.6 (D), Q2_L1.7 (D), Q2_L1.8 (D), Q3_H1.1 (S), Q3_H1.2 (S), Q3_H1.3 (S)
- net Cell3: now also J10.14 (Pin_14), Q13_L1.5 (D), Q13_L1.6 (D), Q13_L1.7 (D), Q13_L1.8 (D), Q14_H1.1 (S), Q14_H1.2 (S), Q14_H1.3 (S); no longer J10.4 (Pin_4), Q3_L1.5 (D), Q3_L1.6 (D), Q3_L1.7 (D), Q3_L1.8 (D), Q4_H1.1 (S), Q4_H1.2 (S), Q4_H1.3 (S)
- net Cell4: now also J10.13 (Pin_13), Q12_L1.5 (D), Q12_L1.6 (D), Q12_L1.7 (D), Q12_L1.8 (D), Q13_H1.1 (S), Q13_H1.2 (S), Q13_H1.3 (S); no longer J10.5 (Pin_5), Q4_L1.5 (D), Q4_L1.6 (D), Q4_L1.7 (D), Q4_L1.8 (D), Q5_H1.1 (S), Q5_H1.2 (S), Q5_H1.3 (S)
- net Cell5: now also J10.12 (Pin_12), Q11_L1.5 (D), Q11_L1.6 (D), Q11_L1.7 (D), Q11_L1.8 (D), Q12_H1.1 (S), Q12_H1.2 (S), Q12_H1.3 (S); no longer J10.6 (Pin_6), Q5_L1.5 (D), Q5_L1.6 (D), Q5_L1.7 (D), Q5_L1.8 (D), Q6_H1.1 (S), Q6_H1.2 (S), Q6_H1.3 (S)
- net Cell6: now also J10.11 (Pin_11), Q10_L1.5 (D), Q10_L1.6 (D), Q10_L1.7 (D), Q10_L1.8 (D), Q11_H1.1 (S), Q11_H1.2 (S), Q11_H1.3 (S); no longer J10.7 (Pin_7), Q6_L1.5 (D), Q6_L1.6 (D), Q6_L1.7 (D), Q6_L1.8 (D), Q7_H1.1 (S), Q7_H1.2 (S), Q7_H1.3 (S)
- net Cell7: now also J10.10 (Pin_10), Q10_H1.1 (S), Q10_H1.2 (S), Q10_H1.3 (S), Q9_L1.5 (D), Q9_L1.6 (D), Q9_L1.7 (D), Q9_L1.8 (D); no longer J10.8 (Pin_8), Q7_L1.5 (D), Q7_L1.6 (D), Q7_L1.7 (D), Q7_L1.8 (D), Q8_H1.1 (S), Q8_H1.2 (S), Q8_H1.3 (S)
- net Cell9: now also J10.8 (Pin_8), Q7_L1.5 (D), Q7_L1.6 (D), Q7_L1.7 (D), Q7_L1.8 (D), Q8_H1.1 (S), Q8_H1.2 (S), Q8_H1.3 (S); no longer J10.10 (Pin_10), Q10_H1.1 (S), Q10_H1.2 (S), Q10_H1.3 (S), Q9_L1.5 (D), Q9_L1.6 (D), Q9_L1.7 (D), Q9_L1.8 (D)
- net GND_float2: now also U10.2, U10.4, U10.6, U10.8, U11.2, U11.4, U11.6, U11.8, U12.2, U12.4, U12.6, U12.8, U9.2, U9.4, U9.6, U9.8
- removed net +5V: R22.1, R23.1, R24.1, R26.1, R27.1, R28.1, R29.1, R30.1, R31.1, R32.1, R33.1, R34.1, R35.1, R36.1, R37.1, R38.1

Commit message: layout
Parts:
- removed J10: Screw_Terminal_01x17, symbol Connector:Screw_Terminal_01x17
- added J10, J11, J12, J13, J7, J8: Screw_Terminal_01x03, TerminalBlock_CUI:TerminalBlock_CUI_TB007-508-03_1x03_P5.08mm_Horizontal, symbol Connector:Screw_Terminal_01x03
- renumbered Q1_L1 to Q15_L1
Connections:
- net Cell0: now also J13.2 (Pin_2)
- net Cell1: now also J13.1 (Pin_1)
- net Cell10: now also J10.1 (Pin_1)
- net Cell11: now also J8.3 (Pin_3)
- net Cell12: now also J8.2 (Pin_2)
- net Cell13: now also J8.1 (Pin_1)
- net Cell14: now also J7.3 (Pin_3)
- net Cell15: now also J7.2 (Pin_2)
- net Cell16: now also J7.1 (Pin_1)
- net Cell2: now also J12.3 (Pin_3)
- net Cell3: now also J12.2 (Pin_2)
- net Cell4: now also J12.1 (Pin_1)
- net Cell5: now also J11.3 (Pin_3)
- net Cell6: now also J11.2 (Pin_2)
- net Cell7: now also J11.1 (Pin_1)
- net Cell8: now also J10.3 (Pin_3)
- net Cell9: now also J10.2 (Pin_2)

Commit message: layout
Parts:
- Q10_H1: renamed from Q7_H1; footprint Aktive_Bal_Footprints:8-WDFN -> Aktive_Bal_Footprints:TRANS_NVTFS5116PLTAG
- Q10_L1: renamed from Q7_L1; footprint Aktive_Bal_Footprints:8-WDFN -> Aktive_Bal_Footprints:TRANS_NVTFS5116PLTAG
- Q11_H1: renamed from Q6_H1; footprint Aktive_Bal_Footprints:8-WDFN -> Aktive_Bal_Footprints:TRANS_NVTFS5116PLTAG
- Q11_L1: renamed from Q6_L1; footprint Aktive_Bal_Footprints:8-WDFN -> Aktive_Bal_Footprints:TRANS_NVTFS5116PLTAG
- Q12_H1: renamed from Q5_H1; footprint Aktive_Bal_Footprints:8-WDFN -> Aktive_Bal_Footprints:TRANS_NVTFS5116PLTAG
- Q12_L1: renamed from Q5_L1; footprint Aktive_Bal_Footprints:8-WDFN -> Aktive_Bal_Footprints:TRANS_NVTFS5116PLTAG
- Q13_H1: renamed from Q4_H1; footprint Aktive_Bal_Footprints:8-WDFN -> Aktive_Bal_Footprints:TRANS_NVTFS5116PLTAG
- Q13_L1: renamed from Q4_L1; footprint Aktive_Bal_Footprints:8-WDFN -> Aktive_Bal_Footprints:TRANS_NVTFS5116PLTAG
- Q14_H1: renamed from Q3_H1; footprint Aktive_Bal_Footprints:8-WDFN -> Aktive_Bal_Footprints:TRANS_NVTFS5116PLTAG
- Q14_L1: renamed from Q3_L1; footprint Aktive_Bal_Footprints:8-WDFN -> Aktive_Bal_Footprints:TRANS_NVTFS5116PLTAG
- Q15_H1: renamed from Q2_H1; footprint Aktive_Bal_Footprints:8-WDFN -> Aktive_Bal_Footprints:TRANS_NVTFS5116PLTAG
- Q15_L1: renamed from Q2_L1; footprint Aktive_Bal_Footprints:8-WDFN -> Aktive_Bal_Footprints:TRANS_NVTFS5116PLTAG
- Q16_H1: renamed from Q1_H1; footprint Aktive_Bal_Footprints:8-WDFN -> Aktive_Bal_Footprints:TRANS_NVTFS5116PLTAG
- Q16_L1, Q2_L1: renamed from Q15_L1; footprint Aktive_Bal_Footprints:8-WDFN -> Aktive_Bal_Footprints:TRANS_NVTFS5116PLTAG
- Q1_H1: renamed from Q16_H1; footprint Aktive_Bal_Footprints:8-WDFN -> Aktive_Bal_Footprints:TRANS_NVTFS5116PLTAG
- Q1_L1: renamed from Q16_L1; footprint Aktive_Bal_Footprints:8-WDFN -> Aktive_Bal_Footprints:TRANS_NVTFS5116PLTAG
- Q2_H1: renamed from Q15_H1; footprint Aktive_Bal_Footprints:8-WDFN -> Aktive_Bal_Footprints:TRANS_NVTFS5116PLTAG
- Q3_H1: renamed from Q14_H1; footprint Aktive_Bal_Footprints:8-WDFN -> Aktive_Bal_Footprints:TRANS_NVTFS5116PLTAG
- Q3_L1: renamed from Q14_L1; footprint Aktive_Bal_Footprints:8-WDFN -> Aktive_Bal_Footprints:TRANS_NVTFS5116PLTAG
- Q4_H1: renamed from Q13_H1; footprint Aktive_Bal_Footprints:8-WDFN -> Aktive_Bal_Footprints:TRANS_NVTFS5116PLTAG
- Q4_L1: renamed from Q13_L1; footprint Aktive_Bal_Footprints:8-WDFN -> Aktive_Bal_Footprints:TRANS_NVTFS5116PLTAG
- Q5_H1: renamed from Q12_H1; footprint Aktive_Bal_Footprints:8-WDFN -> Aktive_Bal_Footprints:TRANS_NVTFS5116PLTAG
- Q5_L1: renamed from Q12_L1; footprint Aktive_Bal_Footprints:8-WDFN -> Aktive_Bal_Footprints:TRANS_NVTFS5116PLTAG
- Q6_H1: renamed from Q11_H1; footprint Aktive_Bal_Footprints:8-WDFN -> Aktive_Bal_Footprints:TRANS_NVTFS5116PLTAG
- Q6_L1: renamed from Q11_L1; footprint Aktive_Bal_Footprints:8-WDFN -> Aktive_Bal_Footprints:TRANS_NVTFS5116PLTAG
- Q7_H1: renamed from Q10_H1; footprint Aktive_Bal_Footprints:8-WDFN -> Aktive_Bal_Footprints:TRANS_NVTFS5116PLTAG
- Q7_L1: renamed from Q10_L1; footprint Aktive_Bal_Footprints:8-WDFN -> Aktive_Bal_Footprints:TRANS_NVTFS5116PLTAG
- Q8_H1: renamed from Q9_H1; footprint Aktive_Bal_Footprints:8-WDFN -> Aktive_Bal_Footprints:TRANS_NVTFS5116PLTAG
- Q8_L1: renamed from Q9_L1; footprint Aktive_Bal_Footprints:8-WDFN -> Aktive_Bal_Footprints:TRANS_NVTFS5116PLTAG
- Q9_H1: renamed from Q8_H1; footprint Aktive_Bal_Footprints:8-WDFN -> Aktive_Bal_Footprints:TRANS_NVTFS5116PLTAG
- Q9_L1: renamed from Q8_L1; footprint Aktive_Bal_Footprints:8-WDFN -> Aktive_Bal_Footprints:TRANS_NVTFS5116PLTAG
- renumbered J7 to J12, J8 to J13, J10 to J14, J11 to J15, J12 to J16, J13 to J17, R22 to R12, R23 to R13, R24 to R14, R26 to R15, R27 to R16, R28 to R17, R29 to R18, R30 to R19, R31 to R20, R32 to R21, R33 to R22, R34 to R23, R35 to R24, R36 to R25, R37 to R26, R38 to R27, R56 to R28, R57 to R29, R58 to R30, R59 to R31, R60 to R32, R61 to R33, R62 to R34, R63 to R35, R64 to R36, R65 to R37, R66 to R38, R67 to R39, R68 to R40, R69 to R41, R70 to R42, R71 to R43, R39 to R44, R41 to R45, R43 to R46, R45 to R47, R47 to R48, R51 to R50, R53 to R51, R40 to R52, R42 to R53, R44 to R54, R46 to R55, R48 to R56, R50 to R57, R52 to R58, R55 to R59, R72 to R60, R74 to R61, R76 to R62, R78 to R63, R80 to R64, R82 to R65, R84 to R66, R86 to R67, R88 to R68, R90 to R69, R92 to R70, R94 to R71, R96 to R72, R98 to R73, R100 to R74, R102 to R75, R73 to R76, R75 to R77, R77 to R78, R81 to R80, R83 to R81, R85 to R82, R87 to R83, R89 to R84, R91 to R85, R93 to R86, R95 to R87, R97 to R88, R99 to R89, R101 to R90, R103 to R91, R54 to R92, U9 to U10, U10 to U11, U11 to U12, U12 to U13
Connections:
- net B1: now also R27.1, R75.1; no longer R12.1, R60.1
- net B10: now also R18.1, R66.1; no longer R21.1, R69.1
- net B11: now also R17.1, R65.1; no longer R22.1, R70.1
- net B12: now also R16.1, R64.1; no longer R23.1, R71.1
- net B13: now also R15.1, R63.1; no longer R24.1, R72.1
- net B14: now also R14.1, R62.1; no longer R25.1, R73.1
- net B15: now also R13.1, R61.1; no longer R26.1, R74.1
- net B16: now also R12.1, R60.1; no longer R27.1, R75.1
- net B2: now also R26.1, R74.1; no longer R13.1, R61.1
- net B3: now also R25.1, R73.1; no longer R14.1, R62.1
- net B4: now also R24.1, R72.1; no longer R15.1, R63.1
- net B5: now also R23.1, R71.1; no longer R16.1, R64.1
- net B6: now also R22.1, R70.1; no longer R17.1, R65.1
- net B7: now also R21.1, R69.1; no longer R18.1, R66.1
- net B8: now also R20.1, R68.1; no longer R19.1, R67.1
- net B9: now also R19.1, R67.1; no longer R20.1, R68.1

Commit message: Schaltung Review + Layout
Schaltung Review + Layout
Parts:
- renumbered J12 to J15, J13 to J16, J14 to J17, J15 to J18, J16 to J19, J17 to J20
Connections:
- no-connect marks 0 -> 1

Commit message: neuer stand
Connections:
- net Bal: now also Q10_H1.5_6_7_8 (D), Q11_H1.5_6_7_8 (D), Q12_H1.5_6_7_8 (D), Q13_H1.5_6_7_8 (D), Q14_H1.5_6_7_8 (D), Q15_H1.5_6_7_8 (D), Q16_H1.5_6_7_8 (D), Q1_H1.5_6_7_8 (D), Q2_H1.5_6_7_8 (D), Q3_H1.5_6_7_8 (D), Q4_H1.5_6_7_8 (D), Q5_H1.5_6_7_8 (D), Q6_H1.5_6_7_8 (D), Q7_H1.5_6_7_8 (D), Q8_H1.5_6_7_8 (D), Q9_H1.5_6_7_8 (D); no longer Q10_H1.5 (D), Q10_H1.6 (D), Q10_H1.7 (D), Q10_H1.8 (D), Q11_H1.5 (D), Q11_H1.6 (D), Q11_H1.7 (D), Q11_H1.8 (D), Q12_H1.5 (D), Q12_H1.6 (D), Q12_H1.7 (D), Q12_H1.8 (D), Q13_H1.5 (D), Q13_H1.6 (D), Q13_H1.7 (D), Q13_H1.8 (D), Q14_H1.5 (D), Q14_H1.6 (D), Q14_H1.7 (D), Q14_H1.8 (D), Q15_H1.5 (D), Q15_H1.6 (D), Q15_H1.7 (D), Q15_H1.8 (D), Q16_H1.5 (D), Q16_H1.6 (D), Q16_H1.7 (D), Q16_H1.8 (D), Q1_H1.5 (D), Q1_H1.6 (D), Q1_H1.7 (D), Q1_H1.8 (D), Q2_H1.5 (D), Q2_H1.6 (D), Q2_H1.7 (D), Q2_H1.8 (D), Q3_H1.5 (D), Q3_H1.6 (D), Q3_H1.7 (D), Q3_H1.8 (D), Q4_H1.5 (D), Q4_H1.6 (D), Q4_H1.7 (D), Q4_H1.8 (D), Q5_H1.5 (D), Q5_H1.6 (D), Q5_H1.7 (D), Q5_H1.8 (D), Q6_H1.5 (D), Q6_H1.6 (D), Q6_H1.7 (D), Q6_H1.8 (D), Q7_H1.5 (D), Q7_H1.6 (D), Q7_H1.7 (D), Q7_H1.8 (D), Q8_H1.5 (D), Q8_H1.6 (D), Q8_H1.7 (D), Q8_H1.8 (D), Q9_H1.5 (D), Q9_H1.6 (D), Q9_H1.7 (D), Q9_H1.8 (D)
- net Cell0: now also Q1_L1.5_6_7_8 (D); no longer Q1_L1.5 (D), Q1_L1.6 (D), Q1_L1.7 (D), Q1_L1.8 (D)
- net Cell1: now also Q2_L1.5_6_7_8 (D); no longer Q2_L1.5 (D), Q2_L1.6 (D), Q2_L1.7 (D), Q2_L1.8 (D)
- net Cell10: now also Q11_L1.5_6_7_8 (D); no longer Q11_L1.5 (D), Q11_L1.6 (D), Q11_L1.7 (D), Q11_L1.8 (D)
- net Cell11: now also Q12_L1.5_6_7_8 (D); no longer Q12_L1.5 (D), Q12_L1.6 (D), Q12_L1.7 (D), Q12_L1.8 (D)
- net Cell12: now also Q13_L1.5_6_7_8 (D); no longer Q13_L1.5 (D), Q13_L1.6 (D), Q13_L1.7 (D), Q13_L1.8 (D)
- net Cell13: now also Q14_L1.5_6_7_8 (D); no longer Q14_L1.5 (D), Q14_L1.6 (D), Q14_L1.7 (D), Q14_L1.8 (D)
- net Cell14: now also Q15_L1.5_6_7_8 (D); no longer Q15_L1.5 (D), Q15_L1.6 (D), Q15_L1.7 (D), Q15_L1.8 (D)
- net Cell15: now also Q16_L1.5_6_7_8 (D); no longer Q16_L1.5 (D), Q16_L1.6 (D), Q16_L1.7 (D), Q16_L1.8 (D)
- net Cell2: now also Q3_L1.5_6_7_8 (D); no longer Q3_L1.5 (D), Q3_L1.6 (D), Q3_L1.7 (D), Q3_L1.8 (D)
- net Cell3: now also Q4_L1.5_6_7_8 (D); no longer Q4_L1.5 (D), Q4_L1.6 (D), Q4_L1.7 (D), Q4_L1.8 (D)
- net Cell4: now also Q5_L1.5_6_7_8 (D); no longer Q5_L1.5 (D), Q5_L1.6 (D), Q5_L1.7 (D), Q5_L1.8 (D)
- net Cell5: now also Q6_L1.5_6_7_8 (D); no longer Q6_L1.5 (D), Q6_L1.6 (D), Q6_L1.7 (D), Q6_L1.8 (D)
- net Cell6: now also Q7_L1.5_6_7_8 (D); no longer Q7_L1.5 (D), Q7_L1.6 (D), Q7_L1.7 (D), Q7_L1.8 (D)
- net Cell7: now also Q8_L1.5_6_7_8 (D); no longer Q8_L1.5 (D), Q8_L1.6 (D), Q8_L1.7 (D), Q8_L1.8 (D)
- net Cell8: now also Q9_L1.5_6_7_8 (D); no longer Q9_L1.5 (D), Q9_L1.6 (D), Q9_L1.7 (D), Q9_L1.8 (D)
- net Cell9: now also Q10_L1.5_6_7_8 (D); no longer Q10_L1.5 (D), Q10_L1.6 (D), Q10_L1.7 (D), Q10_L1.8 (D)

Commit message: Layout kompakter gemacht
Ich habe die Sektion mit dem Mosfets gemacht. Weber hat es nicht anders gewollt...
Parts:
- J15, J16, J17, J18, J19, J20: footprint TerminalBlock_CUI:TerminalBlock_CUI_TB007-508-03_1x03_P5.08mm_Horizontal -> TerminalBlock_4Ucon:TerminalBlock_4Ucon_1x03_P3.50mm_Horizontal
Changed lines of the file:
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@@
 			)
 		)
-		(property "Footprint" "TerminalBlock_CUI:TerminalBlock_CUI_TB007-508-03_1x03_P5.08mm_Horizontal"
+		(property "Footprint" "TerminalBlock_4Ucon:TerminalBlock_4Ucon_1x03_P3.50mm_Horizontal"
 			(at 203.2 57.15 0)
 			(hide yes)
@@
 			)
 		)
-		(property "Footprint" "TerminalBlock_CUI:TerminalBlock_CUI_TB007-508-03_1x03_P5.08mm_Horizontal"
+		(property "Footprint" "TerminalBlock_4Ucon:TerminalBlock_4Ucon_1x03_P3.50mm_Horizontal"
 			(at 203.2 49.53 0)
 			(hide yes)
@@
 			)
 		)
-		(property "Footprint" "TerminalBlock_CUI:TerminalBlock_CUI_TB007-508-03_1x03_P5.08mm_Horizontal"
+		(property "Footprint" "TerminalBlock_4Ucon:TerminalBlock_4Ucon_1x03_P3.50mm_Horizontal"
 			(at 203.2 41.91 0)
 			(hide yes)
@@
 			)
 		)
-		(property "Footprint" "TerminalBlock_CUI:TerminalBlock_CUI_TB007-508-03_1x03_P5.08mm_Horizontal"
+		(property "Footprint" "TerminalBlock_4Ucon:TerminalBlock_4Ucon_1x03_P3.50mm_Horizontal"
 			(at 203.2 64.77 0)
 			(hide yes)
@@
 			)
 		)
-		(property "Footprint" "TerminalBlock_CUI:TerminalBlock_CUI_TB007-508-03_1x03_P5.08mm_Horizontal"
+		(property "Footprint" "TerminalBlock_4Ucon:TerminalBlock_4Ucon_1x03_P3.50mm_Horizontal"
 			(at 203.2 34.29 0)
 			(hide yes)
@@
 			)
 		)
-		(property "Footprint" "TerminalBlock_CUI:TerminalBlock_CUI_TB007-508-03_1x03_P5.08mm_Horizontal"
+		(property "Footprint" "TerminalBlock_4Ucon:TerminalBlock_4Ucon_1x03_P3.50mm_Horizontal"
 			(at 203.2 72.39 0)
 			(hide yes)

Commit message: alles neu
Connections:
- net GND_float2: now also R92.2; no longer R92.3, R92.4
- net V_I_Bal: now also Q10_L1.1 (S), Q10_L1.2 (S), Q10_L1.3 (S), Q11_L1.1 (S), Q11_L1.2 (S), Q11_L1.3 (S), Q12_L1.1 (S), Q12_L1.2 (S), Q12_L1.3 (S), Q13_L1.1 (S), Q13_L1.2 (S), Q13_L1.3 (S), Q14_L1.1 (S), Q14_L1.2 (S), Q14_L1.3 (S), Q15_L1.1 (S), Q15_L1.2 (S), Q15_L1.3 (S), Q16_L1.1 (S), Q16_L1.2 (S), Q16_L1.3 (S), Q1_L1.1 (S), Q1_L1.2 (S), Q1_L1.3 (S), Q2_L1.1 (S), Q2_L1.2 (S), Q2_L1.3 (S), Q3_L1.1 (S), Q3_L1.2 (S), Q3_L1.3 (S), Q4_L1.1 (S), Q4_L1.2 (S), Q4_L1.3 (S), Q5_L1.1 (S), Q5_L1.2 (S), Q5_L1.3 (S), Q6_L1.1 (S), Q6_L1.2 (S), Q6_L1.3 (S), Q7_L1.1 (S), Q7_L1.2 (S), Q7_L1.3 (S), Q8_L1.1 (S), Q8_L1.2 (S), Q8_L1.3 (S), Q9_L1.1 (S), Q9_L1.2 (S), Q9_L1.3 (S), R92.1; no longer R92.2
Changed lines of the file:
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@@
 	)
 	(junction
+		(at 331.47 232.41)
+		(diameter 0)
+		(color 0 0 0 0)
+	)
+	(junction
 		(at 271.78 31.75)
 		(diameter 0)
@@
 	(wire
 		(pts
-			(xy 334.01 234.95) (xy 337.82 234.95)
+			(xy 331.47 232.41) (xy 335.28 232.41)
 		)
 		(stroke
@@
 	(global_label "V_I_Bal"
 		(shape output)
-		(at 337.82 234.95 0)
+		(at 335.28 232.41 0)
 		(fields_autoplaced yes)
 		(effects
@@
 		)
 		(property "Intersheetrefs" "${INTERSHEET_REFS}"
-			(at 347.518 234.95 0)
+			(at 344.978 232.41 0)
 			(hide yes)
 			(show_name no)
@@
 			)
 		)
-		(pin "3"
-		)
 		(pin "2"
 		)
-		(pin "4"
-		)
 		(pin "1"
 		)
@@
 					(unit 1)
 				)
-			)
-		)
-	)
-	(symbol
-		(lib_id "power:GND")
-		(at 334.01 240.03 90)
-		(unit 1)
-		(body_style 1)
-		(exclude_from_sim no)
-		(in_bom yes)
-		(on_board yes)
-		(in_pos_files yes)
-		(dnp no)
-		(property "Reference" "#PWR0109"
-			(at 340.36 240.03 0)
-			(hide yes)
-			(show_name no)
-			(do_not_autoplace no)
-			(effects
-				(font
-					(size 1.27 1.27)
-				)
-			)
-		)
-		(property "Value" "GND_float2"
-			(at 337.566 240.03 90)
-			(show_name no)
-			(do_not_autoplace no)
-			(effects
-				(font
-					(size 1.27 1.27)
-				)
-				(justify right)
-			)
-		)
-		(property "Footprint" ""
-			(at 334.01 240.03 0)
-			(hide yes)
-			(show_name no)
-			(do_not_autoplace no)
-			(effects
-				(font
-					(size 1.27 1.27)
-				)
-			)
-		)
-		(property "Datasheet" ""
-			(at 334.01 240.03 0)
-			(hide yes)
-			(show_name no)
-			(do_not_autoplace no)
-			(effects
-				(font
-					(size 1.27 1.27)
-				)
-			)
-		)
-		(property "Description" "Power symbol creates a global label with name \"GND\" , ground"
-			(at 334.01 240.03 0)
-			(hide yes)
-			(show_name no)
-			(do_not_autoplace no)
-			(effects
-				(font
-					(size 1.27 1.27)
-				)
-			)
-		)
-		(pin "1"
-		)
-		(instances
-			(project "Aktive_Bal"
-				(path "/7c40c112-cd2b-4a48-9744-14a65613b3b5/45fa0e45-d26c-4c22-a735-03b29ef7d197"
-					(reference "#PWR0109")
-					(unit 1)
-				)

Commit message: review
Changed lines of the file:
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@@
 	)
 	(junction
+		(at 331.47 243.84)
+		(diameter 0)
+		(color 0 0 0 0)
+	)
+	(junction
 		(at 271.78 120.65)
 		(diameter 0)
@@
 	(wire
 		(pts
+			(xy 331.47 246.38) (xy 331.47 243.84)
+		)
+		(stroke
+			(width 0)
+			(type default)
+		)
+	)
+	(wire
+		(pts
 			(xy 39.37 209.55) (xy 52.07 209.55)
 		)
@@
 	(wire
 		(pts
+			(xy 335.28 243.84) (xy 331.47 243.84)
+		)
+		(stroke
+			(width 0)
+			(type default)
+		)
+	)
+	(wire
+		(pts
 			(xy 190.5 57.15) (xy 198.12 57.15)
 		)
@@
 	(wire
 		(pts
+			(xy 331.47 243.84) (xy 331.47 242.57)
+		)
+		(stroke
+			(width 0)
+			(type default)
+		)
+	)
+	(wire
+		(pts
 			(xy 146.05 224.79) (xy 148.59 224.79)
 		)
@@
 		)
 	)
+	(global_label "GNDShunt"
+		(shape input)
+		(at 335.28 243.84 0)
+		(fields_autoplaced yes)
+		(effects
+			(font
+				(size 1.27 1.27)
+			)
+			(justify left)
+		)
+		(property "Intersheetrefs" "${INTERSHEET_REFS}"
+			(at 347.5179 243.84 0)
+			(hide yes)
+			(show_name no)
+			(do_not_autoplace no)
+			(effects
+				(font
+					(size 1.27 1.27)
+				)
+				(justify left)
+			)
+		)
+	)
 	(global_label "Cell8"
 		(shape input)
@@
 	(symbol
 		(lib_id "power:GND")
-		(at 331.47 242.57 0)
+		(at 331.47 246.38 0)
 		(unit 1)
 		(body_style 1)
@@
 		(dnp no)
 		(property "Reference" "#PWR0108"
-			(at 331.47 248.92 0)
+			(at 331.47 252.73 0)
 			(hide yes)
 			(show_name no)
@@
 		)
 		(property "Value" "GND_float2"
-			(at 344.17 244.348 0)
+			(at 344.17 248.158 0)
 			(show_name no)
 			(do_not_autoplace no)
@@
 		)
 		(property "Footprint" ""
-			(at 331.47 242.57 0)
+			(at 331.47 246.38 0)
 			(hide yes)
 			(show_name no)
@@
 		)
 		(property "Datasheet" ""
-			(at 331.47 242.57 0)
+			(at 331.47 246.38 0)
 			(hide yes)
 			(show_name no)
@@
 		)
 		(property "Description" "Power symbol creates a global label with name \"GND\" , ground"
-			(at 331.47 242.57 0)
+			(at 331.47 246.38 0)
 			(hide yes)
 			(show_name no)
