File: Aktive_Balancing/KiCAD/Aktive_Bal/power_mosfet.kicad_sch (KiCad schematic)
At the start: 123 parts, among them J15 Screw_Terminal_01x03, J16 Screw_Terminal_01x03, J17 Screw_Terminal_01x03, J18 Screw_Terminal_01x03, J19 Screw_Terminal_01x03, J20 Screw_Terminal_01x03, Q10_H1 NTTFS6H888NL, Q10_L1 NTTFS6H888NL, Q11_H1 NTTFS6H888NL, Q11_L1 NTTFS6H888NL, Q12_H1 NTTFS6H888NL, Q12_L1 NTTFS6H888NL, Q13_H1 NTTFS6H888NL, Q13_L1 NTTFS6H888NL, Q14_H1 NTTFS6H888NL, Q14_L1 NTTFS6H888NL, Q15_H1 NTTFS6H888NL, Q15_L1 NTTFS6H888NL, Q16_H1 NTTFS6H888NL, Q16_L1 NTTFS6H888NL, Q1_H1 NTTFS6H888NL, Q1_L1 NTTFS6H888NL, Q2_H1 NTTFS6H888NL, Q2_L1 NTTFS6H888NL, Q3_H1 NTTFS6H888NL, Q3_L1 NTTFS6H888NL, Q4_H1 NTTFS6H888NL, Q4_L1 NTTFS6H888NL, Q5_H1 NTTFS6H888NL, Q5_L1 NTTFS6H888NL, Q6_H1 NTTFS6H888NL, Q6_L1 NTTFS6H888NL, Q7_H1 NTTFS6H888NL, Q7_L1 NTTFS6H888NL, Q8_H1 NTTFS6H888NL, Q8_L1 NTTFS6H888NL, Q9_H1 NTTFS6H888NL, Q9_L1 NTTFS6H888NL, U10 LTV-847S, U11 LTV-847S, U12 LTV-847S, U13 LTV-847S

Commit message: Vorläufige finale Version
Diese Version soll in die Fertigung gehen.
Parts:
- added R202: 0, Resistor_SMD:R_0805_2012Metric, symbol Device:R
Connections:
- net GND_float2: now also R202.1; no longer R92.2
- new net V_Shunt_Low: R202.2, R92.2
Changed lines of the file:
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@@
 	)
 	(junction
-		(at 331.47 243.84)
-		(diameter 0)
-		(color 0 0 0 0)
-	)
-	(junction
 		(at 271.78 120.65)
 		(diameter 0)
@@
 	)
 	(junction
+		(at 331.47 243.84)
+		(diameter 0)
+		(color 0 0 0 0)
+	)
+	(junction
 		(at 331.47 138.43)
 		(diameter 0)
@@
 	(wire
 		(pts
-			(xy 331.47 246.38) (xy 331.47 243.84)
-		)
-		(stroke
-			(width 0)
-			(type default)
-		)
-	)
-	(wire
-		(pts
 			(xy 39.37 209.55) (xy 52.07 209.55)
 		)
@@
 	(wire
 		(pts
+			(xy 331.47 245.11) (xy 331.47 243.84)
+		)
+		(stroke
+			(width 0)
+			(type default)
+		)
+	)
+	(wire
+		(pts
 			(xy 96.52 138.43) (xy 96.52 140.97)
 		)
@@
 	(wire
 		(pts
+			(xy 331.47 243.84) (xy 331.47 242.57)
+		)
+		(stroke
+			(width 0)
+			(type default)
+		)
+	)
+	(wire
+		(pts
 			(xy 271.78 69.85) (xy 271.78 73.66)
 		)
@@
 	(wire
 		(pts
-			(xy 335.28 243.84) (xy 331.47 243.84)
-		)
-		(stroke
-			(width 0)
-			(type default)
-		)
-	)
-	(wire
-		(pts
 			(xy 190.5 57.15) (xy 198.12 57.15)
 		)
@@
 	(wire
 		(pts
+			(xy 331.47 243.84) (xy 340.36 243.84)
+		)
+		(stroke
+			(width 0)
+			(type default)
+		)
+	)
+	(wire
+		(pts
 			(xy 135.89 172.72) (xy 138.43 172.72)
 		)
@@
 	(wire
 		(pts
-			(xy 331.47 243.84) (xy 331.47 242.57)
+			(xy 146.05 224.79) (xy 148.59 224.79)
 		)
 		(stroke
@@
 	(wire
 		(pts
-			(xy 146.05 224.79) (xy 148.59 224.79)
+			(xy 88.9 168.91) (xy 128.27 168.91)
 		)
 		(stroke
@@
 	(wire
 		(pts
-			(xy 88.9 168.91) (xy 128.27 168.91)
+			(xy 331.47 87.63) (xy 331.47 100.33)
 		)
 		(stroke
@@
 	(wire
 		(pts
-			(xy 331.47 87.63) (xy 331.47 100.33)
+			(xy 331.47 255.27) (xy 331.47 252.73)
 		)
 		(stroke
@@
 		)
 	)
+	(global_label "V_Shunt_Low"
+		(shape output)
+		(at 340.36 243.84 0)
+		(fields_autoplaced yes)
+		(effects
+			(font
+				(size 1.27 1.27)
+			)
+			(justify left)
+		)
+		(property "Intersheetrefs" "${INTERSHEET_REFS}"
+			(at 355.2588 243.84 0)
+			(hide yes)
+			(show_name no)
+			(do_not_autoplace no)
+			(effects
+				(font
+					(size 1.27 1.27)
+				)
+				(justify left)
+			)
+		)
+	)
 	(global_label "Cell1"
 		(shape input)
@@
 		)
 	)
-	(global_label "GNDShunt"
-		(shape input)
-		(at 335.28 243.84 0)
-		(fields_autoplaced yes)
-		(effects
-			(font
-				(size 1.27 1.27)
-			)
-			(justify left)
-		)
-		(property "Intersheetrefs" "${INTERSHEET_REFS}"
-			(at 347.5179 243.84 0)
-			(hide yes)
-			(show_name no)
-			(do_not_autoplace no)
-			(effects
-				(font
-					(size 1.27 1.27)
-				)
-				(justify left)
-			)
-		)
-	)
 	(global_label "Cell8"
 		(shape input)
@@
 		(length 2.54)
 		(shape round)
+		(at 331.47 254 270)
+		(fields_autoplaced yes)
+		(effects
+			(font
+				(size 1.27 1.27)
+			)
+			(justify right bottom)
+		)
+		(property "Netzklasse" "power"
+			(at 334.01 253.3015 90)
+			(show_name no)
+			(do_not_autoplace no)
+			(effects
+				(font
+					(size 1.27 1.27)
+				)
+				(justify left)
+			)
+		)
+		(property "Component Class" ""
+			(at -58.42 40.64 0)
+			(show_name no)
+			(do_not_autoplace no)
+			(effects
+				(font
+					(size 1.27 1.27)
+					(italic yes)
+				)
+			)
+		)
+	)
+	(netclass_flag ""
+		(length 2.54)
+		(shape round)
 		(at 93.98 97.79 0)
 		(fields_autoplaced yes)
@@
 		(length 2.54)
 		(shape round)
+		(at 331.47 245.11 270)
+		(fields_autoplaced yes)
+		(effects
+			(font
+				(size 1.27 1.27)
+			)
+			(justify right bottom)
+		)
+		(property "Netzklasse" "power"
+			(at 334.01 244.4115 90)
+			(show_name no)
+			(do_not_autoplace no)
+			(effects
+				(font
+					(size 1.27 1.27)
+				)
+				(justify left)
+			)
+		)
+		(property "Component Class" ""
+			(at -58.42 31.75 0)
+			(show_name no)
+			(do_not_autoplace no)
+			(effects
+				(font
+					(size 1.27 1.27)
+					(italic yes)
+				)
+			)
+		)
+	)
+	(netclass_flag ""
+		(length 2.54)
+		(shape round)
 		(at 287.02 95.25 0)
 		(effects
@@
 	)
 	(symbol
+		(lib_id "Device:R")
+		(at 331.47 248.92 180)
+		(unit 1)
+		(body_style 1)
+		(exclude_from_sim no)
+		(in_bom yes)
+		(on_board yes)
+		(in_pos_files yes)
+		(dnp no)
+		(property "Reference" "R202"
+			(at 333.756 248.92 90)
+			(show_name no)
+			(do_not_autoplace no)
+			(effects
+				(font
+					(size 1.27 1.27)
+				)
+			)
+		)
+		(property "Value" "0"
+			(at 335.28 248.92 90)
+			(show_name no)
+			(do_not_autoplace no)
+			(effects
+				(font
+					(size 1.27 1.27)
+				)
+			)
+		)
+		(property "Footprint" "Resistor_SMD:R_0805_2012Metric"
+			(at 333.248 248.92 90)
+			(hide yes)
+			(show_name no)
+			(do_not_autoplace no)
+			(effects
+				(font
+					(size 1.27 1.27)
+				)
+			)
+		)
+		(property "Datasheet" ""
+			(at 331.47 248.92 0)
+			(hide yes)
+			(show_name no)
+			(do_not_autoplace no)
+			(effects
+				(font
+					(size 1.27 1.27)
+				)
+			)
+		)
+		(property "Description" "Resistor"
+			(at 331.47 248.92 0)
+			(hide yes)
+			(show_name no)
+			(do_not_autoplace no)
+			(effects
+				(font
+					(size 1.27 1.27)
+				)
+			)
+		)
+		(pin "2"
+		)
+		(pin "1"
+		)
+		(instances
+			(project "Aktive_Bal"
+				(path "/7c40c112-cd2b-4a48-9744-14a65613b3b5/45fa0e45-d26c-4c22-a735-03b29ef7d197"
+					(reference "R202")
+					(unit 1)
+				)
+			)
+		)
+	)
+	(symbol
 		(lib_id "power:GND")
 		(at 39.37 189.23 270)
@@
 	(symbol
 		(lib_id "power:GND")
-		(at 331.47 246.38 0)
+		(at 331.47 255.27 0)
 		(unit 1)
 		(body_style 1)
@@
 		(dnp no)
 		(property "Reference" "#PWR0108"
-			(at 331.47 252.73 0)
+			(at 331.47 261.62 0)
 			(hide yes)
 			(show_name no)
@@
 		)
 		(property "Value" "GND_float2"
-			(at 344.17 248.158 0)
+			(at 344.17 257.048 0)
 			(show_name no)
 			(do_not_autoplace no)
@@
 		)
 		(property "Footprint" ""
-			(at 331.47 246.38 0)
+			(at 331.47 255.27 0)
 			(hide yes)
 			(show_name no)
@@
 		)
 		(property "Datasheet" ""
-			(at 331.47 246.38 0)
+			(at 331.47 255.27 0)
 			(hide yes)
 			(show_name no)
@@
 		)
 		(property "Description" "Power symbol creates a global label with name \"GND\" , ground"
-			(at 331.47 246.38 0)
+			(at 331.47 255.27 0)
 			(hide yes)
 			(show_name no)
