File: BM107/BM107_V6_Layout/Spannungsversorgungen.kicad_sch (KiCad schematic)
At the start: 29 parts, among them U1 R-78K15-0.5, U3 LM317_SOT-223, U4 AD8031, U5 R-78K5.0-0.5, U6 LD1117S33TR_SOT223

Commit message: neuneuenu
Parts:
- gave numbers to parts that had none: 3
- renumbered C9 to C10, C7 to C11, C10 to C12, C11 to C13, C12 to C14, C13 to C15, C14 to C18, C15 to C19, C1 to C3, C3 to C4, C2 to C6, C4 to C7, C6 to C9, R1 to R2, R2 to R3, R3 to R4, R4 to R5, U1 to U4, U3 to U6, U5 to U7, U4 to U8, U6 to U9

Commit message: NEuneuenuenbeuebu
Parts:
- C10: renamed from C8; footprint (none) -> Capacitor_SMD:C_0805_2012Metric
- C11: renamed from C9; value 1u -> 1u Elko; footprint (none) -> Capacitor_SMD:CP_Elec_5x5.3
- C12: renamed from C10; value 10u -> 10u Elko; footprint (none) -> Capacitor_SMD:CP_Elec_5x5.3
- C13: renamed from C11; footprint (none) -> Capacitor_SMD:C_0805_2012Metric
- C14: renamed from C12; footprint (none) -> Capacitor_SMD:C_0805_2012Metric
- C15: renamed from C13; value 10u -> 10u Elko; footprint (none) -> Capacitor_SMD:CP_Elec_5x5.3
- C16: renamed from C14; footprint (none) -> Capacitor_SMD:C_0805_2012Metric
- C17: renamed from C15; value 10u -> 10u Elko; footprint (none) -> Capacitor_SMD:CP_Elec_5x5.3
- C18: renamed from C16; value 10u -> 10u Elko; footprint (none) -> Capacitor_SMD:CP_Elec_5x5.3
- C19: renamed from C17; footprint (none) -> Capacitor_SMD:C_0805_2012Metric
- C20: renamed from C18; value 10u -> 10u Elko; footprint (none) -> Capacitor_SMD:CP_Elec_5x5.3
- C21: renamed from C19; value 10u -> 10u Elko; footprint (none) -> Capacitor_SMD:CP_Elec_5x5.3
- C5: renamed from C3; value 10u -> 10u Elko; footprint (none) -> Capacitor_SMD:CP_Elec_5x5.3
- C6: renamed from C4; footprint (none) -> Capacitor_SMD:C_0805_2012Metric
- C7: renamed from C5; value 10u -> 10u Elko; footprint (none) -> Capacitor_SMD:CP_Elec_5x5.3
- C8: renamed from C6; value 1u -> 1u Elko; footprint (none) -> Capacitor_SMD:CP_Elec_5x5.3
- C9: renamed from C7; footprint (none) -> Capacitor_SMD:C_0805_2012Metric
- R2, R3, R4, R5: footprint (none) -> Resistor_SMD:R_0805_2012Metric
- renumbered U4 to U3, U5 to U4, U6 to U5, U7 to U6, U8 to U7, U9 to U8
Connections:
- net 1.5V renamed +1.5V
