File: BM107/BM107_V6_Layout/Spannungsversorgungen.kicad_sch (KiCad schematic)
At the start: 29 parts, among them U3 R-78K15-0.5, U4 ADR3036, U5 LM317_SOT-223, U6 R-78K5.0-0.5, U7 AD8031, U8 LD1117S33TR_SOT223

Commit message: bm107neuneuneu
Parts:
- R4, R5: value R -> 10k
Connections:
- net +3V renamed +3.0V
Changed lines of the file:
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@@
 		)
 	)
-	(global_label "+3V"
+	(global_label "+3.0V"
 		(shape input)
 		(at 173.99 101.6 90)
@@
 		)
 		(property "Intersheetrefs" "${INTERSHEET_REFS}"
-			(at 173.99 94.7443 90)
-			(hide yes)
-			(show_name no)
-			(do_not_autoplace no)
-			(effects
-				(font
-					(size 1.27 1.27)
-				)
-				(justify left)
-			)
-		)
-	)
-	(global_label "+3V"
+			(at 173.99 92.93 90)
+			(hide yes)
+			(show_name no)
+			(do_not_autoplace no)
+			(effects
+				(font
+					(size 1.27 1.27)
+				)
+				(justify left)
+			)
+		)
+	)
+	(global_label "+3.0V"
 		(shape input)
 		(at 118.11 114.3 0)
@@
 		)
 		(property "Intersheetrefs" "${INTERSHEET_REFS}"
-			(at 124.9657 114.3 0)
+			(at 126.78 114.3 0)
 			(hide yes)
 			(show_name no)
@@
 			)
 		)
-		(property "Value" "R"
+		(property "Value" "10k"
 			(at 176.53 121.9199 0)
 			(show_name no)
@@
 			)
 		)
-		(property "Value" "R"
+		(property "Value" "10k"
 			(at 176.53 111.7599 0)
 			(show_name no)
