File: BM107/BM107_V6_Layout/BM107_V6_Layout.kicad_pcb (KiCad board)
At the start: 2 copper layers, 90 parts, among them J1 PC5930T, J2 PC5930T, J3 WAGO_1_5, J4 DE9_Pins_MountingHoles, J5 PC5930T, J6 PC5930T, J7 Sockel_BluePill, J8 Conn_01x02_Pin, Q1 BSC016N06NS, Q2 BSC016N06NS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

Commit message: bm107 neu
Parts:
- removed R19: 500u, Aktive_Bal_Footprints:CMP-R100-1.0
- added R26: Shunt_BVT-M-R0005, Aktive_Bal_Footprints:Shunt_BVT-M-R0005, F.Cu at (87.0, 109.7)
Changed lines of the file:
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@@
 		)
 	)
+	(footprint "Aktive_Bal_Footprints:Shunt_BVT-M-R0005"
+		(layer "F.Cu")
+		(at 87.001 109.712)
+		(property "Reference" "R26"
+			(at 0.254 -1.524 0)
+			(unlocked yes)
+			(layer "F.SilkS")
+			(effects
+				(font
+					(size 1 1)
+					(thickness 0.1)
+				)
+			)
+		)
+		(property "Value" "Shunt_BVT-M-R0005"
+			(at 0 1 0)
+			(unlocked yes)
+			(layer "F.Fab")
+			(effects
+				(font
+					(size 1 1)
+					(thickness 0.15)
+				)
+			)
+		)
+		(property "Datasheet" ""
+			(at 0 0 0)
+			(unlocked yes)
+			(layer "F.Fab")
+			(hide yes)
+			(effects
+				(font
+					(size 1 1)
+					(thickness 0.15)
+				)
+			)
+		)
+		(property "Description" "Shunt resistor with Kelvin connections"
+			(at 0 0 0)
+			(unlocked yes)
+			(layer "F.Fab")
+			(hide yes)
+			(effects
+				(font
+					(size 1 1)
+					(thickness 0.15)
+				)
+			)
+		)
+		(property ki_fp_filters "R_*Shunt*")
+		(sheetname "/H_Bruecke/")
+		(sheetfile "H_Bruecke.kicad_sch")
+		(units
+			(unit
+				(name "A")
+				(pins "1" "4" "2" "3")
+			)
+		)
+		(attr smd)
+		(duplicate_pad_numbers_are_jumpers no)
+		(fp_line
+			(start -0.025 2)
+			(end 2.225 2)
+			(stroke
+				(width 0.3)
+				(type solid)
+			)
+			(layer "F.Cu")
+		)
+		(fp_line
+			(start 0 0.5)
+			(end 0 2)
+			(stroke
+				(width 0.3)
+				(type solid)
+			)
+			(layer "F.Cu")
+		)
+		(fp_line
+			(start 0 3)
+			(end 2.25 3)
+			(stroke
+				(width 0.3)
+				(type solid)
+			)
+			(layer "F.Cu")
+		)
+		(fp_line
+			(start 0 4.5)
+			(end 0 3)
+			(stroke
+				(width 0.3)
+				(type solid)
+			)
+			(layer "F.Cu")
+		)
+		(fp_rect
+			(start -1.651 -0.762)
+			(end 1.651 5.842)
+			(stroke
+				(width 0.1)
+				(type default)
+			)
+			(fill no)
+			(layer "F.SilkS")
+		)
+		(fp_circle
+			(center -1.143 1.017999)
+			(end -1.017999 1.017999)
+			(stroke
+				(width 0.25)
+				(type solid)
+			)
+			(fill no)
+			(layer "F.SilkS")
+		)
+		(fp_rect
+			(start -1.651 -0.762)
+			(end 1.651 5.85)
+			(stroke
+				(width 0.05)
+				(type default)
+			)
+			(fill no)
+			(layer "F.CrtYd")
+		)
+		(fp_text user "${REFERENCE}"
+			(at 0 2.5 0)
+			(unlocked yes)
+			(layer "F.Fab")
+			(effects
+				(font
+					(size 1 1)
+					(thickness 0.15)
+				)
+			)
+		)
+		(pad "1" smd rect
+			(at 0 0)
+			(size 3 1.25)
+			(layers "F.Cu" "F.Mask" "F.Paste")
+			(net "V_Motor-")
+			(pintype "passive")
+		)
+		(pad "2" smd circle
+			(at 2.25 2)
+			(size 0.3 0.3)
+			(layers "F.Cu" "F.Mask" "F.Paste")
+			(net "IS-")
+			(pintype "passive")
+		)
+		(pad "3" smd circle
+			(at 2.25 3)
+			(size 0.3 0.3)
+			(layers "F.Cu" "F.Mask" "F.Paste")
+			(net "IS+")
+			(pintype "passive")
+		)
+		(pad "4" smd rect
+			(at 0 5.1)
+			(size 3 1.25)
+			(layers "F.Cu" "F.Mask" "F.Paste")
+			(net "Net-(Q4-D)")
+			(pintype "passive")
+		)
+		(embedded_fonts no)
+	)
 	(footprint "Capacitor_SMD:C_0805_2012Metric"
 		(layer "F.Cu")
@@
 		)
 	)
-	(footprint "Aktive_Bal_Footprints:CMP-R100-1.0"
-		(layer "F.Cu")
-		(at 86.211 110.612)
-		(property "Reference" "R19"
-			(at 0.254 -1.524 0)
-			(unlocked yes)
-			(layer "F.SilkS")
-			(effects
-				(font
-					(size 1 1)
-					(thickness 0.1)
-				)
-			)
-		)
-		(property "Value" "500u"
-			(at 0 1 0)
-			(unlocked yes)
-			(layer "F.Fab")
-			(effects
-				(font
-					(size 1 1)
-					(thickness 0.15)
-				)
-			)
-		)
-		(property "Datasheet" ""
-			(at 0 0 0)
-			(unlocked yes)
-			(layer "F.Fab")
-			(hide yes)
-			(effects
-				(font
-					(size 1 1)
-					(thickness 0.15)
-				)
-			)
-		)
-		(property "Description" "Shunt resistor with Kelvin connections"
-			(at 0 0 0)
-			(unlocked yes)
-			(layer "F.Fab")
-			(hide yes)
-			(effects
-				(font
-					(size 1 1)
-					(thickness 0.15)
-				)
-			)
-		)
-		(property ki_fp_filters "R_*Shunt*")
-		(sheetname "/H_Bruecke/")
-		(sheetfile "H_Bruecke.kicad_sch")
-		(units
-			(unit
-				(name "A")
-				(pins "1" "4" "2" "3")
-			)
-		)
-		(attr smd)
-		(duplicate_pad_numbers_are_jumpers no)
-		(fp_line
-			(start 0 0.625)
-			(end 0 2)
-			(stroke
-				(width 0.3)
-				(type solid)
-			)
-			(layer "F.Cu")
-		)
-		(fp_line
-			(start 0 2)
-			(end 2.25 2)
-			(stroke
-				(width 0.3)
-				(type solid)
-			)
-			(layer "F.Cu")
-		)
-		(fp_line
-			(start 0 3)
-			(end 2.25 3)
-			(stroke
-				(width 0.3)
-				(type solid)
-			)
-			(layer "F.Cu")
-		)
-		(fp_line
-			(start 0 4.375)
-			(end 0 3)
-			(stroke
-				(width 0.3)
-				(type solid)
-			)
-			(layer "F.Cu")
-		)
-		(fp_rect
-			(start -1.651 -0.762)
-			(end 1.651 5.842)
-			(stroke
-				(width 0.1)
-				(type default)
-			)
-			(fill no)
-			(layer "F.SilkS")
-		)
-		(fp_circle
-			(center -1.143 1.017999)
-			(end -1.017999 1.017999)
-			(stroke
-				(width 0.25)
-				(type solid)
-			)
-			(fill no)
-			(layer "F.SilkS")
-		)
-		(fp_rect
-			(start -1.651 -0.762)
-			(end 1.651 5.715)
-			(stroke
-				(width 0.05)
-				(type default)
-			)
-			(fill no)
-			(layer "F.CrtYd")
-		)
-		(fp_text user "${REFERENCE}"
-			(at 0 2.5 0)
-			(unlocked yes)
-			(layer "F.Fab")
-			(effects
-				(font
-					(size 1 1)
-					(thickness 0.15)
-				)
-			)
-		)
-		(pad "1" smd rect
-			(at 0 0)
-			(size 3 1.25)
-			(layers "F.Cu" "F.Mask" "F.Paste")
-			(net "V_Motor-")
-			(pintype "passive")
-		)
-		(pad "2" smd circle
-			(at 2.25 2)
-			(size 0.3 0.3)
-			(layers "F.Cu" "F.Mask" "F.Paste")
-			(net "IS-")
-			(pintype "passive")
-		)
-		(pad "3" smd circle
-			(at 2.25 3)
-			(size 0.3 0.3)
-			(layers "F.Cu" "F.Mask" "F.Paste")
-			(net "IS+")
-			(pintype "passive")
-		)
-		(pad "4" smd rect
-			(at 0 5)
-			(size 3 1.25)
-			(layers "F.Cu" "F.Mask" "F.Paste")
-			(net "Net-(Q4-D)")
-			(pintype "passive")
-		)
-		(embedded_fonts no)
-	)
 	(footprint "Capacitor_SMD:CP_Elec_5x5.3"
