File: BM107/BM107_V6_Layout/BM107_V6_Layout.kicad_pcb (KiCad board)
At the start: 2 copper layers, 90 parts, among them J1 WAGO_1_5, J2 PC5930T, J3 PC5930T, J4 DE9_Pins_MountingHoles, J5 PC5930T, J6 PC5930T, J7 Sockel_BluePill, J8 Conn_01x02_Pin, Q1 BSC016N06NS, Q2 BSC016N06NS, Q3 BSC016N06NS, Q4 BSC016N06NS, U1 LT1999-50, U10 UCC27734, U2 SN65HVD233, U3 R-78K15-0.5, U4 ADR3036, U5 LM317_SOT-223, U6 R-78K5.0-0.5, U7 AD8031, U8 LD1117S33TR_SOT223, U9 UCC27734

Commit message: bmschießmichtot
Parts:
- moved J2 230.2 mm to (14.2, 27.5), turned to -90 degrees
- moved J3 204.1 mm to (14.2, 48.2), turned to -90 degrees
- moved J5 154.6 mm to (115.6, 48.1), turned to 90 degrees
- moved C2 135.5 mm to (100.5, 146.5)
- moved C3 135.5 mm to (100.5, 149.5)
- moved C4 135.5 mm to (100.5, 152.5)
- moved J8 135.5 mm to (100.6, 167.5)
- moved JP1 135.5 mm to (100.5, 177.1)
- moved R1 135.5 mm to (100.5, 173.8)
- moved U2 135.5 mm to (102.0, 162.9)
- moved J4 97.0 mm to (92.0, 115.2)
- moved J7 94.2 mm to (110.5, 110.7), turned to 180 degrees
- moved U1 88.5 mm to (75.5, 87.4)
- moved Q3 85.4 mm to (71.1, 25.6), turned to 90 degrees
- moved Q4 83.2 mm to (71.1, 34.5), turned to 90 degrees
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Connections:
- Q2 pad 4: G1 -> G2
- Q3 pad 4: G1 -> G3
- Q4 pad 4: G1 -> G4
- R13 pad 2: G1 -> G3
- R14 pad 2: G1 -> G4
- R7 pad 2: G1 -> G2
Routing:
- net GND: track 0.00 -> 9.11 mm
- added copper zone on F.Cu, net +24V
- added copper zone on F.Cu, net GND
- added copper zone on In1.Cu, net GND
- added copper zone on F.Cu, net Net-(Q4-D)
- added copper zone on F.Cu, net V_Motor+
- added copper zone on F.Cu, net V_Motor-
Other:
- board outline added: 100 x 100 mm
- copper layers 2 -> 4

Commit message: bm107neuneuneu
Parts:
- removed C3: 10p, Capacitor_SMD:C_0805_2012Metric
- added R26: 4k, Resistor_SMD:R_0805_2012Metric, F.Cu at (77.2, 112.1)
- R4, R5: value R -> 10k
- moved R11 136.2 mm to (54.0, 29.2), turned to -90 degrees
- moved R12 135.7 mm to (44.5, 33.2), turned to 90 degrees
- moved C26 135.5 mm to (56.5, 29.2), turned to -90 degrees
- moved C29 132.3 mm to (69.0, 25.2)
- moved R15 128.7 mm to (69.0, 27.8), turned to 180 degrees
- moved C27 127.9 mm to (44.5, 29.2), turned to -90 degrees
- moved C30 123.5 mm to (67.5, 37.2), turned to 180 degrees
- moved D3 122.2 mm to (52.6, 57.1)
- moved D8 120.0 mm to (84.0, 60.0), turned to 180 degrees
- moved R16 118.6 mm to (67.5, 40.8)
- moved D1 116.9 mm to (19.0, 68.5), turned to -90 degrees
- moved D4 115.8 mm to (47.1, 56.1), turned to 90 degrees
- moved C12 113.6 mm to (39.0, 67.2), turned to 90 degrees
- moved D6 112.4 mm to (74.0, 68.5), turned to 90 degrees
- moved D7 110.9 mm to (68.0, 65.5), turned to 180 degrees
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Connections:
- C11 pad 1: +3V -> +3.0V
- C13 pad 1: +3V -> +3.0V
- R4 pad 1: +3V -> +3.0V
- U4 pad 6: +3V -> +3.0V
Other:
- board size 100 x 100 mm -> 78.6 x 100 mm

Commit message: bm107
Parts:
- moved R13 32.4 mm to (67.0, 29.2)
- moved R14 32.1 mm to (63.7, 40.8), turned to 0 degrees
- moved R6 25.1 mm to (53.8, 30.4), turned to 90 degrees
- moved R7 24.0 mm to (50.8, 41.8), turned to 0 degrees
- moved R11 3.22 mm to (56.8, 30.8)
- moved R15 2.00 mm to (71.0, 27.8)
- moved C26 1.95 mm to (57.2, 27.4)
- turned R12 to -90 degrees
Routing:
- net +24V: track 0.00 -> 70.5 mm
- net Sp_A: track 0.00 -> 57.0 mm
- net Sp_B: track 0.00 -> 54.0 mm
- net GND: track 9.11 -> 58.0 mm, vias 0 -> 3
- net CANL: track 0.00 -> 20.5 mm
- net CANH: track 0.00 -> 20.4 mm
- net +3.0V: track 0.00 -> 18.5 mm
- net TX: track 0.00 -> 15.6 mm
- net Net-(Q4-D): track 0.00 -> 12.6 mm
- net RX: track 0.00 -> 11.4 mm
- net G2: track 0.00 -> 4.39 mm, vias 0 -> 1
- net +3.3V: track 0.00 -> 4.14 mm
- net G1: track 0.00 -> 3.60 mm, vias 0 -> 1
- net Net-(C30-Pad2): track 0.00 -> 3.51 mm
- net V_Motor+: track 0.00 -> 3.49 mm
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
Commit message: bm107
Other:
- board text added: "Analog_Signal"
Changed lines of the file:
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@@
+	)
+	(gr_rect
+		(start 74 89.4)
+		(end 90.4 116.2)
+		(stroke
+			(width 0.1)
+			(type default)
+		)
+		(fill no)
+		(layer "F.SilkS")
 	)
 	(gr_rect
@@
 		(layer "Edge.Cuts")
 	)
+	(gr_text "Analog_Signal\n"
+		(at 77.2 118 0)
+		(layer "F.SilkS")
+		(effects
+			(font
+				(size 1 1)
+				(thickness 0.1)
+			)
+			(justify left bottom)
+		)
+	)
 	(segment
 		(start 63.085 25.25)
@@
 		(polygon
 			(pts
-				(xy 16 22) (xy 92.25 22) (xy 92.25 120) (xy 16 120)
+				(xy 16 22) (xy 92.25 22) (xy 92.25 120.02111) (xy 71.467875 119.97933) (xy 71.467833 120) (xy 16 120)
 			)
 		)

Commit message: bm107
Parts:
- Q1, Q2, Q3, Q4: footprint Package_TO_SOT_SMD:TDSON-8-1 -> Aktive_Bal_Footprints:BSC016N06NS

Commit message: bm107 geroutet
Parts:
- moved C28 4.93 mm to (44.6, 61.6), turned to -90 degrees
- moved C34 2.00 mm to (72.8, 58.4), turned to 0 degrees
Routing:
- net +12V: track 0.00 -> 133.4 mm
- net IS-: track 0.00 -> 110.6 mm, vias 0 -> 2
- net IS+: track 0.00 -> 109.1 mm, vias 0 -> 2
- net GND: track 58.0 -> 154.8 mm, vias 3 -> 37
- net G4_IN: track 0.00 -> 93.6 mm, vias 0 -> 1
- net +5V: track 0.00 -> 85.5 mm
- net G3_IN: track 0.00 -> 75.2 mm, vias 0 -> 1
- net +3.3V: track 4.14 -> 77.0 mm, vias 0 -> 2
- net V_Motor-: track 0.00 -> 53.4 mm, vias 0 -> 1
- net G1_IN: track 0.00 -> 47.4 mm, vias 0 -> 1
- net G2_IN: track 0.00 -> 46.9 mm, vias 0 -> 1
- net V_Isense: track 0.00 -> 43.1 mm, vias 0 -> 1
- net G3: track 3.47 -> 45.7 mm, vias 1 -> 2
- net G4: track 3.08 -> 43.0 mm, vias 1 -> 2
- net V_Motor+: track 3.49 -> 41.9 mm, vias 0 -> 1
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