File: BM107/BM107_V6_Layout/BM107_V6_Layout.kicad_sch (KiCad schematic)
At the start: 2 parts, among them J1 Screw_Terminal_01x02, J2 Screw_Terminal_01x02

Commit message: neuneuenu
Parts:
- added C1: 22u, symbol Device:C_Polarized
Connections:
- net +24V: now also C1.1
- net GND: now also C1.2
Other:
- added sheet Bluepill (Bluepill.kicad_sch)
Changed lines of the file:
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@@
+		)
+	)
+	(junction
+		(at 36.83 36.83)
+		(diameter 0)
+		(color 0 0 0 0)
+	)
+	(junction
+		(at 36.83 27.94)
+		(diameter 0)
+		(color 0 0 0 0)
+	)
+	(wire
+		(pts
+			(xy 36.83 27.94) (xy 36.83 29.21)
+		)
+		(stroke
+			(width 0)
+			(type default)
+		)
+	)
+	(wire
+		(pts
+			(xy 31.75 36.83) (xy 36.83 36.83)
+		)
+		(stroke
+			(width 0)
+			(type default)
 		)
 	)
@@
 	(wire
 		(pts
-			(xy 29.21 27.94) (xy 40.64 27.94)
+			(xy 29.21 27.94) (xy 36.83 27.94)
 		)
 		(stroke
@@
 	(wire
 		(pts
-			(xy 31.75 30.48) (xy 31.75 33.02)
+			(xy 36.83 27.94) (xy 40.64 27.94)
+		)
+		(stroke
+			(width 0)
+			(type default)
+		)
+	)
+	(wire
+		(pts
+			(xy 36.83 36.83) (xy 36.83 41.91)
+		)
+		(stroke
+			(width 0)
+			(type default)
+		)
+	)
+	(wire
+		(pts
+			(xy 31.75 30.48) (xy 31.75 36.83)
 		)
 		(stroke
@@
 	)
 	(symbol
-		(lib_id "power:GND")
-		(at 31.75 33.02 0)
+		(lib_id "Device:C_Polarized")
+		(at 36.83 33.02 0)
 		(unit 1)
 		(body_style 1)
@@
 		(dnp no)
 		(fields_autoplaced yes)
+		(property "Reference" "C1"
+			(at 40.64 30.8609 0)
+			(show_name no)
+			(do_not_autoplace no)
+			(effects
+				(font
+					(size 1.27 1.27)
+				)
+				(justify left)
+			)
+		)
+		(property "Value" "22u"
+			(at 40.64 33.4009 0)
+			(show_name no)
+			(do_not_autoplace no)
+			(effects
+				(font
+					(size 1.27 1.27)
+				)
+				(justify left)
+			)
+		)
+		(property "Footprint" ""
+			(at 37.7952 36.83 0)
+			(hide yes)
+			(show_name no)
+			(do_not_autoplace no)
+			(effects
+				(font
+					(size 1.27 1.27)
+				)
+			)
+		)
+		(property "Datasheet" ""
+			(at 36.83 33.02 0)
+			(hide yes)
+			(show_name no)
+			(do_not_autoplace no)
+			(effects
+				(font
+					(size 1.27 1.27)
+				)
+			)
+		)
+		(property "Description" "Polarized capacitor"
+			(at 36.83 33.02 0)
+			(hide yes)
+			(show_name no)
+			(do_not_autoplace no)
+			(effects
+				(font
+					(size 1.27 1.27)
+				)
+			)
+		)
+		(pin "1"
+		)
+		(pin "2"
+		)
+		(instances
+			(project "BM107_V6_Layout"
+				(path "/160d15a2-4a54-4a04-add2-ae6ecbb41248"
+					(reference "C1")
+					(unit 1)
+				)
+			)
+		)
+	)
+	(symbol
+		(lib_id "power:GND")
+		(at 36.83 41.91 0)
+		(unit 1)
+		(body_style 1)
+		(exclude_from_sim no)
+		(in_bom yes)
+		(on_board yes)
+		(in_pos_files yes)
+		(dnp no)
+		(fields_autoplaced yes)
 		(property "Reference" "#PWR01"
-			(at 31.75 39.37 0)
+			(at 36.83 48.26 0)
 			(hide yes)
 			(show_name no)
@@
 		)
 		(property "Value" "GND"
-			(at 31.75 38.1 0)
+			(at 36.83 46.99 0)
 			(show_name no)
 			(do_not_autoplace no)
@@
 		)
 		(property "Footprint" ""
-			(at 31.75 33.02 0)
+			(at 36.83 41.91 0)
 			(hide yes)
 			(show_name no)
@@
 		)
 		(property "Datasheet" ""
-			(at 31.75 33.02 0)
+			(at 36.83 41.91 0)
 			(hide yes)
 			(show_name no)
@@
 		)
 		(property "Description" "Power symbol creates a global label with name \"GND\" , ground"
-			(at 31.75 33.02 0)
+			(at 36.83 41.91 0)
 			(hide yes)
 			(show_name no)
@@
 				)
 			)
+		)
+	)
+	(sheet
+		(at 166.37 132.715)
+		(size 29.21 13.335)
+		(exclude_from_sim no)
+		(in_bom yes)
+		(on_board yes)
+		(dnp no)
+		(fields_autoplaced yes)
+		(stroke
+			(width 0.1524)
+			(type solid)
+		)
+		(fill
+			(color 0 0 0 0)
+		)
+		(property "Sheetname" "Bluepill"
+			(at 166.37 132.0034 0)
+			(show_name no)
+			(do_not_autoplace no)
+			(effects
+				(font
+					(size 1.27 1.27)
+				)
+				(justify left bottom)
+			)
+		)
+		(property "Sheetfile" "Bluepill.kicad_sch"
+			(at 166.37 146.6346 0)
+			(show_name no)
+			(do_not_autoplace no)
+			(effects
+				(font
+					(size 1.27 1.27)
+				)
+				(justify left top)
+			)
+		)
+		(instances
+			(project "BM107_V6_Layout"
+				(path "/160d15a2-4a54-4a04-add2-ae6ecbb41248"
+					(page "5")
+				)
+			)

Commit message: NEuneuenuenbeuebu
Parts:
- removed J1, J2: Screw_Terminal_01x02, symbol Connector:Screw_Terminal_01x02
- added J1, J2, J5, J6: PC5930T, Aktive_Bal_Footprints:PC5930T_Footprint, symbol BM107_Labor_Lib:PC5930T
- added J3: WAGO_1_5, Connector_Wago:Wago_734-135_1x05_P3.50mm_Vertical, symbol BM107_Labor_Lib:WAGO_1_5
- added J4: DE9_Pins_MountingHoles, Aktive_Bal_Footprints:D_SUB9_Stecker, symbol Connector:DE9_Pins_MountingHoles
- C1: value 22u -> 22u Elko; footprint (none) -> Capacitor_SMD:CP_Elec_5x5.3
Connections:
- net +24V: now also J1.1 (Pin_1)
- net GND: now also J2.1 (Pin_1), J3.5 (Pin_5), J4.3, J4.6, J4.SH (PAD)
- net V_Motor+: now also J5.1 (Pin_1)
- net V_Motor-: now also J6.1 (Pin_1)
- new net +3.0V: J3.2 (Pin_2)
- new net CANH: J4.7
- new net CANL: J4.2
- new net Sp_A: J3.1 (Pin_1)
- new net Sp_B: J3.3 (Pin_3)
- no-connect marks 0 -> 6
Other:
- removed sheet Bluepill

Commit message: bm107 neu
Other:
- moved on the sheet: J5, J6
Changed lines of the file:
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@@
 	(wire
 		(pts
-			(xy 228.6 44.45) (xy 233.68 44.45)
+			(xy 139.7 38.1) (xy 144.78 38.1)
 		)
 		(stroke
@@
 	(wire
 		(pts
-			(xy 228.6 35.56) (xy 233.68 35.56)
+			(xy 139.7 29.21) (xy 144.78 29.21)
 		)
 		(stroke
@@
 	(global_label "V_Motor-"
 		(shape input)
-		(at 228.6 44.45 180)
+		(at 139.7 38.1 180)
 		(fields_autoplaced yes)
 		(effects
@@
 		)
 		(property "Intersheetrefs" "${INTERSHEET_REFS}"
-			(at 216.7249 44.45 0)
+			(at 127.8249 38.1 0)
 			(hide yes)
 			(show_name no)
@@
 	(global_label "V_Motor+"
 		(shape input)
-		(at 228.6 35.56 180)
+		(at 139.7 29.21 180)
 		(fields_autoplaced yes)
 		(effects
@@
 		)
 		(property "Intersheetrefs" "${INTERSHEET_REFS}"
-			(at 216.7249 35.56 0)
+			(at 127.8249 29.21 0)
 			(hide yes)
 			(show_name no)
@@
 	(symbol
 		(lib_id "BM107_Labor_Lib:PC5930T")
-		(at 238.76 35.56 0)
+		(at 149.86 29.21 0)
 		(unit 1)
 		(body_style 1)
@@
 		(fields_autoplaced yes)
 		(property "Reference" "J5"
-			(at 238.76 41.91 0)
+			(at 149.86 35.56 0)
 			(show_name no)
 			(do_not_autoplace no)
@@
 		)
 		(property "Value" "PC5930T"
-			(at 238.76 39.37 0)
+			(at 149.86 33.02 0)
 			(show_name no)
 			(do_not_autoplace no)
@@
 		)
 		(property "Footprint" "Aktive_Bal_Footprints:PC5930T_Footprint"
-			(at 238.76 35.56 0)
+			(at 149.86 29.21 0)
 			(hide yes)
 			(show_name no)
@@
 		)
 		(property "Datasheet" ""
-			(at 238.76 35.56 0)
+			(at 149.86 29.21 0)
 			(hide yes)
 			(show_name no)
@@
 		)
 		(property "Description" "Generic screw terminal, single row, 01x01, script generated (kicad-library-utils/schlib/autogen/connector/)"
-			(at 238.76 35.56 0)
+			(at 149.86 29.21 0)
 			(hide yes)
 			(show_name no)
@@
 	(symbol
 		(lib_id "BM107_Labor_Lib:PC5930T")
-		(at 238.76 44.45 0)
+		(at 149.86 38.1 0)
 		(unit 1)
 		(body_style 1)
@@
 		(fields_autoplaced yes)
 		(property "Reference" "J6"
-			(at 238.76 50.8 0)
+			(at 149.86 44.45 0)
 			(show_name no)
 			(do_not_autoplace no)
@@
 		)
 		(property "Value" "PC5930T"
-			(at 238.76 48.26 0)
+			(at 149.86 41.91 0)
 			(show_name no)
 			(do_not_autoplace no)
@@
 		)
 		(property "Footprint" "Aktive_Bal_Footprints:PC5930T_Footprint"
-			(at 238.76 44.45 0)
+			(at 149.86 38.1 0)
 			(hide yes)
 			(show_name no)
@@
 		)
 		(property "Datasheet" ""
-			(at 238.76 44.45 0)
+			(at 149.86 38.1 0)
 			(hide yes)
 			(show_name no)
@@
 		)
 		(property "Description" "Generic screw terminal, single row, 01x01, script generated (kicad-library-utils/schlib/autogen/connector/)"
-			(at 238.76 44.45 0)
-			(hide yes)
-			(show_name no)
+			(at 149.86 38.1 0)
+			(hide yes)
+			(show_name no)
