File: BM107/BM107_V6_Layout/H_Bruecke.kicad_sch (KiCad schematic)
At the start: 0 parts

Commit message: NEuneuenuenbeuebu
Parts:
- added C22, C31: 47u, Capacitor_SMD:C_0805_2012Metric, symbol Device:C
- added C23, C24, C32, C33: 10p, Capacitor_SMD:C_0805_2012Metric, symbol Device:C
- added C25, C34: 4.7u, Capacitor_SMD:C_0805_2012Metric, symbol Device:C
- added C26, C27, C29, C30: 5n, Capacitor_SMD:C_0805_2012Metric, symbol Device:C_Small
- added C28, C35: 220n, Capacitor_SMD:C_0805_2012Metric, symbol Device:C
- added D3, D6: CD1408, Aktive_Bal_Footprints:CD1408_Footprint, symbol BM107_Labor_Lib:CD1408
- added D4, D5, D7, D8: SS24, Diode_SMD:D_SMA, symbol Diode:SS24
- added Q1, Q2, Q3, Q4: BSC016N06NS, Package_TO_SOT_SMD:TDSON-8-1, symbol BM107_Labor_Lib:BSC016N06NS
- added R10, R22: 2.2, Resistor_SMD:R_0805_2012Metric, symbol Device:R
- added R11, R12, R15, R16: 1.5, Resistor_SMD:R_0805_2012Metric, symbol Device:R_Small
- added R13, R14, R6, R7: 100k, Resistor_SMD:R_0805_2012Metric, symbol Device:R
- added R17, R18, R23, R24: 100, Resistor_SMD:R_0805_2012Metric, symbol Device:R
- added R19: 500u, Aktive_Bal_Footprints:CMP-R100-1.0, symbol Device:R_Shunt
- added R20, R21, R8, R9: 49, Resistor_SMD:R_0805_2012Metric, symbol Device:R
- added U10, U9: UCC27734, Aktive_Bal_Footprints:SOIC-8_3.9x4.9mm_P1.27mm_UCC27734, symbol BM107_Labor_Lib:UCC27734
Connections:
- new net: D8.1 (K), R24.1, U10.4 (LO)
- new net: C23.2, R8.2, U9.1 (HI)
- new net: C35.1, D6.1 (K), U10.8 (HB)
- new net: C34.1, D6.2 (A), R22.2, U10.5 (VDD)
- new net: C33.1, R21.2, U10.2 (LI)
- new net: C25.1, D3.2 (A), R10.2, U9.5 (VDD)
- new net: C24.1, R9.2, U9.2 (LI)
- new net: D5.1 (K), R18.1, U9.4 (LO)
- new net: C27.2, R12.1
- new net: C30.1, Q3.1 (S), Q3.2 (S), Q3.3 (S), Q4.5 (D), R13.1, R15.2, R19.4
- new net: C28.1, D3.1 (K), U9.8 (HB)
- new net: C26.2, R11.1
- new net: D4.1 (K), R17.1, U9.7 (HO)
- new net: C29.2, R15.1
- new net: C32.2, R20.2, U10.1 (HI)
- new net: D7.1 (K), R23.1, U10.7 (HO)
- new net: C30.2, R16.1
- new net +12V: C22.1, C31.1, R10.1, R22.1
- new net +24V: C26.1, C29.1, Q1.5 (D), Q3.5 (D)
- new net G1: D4.2 (A), Q1.4 (G), Q2.4 (G), Q3.4 (G), Q4.4 (G), R13.2, R14.2, R17.2, R6.2, R7.2
- new net G1_IN: R8.1
- new net G2: D5.2 (A), R18.2
- new net G2_IN: R9.1
- new net G3: D7.2 (A), R23.2
- new net G3_IN: R20.1
- new net G4: D8.2 (A), R24.2
- new net G4_IN: R21.1
- new net GND: C22.2, C23.1, C24.2, C25.2, C31.2, C32.1, C33.2, C34.2, Q2.1 (S), Q2.2 (S), Q2.3 (S), Q4.1 (S), Q4.2 (S), Q4.3 (S), R12.2, R14.1, R16.2, R7.1, U10.3 (COM), U9.3 (COM)
- new net IS+: R19.3
- new net IS-: R19.2
- new net V_Motor+: C27.1, C28.2, Q1.1 (S), Q1.2 (S), Q1.3 (S), Q2.5 (D), R11.2, R6.1, U9.6 (HS)
- new net V_Motor-: C35.2, R19.1, U10.6 (HS)

Commit message: bm107 neu
Parts:
- removed R19: 500u, Aktive_Bal_Footprints:CMP-R100-1.0, symbol Device:R_Shunt
- added R26: Shunt_BVT-M-R0005, Aktive_Bal_Footprints:Shunt_BVT-M-R0005, symbol BM107_Labor_Lib:Shunt_BVT-M-R0005
Connections:
- net IS+: now also R26.3
- net IS-: now also R26.2
- net V_Motor-: now also R26.1
- net at C30.1, Q3.1 (S), Q3.2 (S)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: now also R26.4
Changed lines of the file:
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@@
 	)
 	(symbol
+		(lib_id "BM107_Labor_Lib:Shunt_BVT-M-R0005")
+		(at 116.84 36.83 270)
+		(unit 1)
+		(body_style 1)
+		(exclude_from_sim no)
+		(in_bom yes)
+		(on_board yes)
+		(in_pos_files yes)
+		(dnp no)
+		(fields_autoplaced yes)
+		(property "Reference" "R26"
+			(at 116.84 30.48 90)
+			(show_name no)
+			(do_not_autoplace no)
+			(effects
+				(font
+					(size 1.27 1.27)
+				)
+			)
+		)
+		(property "Value" "Shunt_BVT-M-R0005"
+			(at 116.84 33.02 90)
+			(show_name no)
+			(do_not_autoplace no)
+			(effects
+				(font
+					(size 1.27 1.27)
+				)
+			)
+		)
+		(property "Footprint" "Aktive_Bal_Footprints:Shunt_BVT-M-R0005"
+			(at 116.84 35.052 90)
+			(show_name no)
+			(do_not_autoplace no)
+			(effects
+				(font
+					(size 1.27 1.27)
+				)
+			)
+		)
+		(property "Datasheet" ""
+			(at 116.84 36.83 0)
+			(hide yes)
+			(show_name no)
+			(do_not_autoplace no)
+			(effects
+				(font
+					(size 1.27 1.27)
+				)
+			)
+		)
+		(property "Description" "Shunt resistor with Kelvin connections"
+			(at 116.84 36.83 0)
+			(hide yes)
+			(show_name no)
+			(do_not_autoplace no)
+			(effects
+				(font
+					(size 1.27 1.27)
+				)
+			)
+		)
+		(pin "1"
+		)
+		(pin "3"
+		)
+		(pin "2"
+		)
+		(pin "4"
+		)
+		(instances
+			(project "BM107_V6_Layout"
+				(path "/160d15a2-4a54-4a04-add2-ae6ecbb41248/4c1a8778-342d-4b78-bb3f-0bf650e43a5b"
+					(reference "R26")
+					(unit 1)
+				)
+			)
+		)
+	)
+	(symbol
 		(lib_id "BM107_Labor_Lib:CD1408")
 		(at 219.71 114.3 270)
@@
 					(unit 1)
 				)
-			)
-		)
-	)
-	(symbol
-		(lib_id "Device:R_Shunt")
-		(at 116.84 36.83 270)
-		(unit 1)
-		(body_style 1)
-		(exclude_from_sim no)
-		(in_bom yes)
-		(on_board yes)
-		(in_pos_files yes)
-		(dnp no)
-		(fields_autoplaced yes)
-		(property "Reference" "R19"
-			(at 116.84 30.48 90)
-			(show_name no)
-			(do_not_autoplace no)
-			(effects
-				(font
-					(size 1.27 1.27)
-				)
-			)
-		)
-		(property "Value" "500u"
-			(at 116.84 33.02 90)
-			(show_name no)
-			(do_not_autoplace no)
-			(effects
-				(font
-					(size 1.27 1.27)
-				)
-			)
-		)
-		(property "Footprint" "Aktive_Bal_Footprints:CMP-R100-1.0"
-			(at 116.84 35.052 90)
-			(hide yes)
-			(show_name no)
-			(do_not_autoplace no)
-			(effects
-				(font
-					(size 1.27 1.27)
-				)
-			)
-		)
-		(property "Datasheet" ""
-			(at 116.84 36.83 0)
-			(hide yes)
-			(show_name no)
-			(do_not_autoplace no)
-			(effects
-				(font
-					(size 1.27 1.27)
-				)
-			)
-		)
-		(property "Description" "Shunt resistor with Kelvin connections"
-			(at 116.84 36.83 0)
-			(hide yes)
-			(show_name no)
-			(do_not_autoplace no)
-			(effects
-				(font
-					(size 1.27 1.27)
-				)
-			)
-		)
-		(pin "4"
-		)
-		(pin "1"
-		)
-		(pin "2"
-		)
-		(pin "3"
-		)
-		(instances
-			(project "BM107_V6_Layout"
-				(path "/160d15a2-4a54-4a04-add2-ae6ecbb41248/4c1a8778-342d-4b78-bb3f-0bf650e43a5b"
-					(reference "R19")
-					(unit 1)
-				)
