File: BM107/BM107_V6_Layout/H_Bruecke.kicad_sch (KiCad schematic)
At the start: 45 parts, among them Q1 BSC016N06NS, Q2 BSC016N06NS, Q3 BSC016N06NS, Q4 BSC016N06NS, U10 UCC27734, U9 UCC27734

Commit message: bmschießmichtot
Connections:
- net G1: no longer Q2.4 (G), Q3.4 (G), Q4.4 (G), R13.2, R14.2, R7.2
- net G2: now also Q2.4 (G), R7.2
- net G3: now also Q3.4 (G), R13.2
- net G4: now also Q4.4 (G), R14.2
Changed lines of the file:
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@@
 		)
 	)
-	(global_label "G1"
+	(global_label "G4"
 		(shape input)
 		(at 72.39 52.07 180)
@@
 		)
 	)
-	(global_label "G1"
+	(global_label "G2"
 		(shape input)
 		(at 22.86 50.8 180)
@@
 		)
 	)
-	(global_label "G1"
+	(global_label "G3"
 		(shape input)
 		(at 72.39 25.4 180)
@@
 		(dnp no)
 		(fields_autoplaced yes)
-		(property "Reference" "#FLG04"
+		(property "Reference" "#FLG06"
 			(at 212.725 114.3 0)
 			(hide yes)
@@
 			(project "BM107_V6_Layout"
 				(path "/160d15a2-4a54-4a04-add2-ae6ecbb41248/4c1a8778-342d-4b78-bb3f-0bf650e43a5b"
-					(reference "#FLG04")
+					(reference "#FLG06")
 					(unit 1)
 				)
@@
 		(dnp no)
 		(fields_autoplaced yes)
-		(property "Reference" "#FLG03"
+		(property "Reference" "#FLG05"
 			(at 77.47 125.095 0)
 			(hide yes)
@@
 			(project "BM107_V6_Layout"
 				(path "/160d15a2-4a54-4a04-add2-ae6ecbb41248/4c1a8778-342d-4b78-bb3f-0bf650e43a5b"
-					(reference "#FLG03")
-					(unit 1)
-				)
+					(reference "#FLG05")
+					(unit 1)
+				)

Commit message: bm107
Parts:
- Q1, Q2, Q3, Q4: footprint Package_TO_SOT_SMD:TDSON-8-1 -> Aktive_Bal_Footprints:BSC016N06NS
Changed lines of the file:
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@@
 			)
 		)
-		(property "Footprint" "Package_TO_SOT_SMD:TDSON-8-1"
+		(property "Footprint" "Aktive_Bal_Footprints:BSC016N06NS"
 			(at 45.72 27.305 0)
 			(hide yes)
@@
 			)
 		)
-		(property "Footprint" "Package_TO_SOT_SMD:TDSON-8-1"
+		(property "Footprint" "Aktive_Bal_Footprints:BSC016N06NS"
 			(at 95.25 53.975 0)
 			(hide yes)
@@
 			)
 		)
-		(property "Footprint" "Package_TO_SOT_SMD:TDSON-8-1"
+		(property "Footprint" "Aktive_Bal_Footprints:BSC016N06NS"
 			(at 95.25 27.305 0)
 			(hide yes)
@@
 			)
 		)
-		(property "Footprint" "Package_TO_SOT_SMD:TDSON-8-1"
+		(property "Footprint" "Aktive_Bal_Footprints:BSC016N06NS"
 			(at 45.72 52.705 0)
 			(hide yes)
