File: BM107/Labor_6_Schaltplan_Abgabe/BM107_V6_Layout/BM107_V6_Layout.kicad_pcb (KiCad board)
At the start: 2 copper layers, 90 parts, among them J1 WAGO_1_5, J2 PC5930T, J3 PC5930T, J4 DE9_Pins_MountingHoles, J5 PC5930T, J6 PC5930T, J7 Sockel_BluePill, J8 Conn_01x02_Pin, Q1 BSC016N06NS, Q2 BSC016N06NS, Q3 BSC016N06NS, Q4 BSC016N06NS, U1 LT1999-50, U10 UCC27734, U2 SN65HVD233, U3 R-78K15-0.5, U4 ADR3036, U5 LM317_SOT-223, U6 R-78K5.0-0.5, U7 AD8031, U8 LD1117S33TR_SOT223, U9 UCC27734

Commit message: bmschießmichtot
Parts:
- moved J2 194.4 mm to (50.4, 26.4), turned to -90 degrees
- moved J3 167.9 mm to (50.4, 52.6), turned to -90 degrees
- moved J5 130.0 mm to (142.0, 26.6), turned to 90 degrees
- moved U1 127.6 mm to (22.0, 75.0)
- moved C3 127.0 mm to (159.3, 144.7)
- moved J4 127.0 mm to (113.8, 143.5)
- moved J7 127.0 mm to (139.8, 142.2)
- moved JP1 127.0 mm to (159.3, 172.3)
- moved R1 127.0 mm to (159.3, 169.0)
- moved C4 127.0 mm to (159.3, 147.7)
- moved C2 127.0 mm to (159.3, 141.7)
- moved J8 127.0 mm to (159.4, 162.7)
- moved U2 127.0 mm to (160.8, 158.1)
- moved Q3 93.1 mm to (103.4, 23.4), turned to 90 degrees
- moved J1 84.9 mm to (21.6, 104.6), turned to 90 degrees
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Connections:
- Q2 pad 4: G1 -> G2
- Q3 pad 4: G1 -> G3
- Q4 pad 4: G1 -> G4
- R13 pad 2: G1 -> G3
- R14 pad 2: G1 -> G4
- R7 pad 2: G1 -> G2
Other:
- copper layers 2 -> 4
