File: KiCad/Aktive_Bal_Bericht - V3/controller.kicad_sch (KiCad schematic)
At the start: 32 parts, among them J21 Conn_01x02_Pin, J22 Conn_01x02_Pin, J23 Conn_01x02_Pin, J24 Conn_01x02_Pin, Q1 BSS316NH6327XTSA1, U14 TL084, U15 LM2596S-ADJ

Commit message: Alles schöner und 3d
Other:
- note removed: "Differenzspannung messen!!"
- moved on the sheet: C24, C25, C27, C28, C30, C31, J21, J22, J24, L1, R101, R104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
