File: KiCad/Aktive_Bal_Bericht - V3/power_mosfet.kicad_sch (KiCad schematic)
At the start: 124 parts, among them J15 Screw_Terminal_01x03, J16 Screw_Terminal_01x03, J17 Screw_Terminal_01x03, J18 Screw_Terminal_01x03, J19 Screw_Terminal_01x03, J20 Screw_Terminal_01x03, Q10_H1 NTTFS6H888NL, Q10_L1 NTTFS6H888NL, Q11_H1 NTTFS6H888NL, Q11_L1 NTTFS6H888NL, Q12_H1 NTTFS6H888NL, Q12_L1 NTTFS6H888NL, Q13_H1 NTTFS6H888NL, Q13_L1 NTTFS6H888NL, Q14_H1 NTTFS6H888NL, Q14_L1 NTTFS6H888NL, Q15_H1 NTTFS6H888NL, Q15_L1 NTTFS6H888NL, Q16_H1 NTTFS6H888NL, Q16_L1 NTTFS6H888NL, Q1_H1 NTTFS6H888NL, Q1_L1 NTTFS6H888NL, Q2_H1 NTTFS6H888NL, Q2_L1 NTTFS6H888NL, Q3_H1 NTTFS6H888NL, Q3_L1 NTTFS6H888NL, Q4_H1 NTTFS6H888NL, Q4_L1 NTTFS6H888NL, Q5_H1 NTTFS6H888NL, Q5_L1 NTTFS6H888NL, Q6_H1 NTTFS6H888NL, Q6_L1 NTTFS6H888NL, Q7_H1 NTTFS6H888NL, Q7_L1 NTTFS6H888NL, Q8_H1 NTTFS6H888NL, Q8_L1 NTTFS6H888NL, Q9_H1 NTTFS6H888NL, Q9_L1 NTTFS6H888NL, U10 LTV-847S, U11 LTV-847S, U12 LTV-847S, U13 LTV-847S

Commit message: Alles schöner und 3d
Parts:
- J15, J16, J17, J18, J19, J20: footprint TerminalBlock_4Ucon:TerminalBlock_4Ucon_1x03_P3.50mm_Horizontal -> Aktive_Bal_Footprints:TerminalBlock_4Ucon_1x03_P3.50mm_Horizontal_3d
Other:
- moved on the sheet: J15, J16, J17, J18, J19, J20, Q10_L1, Q11_L1, Q12_L1, Q13_L1, Q14_L1, Q15_L1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
