File: KiCad/Aktive_Bal_Bericht - V5/Aktive_Bal.kicad_sch (KiCad schematic)
At the start: 48 parts, among them J10 Conn_01x02_Pin, J11 Conn_01x02_Pin, J14 Conn_01x02_Pin, J2 A-DF_09_A_KG-T4S, J3 Conn_01x02_Pin, J4 Conn_01x02_Pin, J5 Conn_01x02_Pin, J6 Conn_01x02_Pin, J7 Sockel_BluePill, U2 ADUM1250ARZ-RL7, U3 SN65HVD233, U6 PCA9306DC, U7 PCF8575CDB, U9 MCP4725xxx-xCH

Commit message: Überprüfung von Schaltplan
Überprüfung von Schaltplan
Other:
- moved on the sheet: C1, R3
