File: KiCad/Aktive_Bal_Bericht - V5/Spannungsversorgung.kicad_sch (KiCad schematic)
At the start: 22 parts, among them J1 Screw_Terminal_01x02, J12 Conn_01x02_Pin, J13 Conn_01x02_Pin, J9 Conn_01x02_Pin, U1 RFP12N10L, U4 SCW20C-12, U5 EC1SA16N, U8 LM1117MP-3.3

Commit message: Überprüfung von Schaltplan
Überprüfung von Schaltplan
Other:
- note added: "Remote on/off SCW20C offen oder Anschluss an Vcc (>2,5V heißt on)"
- note removed: "Remote on/off SCW20C Offen oder anschluss an Vcc (>2,5V heißt on)"
Changed lines of the file:
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@@
 		(comment 3 "Gideon Jung")
 	)
-	(text "Remote on/off SCW20C\nOffen oder anschluss an \nVcc (>2,5V heißt on)"
+	(text "Remote on/off SCW20C\noffen oder Anschluss an \nVcc (>2,5V heißt on)"
 		(exclude_from_sim no)
 		(at 124.714 33.274 0)
@@
 			(justify right bottom)
 		)
-		(property "Netclass" "power"
+		(property "Netzklasse" "power"
 			(at 68.0085 64.77 0)
 			(show_name no)
@@
 			(justify right bottom)
 		)
-		(property "Netclass" "power"
+		(property "Netzklasse" "power"
 			(at 93.4085 52.07 0)
 			(show_name no)
@@
 			(justify left bottom)
 		)
-		(property "Netclass" "power"
+		(property "Netzklasse" "power"
 			(at 108.6485 41.91 0)
 			(show_name no)
@@
 			(justify left bottom)
 		)
-		(property "Netclass" "power"
+		(property "Netzklasse" "power"
 			(at 87.6935 110.49 0)
 			(show_name no)
@@
 			(justify left bottom)
 		)
-		(property "Netclass" "power"
+		(property "Netzklasse" "power"
 			(at 55.3085 57.15 0)
 			(show_name no)
@@
 			(justify left bottom)
 		)
-		(property "Netclass" "power"
+		(property "Netzklasse" "power"
 			(at 55.3085 36.83 0)
 			(show_name no)
@@
 			(justify left bottom)
 		)
-		(property "Netclass" "power"
+		(property "Netzklasse" "power"
 			(at 150.5585 110.49 0)
 			(show_name no)
@@
 			(justify left bottom)
 		)
-		(property "Netclass" "power"
+		(property "Netzklasse" "power"
 			(at 84.5185 100.33 0)
 			(show_name no)
@@
 			(justify left bottom)
 		)
-		(property "Netclass" "power"
+		(property "Netzklasse" "power"
 			(at 40.0685 102.87 0)
 			(show_name no)
@@
 			(justify right bottom)
 		)
-		(property "Netclass" "power"
+		(property "Netzklasse" "power"
 			(at 40.0685 113.03 0)
 			(show_name no)
@@
 					(unit 1)
 				)
+			)
+		)
+	)
+	(symbol
+		(lib_id "Aktive_Bal_Lib:LOGO")
+		(at 257.81 173.99 0)
+		(unit 1)
+		(body_style 1)
+		(exclude_from_sim no)
+		(in_bom yes)
+		(on_board yes)
+		(in_pos_files yes)
+		(dnp no)
+		(fields_autoplaced yes)
+		(property "Reference" "#G4"
+			(at 257.81 147.7433 0)
+			(hide yes)
+			(show_name no)
+			(do_not_autoplace no)
+			(effects
+				(font
+					(size 1.27 1.27)
+				)
+			)
+		)
+		(property "Value" "LOGO"
+			(at 257.81 200.2367 0)
+			(hide yes)
+			(show_name no)
+			(do_not_autoplace no)
+			(effects
+				(font
+					(size 1.27 1.27)
+				)
+			)
+		)
+		(property "Footprint" "Aktive_Bal_Footprints:Logo"
+			(at 257.81 173.99 0)
+			(hide yes)
+			(show_name no)
+			(do_not_autoplace no)
+			(effects
+				(font
+					(size 1.27 1.27)
+				)
+			)
+		)
+		(property "Datasheet" ""
+			(at 257.81 173.99 0)
+			(hide yes)
+			(show_name no)
+			(do_not_autoplace no)
+			(effects
+				(font
+					(size 1.27 1.27)
+				)
+			)
+		)
+		(property "Description" ""
+			(at 257.81 173.99 0)
+			(hide yes)
+			(show_name no)
+			(do_not_autoplace no)
+			(effects
+				(font
+					(size 1.27 1.27)
+				)
+			)
+		)
+		(instances
+			(project "Aktive_Bal"
+				(path "/7c40c112-cd2b-4a48-9744-14a65613b3b5/5b8cdbf7-6c94-4219-a7d9-e8db0ed1ced2"
+					(reference "#G4")
+					(unit 1)
+				)
