File: KiCad/Aktive_Bal_Bericht - V5/controller.kicad_sch (KiCad schematic)
At the start: 31 parts, among them J21 Conn_01x02_Pin, J22 Conn_01x02_Pin, J23 Conn_01x02_Pin, J24 Conn_01x02_Pin, Q1 BSS316NH6327XTSA1, U14 TL084, U15 LM2596S-ADJ

Commit message: Überprüfung von Schaltplan
Überprüfung von Schaltplan
Changed lines of the file:
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@@
 	)
 	(junction
-		(at 214.63 38.1)
+		(at 163.83 68.58)
 		(diameter 0)
 		(color 0 0 0 0)
 	)
 	(junction
-		(at 163.83 68.58)
+		(at 217.17 38.1)
 		(diameter 0)
 		(color 0 0 0 0)
@@
 	)
 	(junction
-		(at 214.63 73.66)
-		(diameter 0)
-		(color 0 0 0 0)
-	)
-	(junction
 		(at 73.66 48.26)
 		(diameter 0)
@@
 	(wire
 		(pts
-			(xy 214.63 73.66) (xy 214.63 38.1)
+			(xy 217.17 73.66) (xy 217.17 38.1)
 		)
 		(stroke
@@
 	(wire
 		(pts
-			(xy 213.36 73.66) (xy 214.63 73.66)
+			(xy 213.36 73.66) (xy 217.17 73.66)
 		)
 		(stroke
@@
 	(wire
 		(pts
-			(xy 217.17 73.66) (xy 214.63 73.66)
-		)
-		(stroke
-			(width 0)
-			(type default)
-		)
-	)
-	(wire
-		(pts
 			(xy 40.64 140.97) (xy 40.64 143.51)
 		)
@@
 	(wire
 		(pts
-			(xy 214.63 38.1) (xy 228.6 38.1)
+			(xy 217.17 38.1) (xy 228.6 38.1)
 		)
 		(stroke
@@
 	(wire
 		(pts
-			(xy 185.42 38.1) (xy 214.63 38.1)
+			(xy 185.42 38.1) (xy 217.17 38.1)
 		)
 		(stroke
@@
 			(justify left bottom)
 		)
-		(property "Netclass" "analog"
+		(property "Netzklasse" "analog"
 			(at 38.7985 54.61 0)
 			(show_name no)
@@
 		(length 2.54)
 		(shape round)
-		(at 214.63 66.04 90)
+		(at 217.17 66.04 90)
 		(fields_autoplaced yes)
 		(effects
@@
 			(justify left bottom)
 		)
-		(property "Netclass" "power"
-			(at 212.09 65.3415 90)
+		(property "Netzklasse" "power"
+			(at 214.63 65.3415 90)
 			(show_name no)
 			(do_not_autoplace no)
@@
 		)
 		(property "Component Class" ""
-			(at -22.86 11.43 0)
+			(at -20.32 11.43 0)
 			(show_name no)
 			(do_not_autoplace no)
@@
 			(justify left bottom)
 		)
-		(property "Netclass" "analog"
+		(property "Netzklasse" "analog"
 			(at 92.71 128.27 0)
 			(show_name no)
@@
 			(justify left bottom)
 		)
-		(property "Netclass" "analog"
+		(property "Netzklasse" "analog"
 			(at 149.1615 140.97 0)
 			(show_name no)
@@
 			(justify right bottom)
 		)
-		(property "Netclass" "power"
+		(property "Netzklasse" "power"
 			(at 44.704 125.984 90)
 			(show_name no)
@@
 			(justify left bottom)
 		)
-		(property "Netclass" "analog"
+		(property "Netzklasse" "analog"
 			(at 69.2785 54.61 0)
 			(show_name no)
@@
 			(justify left bottom)
 		)
-		(property "Netclass" "analog"
+		(property "Netzklasse" "analog"
 			(at 88.3285 54.61 0)
 			(show_name no)
@@
 			(justify left bottom)
 		)
-		(property "Netclass" "analog"
+		(property "Netzklasse" "analog"
 			(at 122.936 127 0)
 			(show_name no)
@@
 			(justify right bottom)
 		)
-		(property "Netclass" "power"
+		(property "Netzklasse" "power"
 			(at 44.958 145.542 90)
 			(show_name no)
@@
 			(justify left bottom)
 		)
-		(property "Netclass" "analog"
+		(property "Netzklasse" "analog"
 			(at 92.71 140.97 0)
 			(show_name no)
@@
 			(justify left bottom)
 		)
-		(property "Netclass" "analog"
+		(property "Netzklasse" "analog"
 			(at 149.606 124.714 0)
 			(show_name no)
@@
 			(justify left bottom)
 		)
-		(property "Netclass" "analog"
+		(property "Netzklasse" "analog"
 			(at 57.8485 54.61 0)
 			(show_name no)
@@
 			(justify left bottom)
 		)
-		(property "Netclass" "analog"
+		(property "Netzklasse" "analog"
 			(at 153.0985 35.56 0)
 			(show_name no)
@@
 			(justify left bottom)
 		)
-		(property "Netclass" "analog"
+		(property "Netzklasse" "analog"
 			(at 38.7985 43.18 0)
 			(show_name no)
@@
 			(justify left bottom)
 		)
-		(property "Netclass" "power"
+		(property "Netzklasse" "power"
 			(at 201.422 69.596 0)
 			(show_name no)
@@
 			(justify left bottom)
 		)
-		(property "Netclass" "power"
+		(property "Netzklasse" "power"
 			(at 52.07 33.5915 90)
 			(show_name no)
@@
 			(justify left bottom)
 		)
-		(property "Netclass" "analog"
+		(property "Netzklasse" "analog"
 			(at 184.8485 53.34 0)
 			(show_name no)
@@
 			(justify left bottom)
 		)
-		(property "Netclass" "power"
+		(property "Netzklasse" "power"
 			(at 153.162 63.754 90)
 			(show_name no)
@@
 			(justify left bottom)
 		)
-		(property "Netclass" "analog"
+		(property "Netzklasse" "analog"
 			(at 52.7685 43.18 0)
 			(show_name no)
@@
 			(justify left bottom)
 		)
-		(property "Netclass" "analog"
+		(property "Netzklasse" "analog"
 			(at 123.7615 114.3 0)
 			(show_name no)
@@
 			(justify left bottom)
 		)
-		(property "Netclass" "analog"
+		(property "Netzklasse" "analog"
 			(at 108.5215 114.3 0)
 			(show_name no)
@@
 			(justify left bottom)
 		)
-		(property "Netclass" "analog"
+		(property "Netzklasse" "analog"
 			(at 97.2185 54.61 0)
 			(show_name no)
@@
 			(justify left bottom)
 		)
-		(property "Netclass" "analog"
+		(property "Netzklasse" "analog"
 			(at 134.0485 58.42 0)
 			(show_name no)
@@
 			(justify left bottom)
 		)
-		(property "Netclass" "analog"
+		(property "Netzklasse" "analog"
 			(at 111.1885 58.42 0)
 			(show_name no)
@@
 			(justify left bottom)
 		)
-		(property "Netclass" "power"
+		(property "Netzklasse" "power"
 			(at 152.654 58.166 90)
 			(show_name no)
@@
 					(unit 1)
 				)
+			)
+		)
+	)
+	(symbol
+		(lib_id "Aktive_Bal_Lib:LOGO")
+		(at 257.81 173.99 0)
+		(unit 1)
+		(body_style 1)
+		(exclude_from_sim no)
+		(in_bom yes)
+		(on_board yes)
+		(in_pos_files yes)
+		(dnp no)
+		(fields_autoplaced yes)
+		(property "Reference" "#G3"
+			(at 257.81 147.7433 0)
+			(hide yes)
+			(show_name no)
+			(do_not_autoplace no)
+			(effects
+				(font
+					(size 1.27 1.27)
+				)
+			)
+		)
+		(property "Value" "LOGO"
+			(at 257.81 200.2367 0)
+			(hide yes)
+			(show_name no)
+			(do_not_autoplace no)
+			(effects
+				(font
+					(size 1.27 1.27)
+				)
+			)
+		)
+		(property "Footprint" "Aktive_Bal_Footprints:Logo"
+			(at 257.81 173.99 0)
+			(hide yes)
+			(show_name no)
+			(do_not_autoplace no)
+			(effects
+				(font
+					(size 1.27 1.27)
+				)
+			)
+		)
+		(property "Datasheet" ""
+			(at 257.81 173.99 0)
+			(hide yes)
+			(show_name no)
+			(do_not_autoplace no)
+			(effects
+				(font
+					(size 1.27 1.27)
+				)
+			)
+		)
+		(property "Description" ""
+			(at 257.81 173.99 0)
+			(hide yes)
+			(show_name no)
+			(do_not_autoplace no)
+			(effects
+				(font
+					(size 1.27 1.27)
+				)
+			)
+		)
+		(instances
+			(project "Aktive_Bal"
+				(path "/7c40c112-cd2b-4a48-9744-14a65613b3b5/7022d0de-596a-4fda-81a7-762d98787f96"
+					(reference "#G3")
+					(unit 1)
+				)
