File: KiCad/Aktive_Bal_Bericht - V6/Aktive_Bal.kicad_pcb (KiCad board)
At the start: 4 copper layers, 122 x 101.3 mm, 226 parts, among them J1 Screw_Terminal_01x02, J10 Conn_01x02_Pin, J11 Conn_01x02_Pin, J12 Conn_01x02_Pin, J13 Conn_01x02_Pin, J14 Conn_01x02_Pin, J15 Screw_Terminal_01x03, J16 Screw_Terminal_01x03, J17 Screw_Terminal_01x03, J18 Screw_Terminal_01x03, J19 Screw_Terminal_01x03, J2 A-DF_09_A_KG-T4S, J20 Screw_Terminal_01x03, J21 Conn_01x02_Pin, J22 Conn_01x02_Pin, J23 Conn_01x02_Pin, J24 Conn_01x02_Pin, J3 Conn_01x02_Pin, J4 Conn_01x02_Pin, J5 Conn_01x02_Pin, J6 Conn_01x02_Pin, J7 Sockel_BluePill, J9 Conn_01x02_Pin, Q1 BSS316NH6327XTSA1, Q10_H1 NTTFS6H888NL, Q10_L1 NTTFS6H888NL, Q11_H1 NTTFS6H888NL, Q11_L1 NTTFS6H888NL, Q12_H1 NTTFS6H888NL, Q12_L1 NTTFS6H888NL, Q13_H1 NTTFS6H888NL, Q13_L1 NTTFS6H888NL, Q14_H1 NTTFS6H888NL, Q14_L1 NTTFS6H888NL, Q15_H1 NTTFS6H888NL, Q15_L1 NTTFS6H888NL, Q16_H1 NTTFS6H888NL, Q16_L1 NTTFS6H888NL, Q1_H1 NTTFS6H888NL, Q1_L1 NTTFS6H888NL, Q2_H1 NTTFS6H888NL, Q2_L1 NTTFS6H888NL, Q3_H1 NTTFS6H888NL, Q3_L1 NTTFS6H888NL, Q4_H1 NTTFS6H888NL, Q4_L1 NTTFS6H888NL, Q5_H1 NTTFS6H888NL, Q5_L1 NTTFS6H888NL, Q6_H1 NTTFS6H888NL, Q6_L1 NTTFS6H888NL, Q7_H1 NTTFS6H888NL, Q7_L1 NTTFS6H888NL, Q8_H1 NTTFS6H888NL, Q8_L1 NTTFS6H888NL, Q9_H1 NTTFS6H888NL, Q9_L1 NTTFS6H888NL, U1 RFP12N10L, U10 LTV-847S, U11 LTV-847S, U12 LTV-847S, U13 LTV-847S, U14 TL084, U15 LM2596S-ADJ, U2 ADUM1250ARZ-RL7, U3 SN65HVD233, U4 SCW20C-12, U5 EC1SA16N, U6 PCA9306DC, U7 PCF8575CDB, U8 LM1117MP-3.3, U9 MCP4725xxx-xCH

Commit message: sachen halt
Other:
- board text added: "A2"
- board text added: "Bat+"
- board text added: "GND_Bat"
- board text added: "GNDf"
- board text added: "elko smd aendern! C10 footprint zugroß C14 15 zu klein"
Changed lines of the file:
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@@
 		(tags "mountinghole M3")
 		(property "Reference" "H2"
-			(at 0 -4.15 0)
+			(at 0 3 0)
 			(layer "F.SilkS")
 			(effects
@@
 		)
 		(property "Value" "100k"
-			(at 0 1.65 90)
+			(at 0.2 2 90)
 			(layer "F.Fab")
 			(effects
@@
 		)
 		(property "Value" "10k"
-			(at 0 1.65 90)
+			(at 0 3 90)
 			(layer "F.Fab")
 			(effects
@@
 		)
 	)
+	(gr_text "elko smd aendern! \nC10 footprint zugroß\nC14 15 zu klein"
+		(at 189.5 131.804 0)
+		(layer "F.SilkS")
+		(effects
+			(font
+				(size 1 1)
+				(thickness 0.1)
+			)
+			(justify left bottom)
+		)
+	)
 	(gr_text "GND"
 		(at 165.8 62.504 90)
@@
 		)
 	)
+	(gr_text "GND_Bat"
+		(at 121 106.804 0)
+		(layer "F.SilkS")
+		(effects
+			(font
+				(size 1 1)
+				(thickness 0.15)
+			)
+			(justify left bottom)
+		)
+	)
+	(gr_text "Bat+\n"
+		(at 121.5 111.804 0)
+		(layer "F.SilkS")
+		(effects
+			(font
+				(size 1 1)
+				(thickness 0.15)
+			)
+			(justify left bottom)
+		)
+	)
 	(gr_text "VSh*10"
 		(at 129.139 76.914 0)
@@
 		)
 	)
-	(gr_text "A1"
+	(gr_text "A2"
 		(at 166.318945 72.520502 0)
 		(layer "F.SilkS")
@@
 		(layer "F.SilkS")
 		(effects
+			(font
+				(size 1 1)
+				(thickness 0.15)
+			)
+			(justify left bottom)
+		)
+	)
+	(gr_text "GNDf\n"
+		(at 218.25 112.554 0)
+		(layer "F.SilkS")
+		(effects
+			(font
+				(size 1 1)
+				(thickness 0.15)
+			)
+			(justify left bottom)
+		)
+	)
+	(gr_text "3.3V\n"
+		(at 218.75 108.304 0)
+		(layer "F.SilkS")
+		(effects
