File: KiCad/Aktive_Bal_Bericht - V7/Aktive_Bal.kicad_pcb (KiCad board)
At the start: 4 copper layers, 122 x 101.3 mm, 226 parts, among them J1 Screw_Terminal_01x02, J10 Conn_01x02_Pin, J11 Conn_01x02_Pin, J12 Conn_01x02_Pin, J13 Conn_01x02_Pin, J14 Conn_01x02_Pin, J15 Screw_Terminal_01x03, J16 Screw_Terminal_01x03, J17 Screw_Terminal_01x03, J18 Screw_Terminal_01x03, J19 Screw_Terminal_01x03, J2 A-DF_09_A_KG-T4S, J20 Screw_Terminal_01x03, J21 Conn_01x02_Pin, J22 Conn_01x02_Pin, J23 Conn_01x02_Pin, J24 Conn_01x02_Pin, J3 Conn_01x02_Pin, J4 Conn_01x02_Pin, J5 Conn_01x02_Pin, J6 Conn_01x02_Pin, J7 Sockel_BluePill, J9 Conn_01x02_Pin, Q1 BSS316NH6327XTSA1, Q10_H1 NTTFS6H888NL, Q10_L1 NTTFS6H888NL, Q11_H1 NTTFS6H888NL, Q11_L1 NTTFS6H888NL, Q12_H1 NTTFS6H888NL, Q12_L1 NTTFS6H888NL, Q13_H1 NTTFS6H888NL, Q13_L1 NTTFS6H888NL, Q14_H1 NTTFS6H888NL, Q14_L1 NTTFS6H888NL, Q15_H1 NTTFS6H888NL, Q15_L1 NTTFS6H888NL, Q16_H1 NTTFS6H888NL, Q16_L1 NTTFS6H888NL, Q1_H1 NTTFS6H888NL, Q1_L1 NTTFS6H888NL, Q2_H1 NTTFS6H888NL, Q2_L1 NTTFS6H888NL, Q3_H1 NTTFS6H888NL, Q3_L1 NTTFS6H888NL, Q4_H1 NTTFS6H888NL, Q4_L1 NTTFS6H888NL, Q5_H1 NTTFS6H888NL, Q5_L1 NTTFS6H888NL, Q6_H1 NTTFS6H888NL, Q6_L1 NTTFS6H888NL, Q7_H1 NTTFS6H888NL, Q7_L1 NTTFS6H888NL, Q8_H1 NTTFS6H888NL, Q8_L1 NTTFS6H888NL, Q9_H1 NTTFS6H888NL, Q9_L1 NTTFS6H888NL, U1 RFP12N10L, U10 LTV-847S, U11 LTV-847S, U12 LTV-847S, U13 LTV-847S, U14 TL084, U15 LM2596S-ADJ, U2 ADUM1250ARZ-RL7, U3 SN65HVD233, U4 SCW20C-12, U5 EC1SA16N, U6 PCA9306DC, U7 PCF8575CDB, U8 LM1117MP-3.3, U9 MCP4725xxx-xCH

Commit message: sachen halt
Parts:
- removed MH1, MH2, MH3, MH4: MountingHole_3.2mm_M3_ISO7380, MountingHole:MountingHole_3.2mm_M3_ISO7380
- removed R101: 47k, Resistor_SMD:R_0805_2012Metric
- removed U6: PCA9306DC, Package_SO:VSSOP-8_2.3x2mm_P0.5mm
- added G***: LOGO, Aktive_Bal_Footprints:Logo, F.Cu at (125.0, 85.3)
- added H1: MountingHole, MountingHole:MountingHole_3.2mm_M3, F.Cu at (125.0, 56.3)
- added H2: MountingHole, MountingHole:MountingHole_3.2mm_M3, F.Cu at (124.5, 116.3)
- added H3: MountingHole, MountingHole:MountingHole_3.2mm_M3, F.Cu at (239.0, 116.3)
- added H4: MountingHole, MountingHole:MountingHole_3.2mm_M3, F.Cu at (239.0, 22.8)
- added U16: PCA9306, Package_SO:SSOP-8_2.95x2.8mm_P0.65mm, F.Cu at (169.5, 31.6)
- J1: footprint TerminalBlock_MetzConnect:TerminalBlock_MetzConnect_Type055_RT01502HDWU_1x02_P5.00mm_Horizontal -> Aktive_Bal_Footprints:1-2-5mmTerminalBlock_MetzConnect_Type055_RT01502HDWU_1x02_P5.00mm_Horizontal_3d
- J15, J16, J17, J18, J19, J20: footprint TerminalBlock_4Ucon:TerminalBlock_4Ucon_1x03_P3.50mm_Horizontal -> Aktive_Bal_Footprints:TerminalBlock_4Ucon_1x03_P3.50mm_Horizontal_3d
- U7: footprint Package_SO:SSOP-24_5.3x8.2mm_P0.65mm -> Aktive_Bal_Footprints:PCF8575CDB_SSOP-24_5.3x8.2mm_P0.65mm
- turned C12 to 90 degrees
Connections:
- net B1 renamed /B1
- net B10 renamed /B10
- net B11 renamed /B11
- net B12 renamed /B12
- net B13 renamed /B13
- net B14 renamed /B14
- net B15 renamed /B15
- net B16 renamed /B16
- net B2 renamed /B2
- net B3 renamed /B3
- net B4 renamed /B4
- net B5 renamed /B5
- net B6 renamed /B6
- net B7 renamed /B7
- net B8 renamed /B8
- net B9 renamed /B9
- net I_Bal renamed V_I_Bal_Ist
- net I_Bal_Soll renamed V_I_Bal_Soll
- net RX renamed CRX
- net TX renamed CTX
- C1 pad 1: GNDµ -> GND
- C12 pad 1: +12V -> GND_float2
- C12 pad 2: GND_float2 -> +12V
- C2 pad 2: GNDµ -> GND
- C27 pad 2: Net-(C27-Pad2) -> V_Shunt_High
- C3 pad 1: GNDµ -> GND
- C7 pad 2: GNDµ -> GND
- J1 pad 2: Bat_GND -> GND
- J2 pad 3: GNDµ -> GND
- J22 pad 2: V_I_Bal -> V_Shunt_High
- J6 pad 2: GNDµ -> GND
- J7 pad 19: GNDµ -> GND
- Q10_L1 pad 1: V_I_Bal -> V_Shunt_High
- Q10_L1 pad 2: V_I_Bal -> V_Shunt_High
- Q10_L1 pad 3: V_I_Bal -> V_Shunt_High
- Q11_L1 pad 1: V_I_Bal -> V_Shunt_High
- Q11_L1 pad 2: V_I_Bal -> V_Shunt_High
- Q11_L1 pad 3: V_I_Bal -> V_Shunt_High
- Q12_L1 pad 1: V_I_Bal -> V_Shunt_High
- Q12_L1 pad 2: V_I_Bal -> V_Shunt_High
- Q12_L1 pad 3: V_I_Bal -> V_Shunt_High
- Q13_L1 pad 1: V_I_Bal -> V_Shunt_High
- Q13_L1 pad 2: V_I_Bal -> V_Shunt_High
- Q13_L1 pad 3: V_I_Bal -> V_Shunt_High
- Q14_L1 pad 1: V_I_Bal -> V_Shunt_High
- Q14_L1 pad 2: V_I_Bal -> V_Shunt_High
- Q14_L1 pad 3: V_I_Bal -> V_Shunt_High
- Q15_L1 pad 1: V_I_Bal -> V_Shunt_High
- Q15_L1 pad 2: V_I_Bal -> V_Shunt_High
- Q15_L1 pad 3: V_I_Bal -> V_Shunt_High
- Q16_L1 pad 1: V_I_Bal -> V_Shunt_High
- Q16_L1 pad 2: V_I_Bal -> V_Shunt_High
- Q16_L1 pad 3: V_I_Bal -> V_Shunt_High
- Q1_L1 pad 1: V_I_Bal -> V_Shunt_High
- Q1_L1 pad 2: V_I_Bal -> V_Shunt_High
- Q1_L1 pad 3: V_I_Bal -> V_Shunt_High
- Q2_L1 pad 1: V_I_Bal -> V_Shunt_High
- Q2_L1 pad 2: V_I_Bal -> V_Shunt_High
- Q2_L1 pad 3: V_I_Bal -> V_Shunt_High
- Q3_L1 pad 1: V_I_Bal -> V_Shunt_High
- Q3_L1 pad 2: V_I_Bal -> V_Shunt_High
- Q3_L1 pad 3: V_I_Bal -> V_Shunt_High
- Q4_L1 pad 1: V_I_Bal -> V_Shunt_High
- Q4_L1 pad 2: V_I_Bal -> V_Shunt_High
- Q4_L1 pad 3: V_I_Bal -> V_Shunt_High
- Q5_L1 pad 1: V_I_Bal -> V_Shunt_High
- Q5_L1 pad 2: V_I_Bal -> V_Shunt_High
- Q5_L1 pad 3: V_I_Bal -> V_Shunt_High
- Q6_L1 pad 1: V_I_Bal -> V_Shunt_High
- Q6_L1 pad 2: V_I_Bal -> V_Shunt_High
- Q6_L1 pad 3: V_I_Bal -> V_Shunt_High
- Q7_L1 pad 1: V_I_Bal -> V_Shunt_High
- Q7_L1 pad 2: V_I_Bal -> V_Shunt_High
- Q7_L1 pad 3: V_I_Bal -> V_Shunt_High
- Q8_L1 pad 1: V_I_Bal -> V_Shunt_High
- Q8_L1 pad 2: V_I_Bal -> V_Shunt_High
- Q8_L1 pad 3: V_I_Bal -> V_Shunt_High
- Q9_L1 pad 1: V_I_Bal -> V_Shunt_High
- Q9_L1 pad 2: V_I_Bal -> V_Shunt_High
- Q9_L1 pad 3: V_I_Bal -> V_Shunt_High
- R200 pad 2: Net-(C27-Pad2) -> V_Shunt_High
- R3 pad 1: GNDµ -> GND
- R4 pad 2: Bat_GND -> GND
- R92 pad 1: V_I_Bal -> V_Shunt_High
- U1 pad 3: Bat_GND -> GND
- U2 pad 4: GNDµ -> GND
- U3 pad 2: GNDµ -> GND
- U3 pad 5: GNDµ -> GND
- U3 pad 8: GNDµ -> GND
- U5 pad 1: GND_float2 -> +12V
- U5 pad 2: +12V -> GND_float2
Routing:
- net V_Shunt_High: track 0.00 -> 230.4 mm, vias 0 -> 2
- net V_I_Bal: track 224.6 -> 0.00 mm, vias 2 -> 0
- net GND: track 0.00 -> 26.2 mm, vias 0 -> 7
- net GNDµ: track 23.9 -> 0.00 mm, vias 6 -> 0
- net Net-(C27-Pad2): track 6.12 -> 0.00 mm
- net SDA3.3: track 45.8 -> 50.4 mm, vias 0 -> 1
- net +12V: track 234.6 -> 230.2 mm
- net Net-(U16-EN): track 9.04 -> 12.5 mm
- net Bat_GND: track 2.28 -> 0.00 mm, vias 1 -> 0
- net Net-(JP2-B): track 7.35 -> 8.30 mm
- net Net-(JP3-B): track 5.64 -> 6.15 mm
- added copper zone on In1.Cu, net GND
- removed copper zone on In1.Cu, net Bat_GND
- removed copper zone on In1.Cu, net GNDµ
Other:
- board text added: "A2"
- board text added: "Bat+"
- board text added: "GND_Bat"
- board text added: "GNDf"
- board text added: "elko smd aendern! C10 footprint zugroß C14 15 zu klein"
