File: KiCad/Aktive_Bal_Bericht - V8 - Doppelmosfet/Spannungsversorgung.kicad_sch (KiCad schematic)
At the start: 22 parts, among them J1 Screw_Terminal_01x02, J12 Conn_01x02_Pin, J13 Conn_01x02_Pin, J9 Conn_01x02_Pin, U1 RFP12N10L, U4 SCW20C-12, U5 EC1SA16N, U8 LM1117MP-3.3

Commit message: mosfets verkabelt elkos getauscht
Parts:
- C10: footprint Capacitor_SMD:CP_Elec_6.3x5.7 -> Capacitor_SMD:CP_Elec_5x5.3
- C14, C15: footprint Capacitor_SMD:CP_Elec_4x5.4 -> Capacitor_SMD:CP_Elec_5x5.3
Changed lines of the file:
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@@
 			)
 		)
-		(property "Footprint" "Capacitor_SMD:CP_Elec_4x5.4"
+		(property "Footprint" "Capacitor_SMD:CP_Elec_5x5.3"
 			(at 74.93 105.41 0)
 			(hide yes)
@@
 			)
 		)
-		(property "Footprint" "Capacitor_SMD:CP_Elec_6.3x5.7"
+		(property "Footprint" "Capacitor_SMD:CP_Elec_5x5.3"
 			(at 154.94 44.45 0)
 			(hide yes)
@@
 			)
 		)
-		(property "Footprint" "Capacitor_SMD:CP_Elec_4x5.4"
+		(property "Footprint" "Capacitor_SMD:CP_Elec_5x5.3"
 			(at 74.93 110.49 0)
 			(hide yes)
